File: Dome_Controller/Dome_Controller/_autosave-Dome_Controller.kicad_pcb (KiCad board)
At the start: 4 copper layers, 79 x 53 mm, 36 parts, among them J1 USB_B_Micro, J10 Conn_01x03, J2 Servo Header, J3 Conn_02x03_Odd_Even, J4 Conn_01x03, J5 12IN, J6 RSeries Logics, J7 HP, J8 HP Servo, J9 5V Out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

Commit message: Updates to some files
Parts:
- removed D1: APA102-2020, LED_SMD:LED-APA102-2020
- added L1: WS2812B-2020, Custom:WS2812B-2020, F.Cu at (121.4, 106.7)
- added REF**: KiCad-Logo2_5mm_SilkScreen, Symbol:KiCad-Logo2_5mm_SilkScreen, B.Cu at (92.2, 74.8)
- SW1: footprint Custom:GT-TC057A-H050-L1 -> Custom:TS-1101S-B-B-B-W-A
- moved C1 1.17 mm to (110.7, 97.9)
- moved R4 0.82 mm to (121.6, 102.8), turned to -90 degrees
- moved SW1 0.28 mm to (114.8, 101.6), turned to 180 degrees
- moved G*** 0.11 mm to (134.1, 105.9)
Connections:
- R4 pad 1: Net-(D1-Pad4) -> ST_LED_D
- R4 pad 2: ST_LED_D -> Net-(L1-Pad3)
- U1 pad 31: ST_LED_C -> unconnected-(U1-Pad31)
Routing:
- net ST_LED_C: track 31.7 -> 0.00 mm, vias 2 -> 0
- net +3.3V: track 119.1 -> 91.5 mm, vias 1 -> 0
- net +5V: track 157.1 -> 176.3 mm, vias 0 -> 1
- net GND: track 193.5 -> 186.5 mm
- net Net-(D1-Pad4): track 3.84 -> 0.00 mm
- net Net-(L1-Pad3): track 0.00 -> 3.18 mm
- net RESET: track 73.0 -> 73.5 mm
Other:
- outline, holes or cut-outs redrawn
- board text added: "Holo"
- board text added: "JLCJLCJLCJLC"
- board text added: "Manufactured by JLCPCB Order #:"
- board text added: "Reset"
- board text removed: "HP LED"
- board text removed: "HP Servo"
