File: Dome_Controller/Dome_Controller/Dome_Controller.kicad_pcb (KiCad board)
At the start: 4 copper layers, 79 x 53 mm, 37 parts, among them J1 USB_B_Micro, J10 Conn_01x03, J2 Servo Header, J3 Conn_02x03_Odd_Even, J4 Conn_01x03, J5 12IN, J6 RSeries Logics, J7 HP, J8 HP Servo, J9 5V Out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

Commit message: Updates to some files
Parts:
- removed D1: APA102-2020, LED_SMD:LED-APA102-2020
- removed the G*** at (134.0, 114.5)
- added L1: WS2812B-2020, Custom:WS2812B-2020, F.Cu at (121.4, 106.7)
- added REF**: KiCad-Logo2_5mm_SilkScreen, Symbol:KiCad-Logo2_5mm_SilkScreen, B.Cu at (92.2, 74.8)
- SW1: footprint Custom:GT-TC057A-H050-L1 -> Custom:TS-1101S-B-B-B-W-A
- moved C1 1.17 mm to (110.7, 97.9)
- moved R4 0.82 mm to (121.6, 102.8), turned to -90 degrees
- moved SW1 0.28 mm to (114.8, 101.6), turned to 180 degrees
- moved G*** 0.15 mm to (134.1, 105.9)
Connections:
- R4 pad 1: Net-(D1-Pad4) -> ST_LED_D
- R4 pad 2: ST_LED_D -> Net-(L1-Pad3)
- U1 pad 31: ST_LED_C -> unconnected-(U1-Pad31)
Routing:
- net ST_LED_C: track 31.7 -> 0.00 mm, vias 2 -> 0
- net +3.3V: track 119.2 -> 91.5 mm, vias 1 -> 0
- net +5V: track 157.1 -> 176.3 mm, vias 0 -> 1
- net Net-(D1-Pad4): track 3.84 -> 0.00 mm
- net Net-(L1-Pad3): track 0.00 -> 3.18 mm
- net GND: track 189.2 -> 186.5 mm
Other:
- outline, holes or cut-outs redrawn
- board text added: "Holo"
- board text added: "JLCJLCJLCJLC"
- board text added: "Manufactured by JLCPCB Order #:"
- board text added: "Reset"
- board text removed: "HP LED"
- board text removed: "HP Servo"

Commit message: updates to the boards
Parts:
- removed the G*** at (134.1, 105.9)
- added G***: LOGO, Logos:DomeControllerv2, F.Cu at (51.0, 83.7)
- added J11: Conn_02x04_Odd_Even, Connector_PinHeader_2.54mm:PinHeader_2x04_P2.54mm_Vertical, F.Cu at (133.1, 87.0)
- added J12: Conn_01x04, Connector_PinHeader_2.54mm:PinHeader_1x04_P2.54mm_Vertical, F.Cu at (133.1, 79.4)
- added J13: DB25_Female_MountingHoles, Connector_Dsub:DSUB-25_Female_Vertical_P2.77x2.84mm_MountingHoles, F.Cu at (61.8, 64.7)
- added J14: DC-005-5A-2.0, Custom:XKB_DC-005-5A-2.0, F.Cu at (76.2, 61.5)
- moved G*** 88.3 mm to (51.0, 66.7), turned to -90 degrees
- moved U5 37.7 mm to (102.0, 90.0), turned to -90 degrees
- moved U4 31.3 mm to (105.0, 97.6)
- moved C4 31.0 mm to (109.4, 92.6), turned to 90 degrees
- moved C6 29.9 mm to (100.5, 94.8), turned to 90 degrees
- moved REF** 27.3 mm to (50.0, 57.0)
- moved REF** 27.0 mm to (50.0, 103.0)
- moved J2 22.0 mm to (128.0, 97.7), turned to 90 degrees
- moved J4 17.3 mm to (135.7, 92.5), turned to 90 degrees
- moved C1 10.4 mm to (104.8, 89.3)
- moved R1 8.57 mm to (105.3, 90.7)
- moved J7 8.21 mm to (76.0, 99.6)
- moved J9 8.21 mm to (93.8, 99.5)
- moved J8 8.21 mm to (85.0, 99.5)
- moved J3 7.22 mm to (135.7, 73.3), turned to 90 degrees
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Connections:
- U1 pad 34: TXD0 -> RXD0
- U1 pad 35: RXD0 -> TXD0
Routing:
- net SR_SER_TX: track 0.00 -> 124.7 mm
- net SR_SER_RX: track 0.00 -> 116.4 mm
- net SR_I2C_DATA: track 0.00 -> 109.3 mm
- net SR_I2C_CLK: track 0.00 -> 108.7 mm
- net +12V: track 35.9 -> 104.0 mm
- net GND: track 186.5 -> 122.1 mm, vias 0 -> 1
- net unconnected-(J13-Pad0): track 0.00 -> 51.4 mm
- net RESET: track 73.5 -> 42.1 mm
- net TXD0: track 12.8 -> 41.5 mm
- net +5V: track 176.3 -> 203.4 mm
- net RXD0: track 13.3 -> 37.0 mm
- net GPIO0: track 15.7 -> 38.9 mm, vias 2 -> 0
- net +3.3V: track 91.5 -> 112.9 mm
- net D-: track 35.0 -> 15.6 mm
- net D+: track 30.3 -> 17.9 mm
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Other:
- board size 79 x 53 mm -> 107 x 57 mm
- board text added: "3V"
- board text added: "ESP Serial"
- board text added: "I2C"
- board text added: "Radar Eye"
- board text added: "Slip Ring"
- board text removed: "3.3V"
- board text removed: "Camera LEDs"
