File: Dome_Controller/Dome_Controller/Dome_Controller.kicad_sch (KiCad schematic)
At the start: 30 parts, among them J1 USB_B_Micro, J10 Conn_01x03, J2 Servo Header, J3 Conn_02x03_Odd_Even, J4 Conn_01x03, J5 12IN, J6 RSeries Logics, J7 HP, J8 HP Servo, J9 5V Out, SW1 SW_Push, U1 ESP32-WROOM-32D_16MB_, U2 CJ2301_S1, U3 ME6211C33M5G, U4 CH340C, U5 UMH3N, U6 D36V50F5-STEPDOWN

Commit message: Updates to some files
Parts:
- removed D1: APA102-2020, LED_SMD:LED-APA102-2020, symbol LED:APA102-2020
- added L1: WS2812B-2020, Custom:WS2812B-2020, symbol LED:WS2812B-2020
- C1, C3, C6: symbol Device:C_Polarized_Small_US -> Device:C; LCSC (none) -> C307331
- C2, C4: symbol Device:C_Polarized_Small_US -> Device:C; LCSC (none) -> C315248
- C5, C7: symbol Device:C_Polarized_Small_US -> Device:C; LCSC (none) -> C77009
- CR1: LCSC (none) -> C84354
- J1: LCSC (none) -> C132563
- J10, J4: LCSC (none) -> C49257
- J2: LCSC (none) -> C37208
- J3: LCSC (none) -> C492420
- J5, J6, J7, J8, J9: LCSC (none) -> C474892
- R1: LCSC (none) -> C269701
- R2, R3: LCSC (none) -> C25803
- R4: LCSC (none) -> C25091
- SW1: footprint Custom:GT-TC057A-H050-L1 -> Custom:TS-1101S-B-B-B-W-A; LCSC (none) -> C692465
- U1: LCSC (none) -> C529578
- U2: LCSC (none) -> C8547
- U3: LCSC (none) -> C82942
- U4: LCSC (none) -> C84681
- U5: LCSC (none) -> C62892
Connections:
- net +5V: now also L1.4 (VDD)
- net GND: now also L1.2 (VSS)
- net ST_LED_D: now also R4.1; no longer R4.2
- net ST_LED_C: no longer names the net of U1.31 (IO19)
- new net: L1.3 (DI), R4.2
- no-connect marks 34 -> 35

Commit message: updates to the boards
Parts:
- added J11: Conn_02x04_Odd_Even, Connector_PinHeader_2.54mm:PinHeader_2x04_P2.54mm_Vertical, symbol Connector_Generic:Conn_02x04_Odd_Even
- added J12: Conn_01x04, Connector_PinHeader_2.54mm:PinHeader_1x04_P2.54mm_Vertical, symbol Connector_Generic:Conn_01x04
- added J13: DB25_Female_MountingHoles, Connector_Dsub:DSUB-25_Female_Vertical_P2.77x2.84mm_MountingHoles, symbol Connector:DB25_Female_MountingHoles
- added J14: DC-005-5A-2.0, Custom:XKB_DC-005-5A-2.0, symbol Custom:DC-005-5A-2.0
Connections:
- net +12V: now also J13.1, J13.12, J13.13, J13.14 (P14), J13.15 (P15), J13.2, J13.24 (P24), J13.25 (P25), J14.1
- net +5V: now also J11.1 (Pin_1), J11.2 (Pin_2), J12.1 (Pin_1), J13.20 (P20), J13.5
- net GND: now also J11.3 (Pin_3), J11.4 (Pin_4), J12.2 (Pin_2), J13.10, J13.11, J13.16 (P16), J13.17 (P17), J13.18 (P18), J13.22 (P22), J13.23 (P23), J13.3, J13.4, J13.8, J14.2, J14.3
- net RXD0: now also U1.34 (RXD0); no longer U1.35 (TXD0)
- net TXD0: now also U1.35 (TXD0); no longer U1.34 (RXD0)
- new net SR_I2C_CLK: J11.5 (Pin_5), J11.6 (Pin_6), J13.6
- new net SR_I2C_DATA: J11.7 (Pin_7), J11.8 (Pin_8), J13.19 (P19)
- new net SR_SER_RX: J12.4 (Pin_4), J13.9
- new net SR_SER_TX: J12.3 (Pin_3), J13.21 (P21)
- no-connect marks 35 -> 37
Other:
- note added: "LEDs"
- note removed: "Status LED"
- moved on the sheet: C1, C2, C3, C4, C5, C6, C7, CR1, J1, J10, J2, J3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
