File: Body_LED_Controller_Embedded_ESP32/Body_LED_Controller_Embedded_ESP32s.kicad_pcb (KiCad board)
At the start: 4 copper layers, 114 x 73 mm, 109 parts, among them J1 SERIAL, J10 USB_B_Micro, J11 USB_B_Micro, J12 USB_B_Micro, J13 Conn_02x03_Odd_Even, J14 Conn_01x03, J15 Servo Header, J16 Screw_Terminal_01x02, J17 Screw_Terminal_01x02, J18 Screw_Terminal_01x02, J19 Screw_Terminal_01x02, J2 I2C, J20 ICSP, J3 Conn_02x10_Odd_Even, J4 LDP/MAINT, J5 COIN/VU, J6 Batt Level LEDS, J7 Data Panel/ CBI, J8 Spectrum Analyzer, J9 Ext Mic, SW1 SW_Push, SW2 SW_Push, SW3 SW_Push, U1 ATMEGA256016AU, U10 CH340C, U11 UMH3N, U12 ME6211C33M5G, U13 CJ2301_S1, U14 D36V50F5-STEPDOWN, U2 CH340C, U3 CJ2301_S1, U4 ESP32-WROOM-32U_16MB_, U5 CH340C, U6 UMH3N, U7 ME6211C33M5G, U8 CJ2301_S1, U9 ESP32-WROOM-32D_16MB_, Y1 16MHz

Commit message: Updated the body Controller to have SMA and u.fl interfaces for the 32U
Parts:
- added J21: CONSMA008, Custom:LINX_CONSMA008, F.Cu at (183.1, 100.6)
- added J22: U.FL-R-SMT-1(01), Custom:HIROSE_U.FL-R-SMT-1(01), F.Cu at (161.5, 96.1)
Routing:
- net Net-(J21-PadS1): track 0.00 -> 40.7 mm
- net Net-(J21-Pad1): track 0.00 -> 26.6 mm
- net RESET_BL: track 178.9 -> 178.1 mm

Commit message: Updates to some files
Parts:
- removed D3, D4, D5: APA102-2020, LED_SMD:LED-APA102-2020
- removed J21: CONSMA008, Custom:LINX_CONSMA008
- removed J22: U.FL-R-SMT-1(01), Custom:HIROSE_U.FL-R-SMT-1(01)
- removed RN1: 10K, Custom:SOIC127P762X240-14N
- added L1: WS2812B-2020, Custom:WS2812B-2020, F.Cu at (100.9, 117.3)
- added L2: WS2812B-2020, Custom:WS2812B-2020, F.Cu at (155.2, 117.2)
- added L3: WS2812B-2020, Custom:WS2812B-2020, F.Cu at (174.7, 117.3)
- added R29: 10K, Resistor_SMD:R_0402_1005Metric, F.Cu at (128.7, 95.8)
- added R30: 10K, Resistor_SMD:R_0402_1005Metric, F.Cu at (128.7, 94.6)
- added R31: 10K, Resistor_SMD:R_0402_1005Metric, F.Cu at (128.7, 93.3)
- added R32: 10K, Resistor_SMD:R_0402_1005Metric, F.Cu at (128.7, 92.0)
- added R33: 10K, Resistor_SMD:R_0402_1005Metric, F.Cu at (128.7, 90.8)
- added R34: 10K, Resistor_SMD:R_0402_1005Metric, F.Cu at (128.7, 89.5)
- added R35: 10K, Resistor_SMD:R_0402_1005Metric, F.Cu at (122.8, 90.2)
- added R36: 10K, Resistor_SMD:R_0402_1005Metric, F.Cu at (122.8, 91.3)
- added R37: 10K, Resistor_SMD:R_0402_1005Metric, F.Cu at (122.8, 92.5)
- added R38: 10K, Resistor_SMD:R_0402_1005Metric, F.Cu at (122.8, 93.7)
- D1, D2: value LED -> SMD-LED-CLEAR-BLUE(0402); footprint LED_SMD:LED_0402_1005Metric -> Custom:LED-0402
- moved D2 0.07 mm to (109.6, 72.9)
Connections:
- R15 pad 1: +5V_BL -> GND
- R15 pad 2: Net-(D1-Pad2) -> Net-(D1-Pad-)
- R16 pad 1: +5V_BL -> GND
- R16 pad 2: Net-(D2-Pad2) -> Net-(D2-Pad-)
- U1 pad 16: ST_LED_C_BL -> unconnected-(U1-Pad16)
- U4 pad 31: ST_LED_C_BC -> unconnected-(U4-Pad31)
- U9 pad 31: ST_LED_C_BS -> unconnected-(U9-Pad31)
Routing:
- net ST_LED_C_BL: track 92.1 -> 0.00 mm, vias 2 -> 0
- net Net-(J21-PadS1): track 40.7 -> 0.00 mm
- net Net-(J21-Pad1): track 26.6 -> 0.00 mm
- net ST_LED_C_BC: track 24.2 -> 0.00 mm, vias 2 -> 0
- net GND: track 262.6 -> 285.6 mm, vias 24 -> 23
- net ST_LED_C_BS: track 12.1 -> 0.00 mm, vias 2 -> 0
- net +5V_BL: track 205.1 -> 196.4 mm
- net +3.3V_BC: track 90.6 -> 92.8 mm
- net Net-(D2-Pad-): track 0.00 -> 1.14 mm
- net Net-(D2-Pad2): track 1.06 -> 0.00 mm
- net Net-(D1-Pad2): track 1.02 -> 0.00 mm
- net Net-(D1-Pad-): track 0.00 -> 0.98 mm
- net +3.3V_BS: track 79.7 -> 78.9 mm
- net LIMIT8: track 45.3 -> 46.0 mm
- net Net-(R26-Pad1): track 1.44 -> 2.02 mm
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
Commit message: updates to the boards
Connections:
- U1 pad 2: TXD0_BL -> RXD0_BL
- U1 pad 3: RXD0_BL -> TXD0_BL
- U4 pad 34: TXD0_BC -> unconnected-(U4-Pad34)
- U4 pad 35: RXD0_BC -> TXD0_BC
- U9 pad 34: TXD0_BS -> RXD0_BS
- U9 pad 35: RXD0_BS -> TXD0_BS
