File: Body_Servos/Body_Servos/Body_Servos.kicad_pcb (KiCad board)
At the start: 4 copper layers, 80 x 55.1 mm, 38 parts, among them J1 USB_B_Micro, J12 SERIAL_FU, J2 AUX3, J3 AUX1, J4 AUX2, J5 12OUT, J6 12VOUT, J7 5V OUT, J8 5V Out 2, SW1 SW_Push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

Commit message: added LED PCBs
Changed lines of the file:
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@@
       (drillshape 0)
       (scaleselection 1)
-      (outputdirectory "Gerber/Dome_ControllerV2.0/")
+      (outputdirectory "BOM and CPL/")
     )
   )
@@
     (fp_line (start -1.27 -2.92) (end -1.27 2.88) (layer "F.Fab") (width 0.1))
     (fp_line (start -1.27 2.88) (end 8.89 2.88) (layer "F.Fab") (width 0.1))
-    (pad "1" thru_hole roundrect locked (at 0 0 90) (size 1.74 2.19) (drill 1.19) (layers *.Cu *.Mask) (roundrect_rratio 0.143678)
+    (pad "1" thru_hole roundrect locked (at 0 0 90) (size 1.74 2.19) (drill 1.19) (layers *.Cu *.Mask) (roundrect_rratio 0.1436781609)
       (net 2 "GND") (pinfunction "Pin_1") (pintype "passive"))
     (pad "2" thru_hole oval locked (at 2.54 0 90) (size 1.74 2.19) (drill 1.19) (layers *.Cu *.Mask)
@@
     (fp_line (start -0.562893 0) (end -1.27 0.5) (layer "F.Fab") (width 0.1))
     (fp_line (start 8.89 -2.92) (end -1.27 -2.92) (layer "F.Fab") (width 0.1))
-    (pad "1" thru_hole roundrect locked (at 0 0 90) (size 1.74 2.19) (drill 1.19) (layers *.Cu *.Mask) (roundrect_rratio 0.143678)
+    (pad "1" thru_hole roundrect locked (at 0 0 90) (size 1.74 2.19) (drill 1.19) (layers *.Cu *.Mask) (roundrect_rratio 0.1436781609)
       (net 2 "GND") (pinfunction "Pin_1") (pintype "passive"))
     (pad "2" thru_hole oval locked (at 2.54 0 90) (size 1.74 2.19) (drill 1.19) (layers *.Cu *.Mask)
@@
     (fp_line (start -1.27 -2.92) (end -1.27 2.88) (layer "F.Fab") (width 0.1))
     (fp_line (start 8.89 2.88) (end 8.89 -2.92) (layer "F.Fab") (width 0.1))
-    (pad "1" thru_hole roundrect locked (at 0 0 90) (size 1.74 2.19) (drill 1.19) (layers *.Cu *.Mask) (roundrect_rratio 0.143678)
+    (pad "1" thru_hole roundrect locked (at 0 0 90) (size 1.74 2.19) (drill 1.19) (layers *.Cu *.Mask) (roundrect_rratio 0.1436781609)
       (net 2 "GND") (pinfunction "Pin_1") (pintype "passive"))
     (pad "2" thru_hole oval locked (at 2.54 0 90) (size 1.74 2.19) (drill 1.19) (layers *.Cu *.Mask)
@@
     (fp_line (start 6.35 -2.92) (end -1.27 -2.92) (layer "F.Fab") (width 0.1))
     (fp_line (start 6.35 2.88) (end 6.35 -2.92) (layer "F.Fab") (width 0.1))
-    (pad "1" thru_hole roundrect locked (at 0 0 90) (size 1.74 2.19) (drill 1.19) (layers *.Cu *.Mask) (roundrect_rratio 0.143678)
+    (pad "1" thru_hole roundrect locked (at 0 0 90) (size 1.74 2.19) (drill 1.19) (layers *.Cu *.Mask) (roundrect_rratio 0.1436781609)
       (net 2 "GND") (pinfunction "Pin_1") (pintype "passive"))
     (pad "2" thru_hole oval locked (at 2.54 0 90) (size 1.74 2.19) (drill 1.19) (layers *.Cu *.Mask)
