File: Dome_Plate_Controller/Dome_Plate_Controller_V1/Dome_Plate_Controller_V1.kicad_pcb (KiCad board)
At the start: 4 copper layers, 104.2 x 154 mm, 36 parts, among them J1 USB_B_Micro, J10 SERIAL_FU4, J11 SERIAL_FU3, J12 SERIAL_FU, J13 DB25_Female_MountingHoles, J14 DC-005-5A-2.0, J15 SERIAL_FU2, J2 DB25_Female_MountingHoles, J3 12VOUT, J4 SERIAL_RS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

Commit message: Working on new body control board
Parts:
- added G***: LOGO, Logos:R2_Logo_V2, F.Cu at (77.6, 109.7)
- added G***: LOGO, Logos:R2_Logo_V2, F.Cu at (118.6, 109.7)
- added G***: LOGO, Logos:DomePlateLogoWords, F.Cu at (97.9, 109.0)
- added REF**: MountingHole_3.2mm_M3, MountingHole:MountingHole_3.2mm_M3, F.Cu at (45.9, 101.1)
- added REF**: MountingHole_3.2mm_M3, MountingHole:MountingHole_3.2mm_M3, F.Cu at (132.7, 138.0)
- added REF**: MountingHole_3.2mm_M3, MountingHole:MountingHole_3.2mm_M3, F.Cu at (67.7, 138.5)
- added REF**: MountingHole_3.2mm_M3, MountingHole:MountingHole_3.2mm_M3, F.Cu at (128.0, 89.4)
- J13: value DB25_Female_MountingHoles -> DB25_Female_MagTag
- J2: value DB25_Female_MountingHoles -> DB25_Male_SlipRing; footprint Connector_Dsub:DSUB-25_Female_Vertical_P2.77x2.84mm_MountingHoles -> Connector_Dsub:DSUB-25_Male_Vertical_P2.77x2.84mm_MountingHoles
- moved REF** 146.1 mm to (100.4, 106.5)
- moved J8 88.3 mm to (65.3, 98.4), turned to -155 degrees
- moved J7 76.1 mm to (74.0, 95.2), turned to -160 degrees
- moved J3 66.2 mm to (65.2, 121.8), turned to -60 degrees
- moved C7 65.4 mm to (89.8, 102.5), turned to -90 degrees
- moved J13 64.1 mm to (83.2, 150.5), turned to 180 degrees
- moved J6 57.6 mm to (60.6, 113.7), turned to -60 degrees
- moved J9 56.8 mm to (82.9, 92.4), turned to -165 degrees
- moved C2 54.7 mm to (88.3, 85.9), turned to 180 degrees
- moved J1 54.2 mm to (120.1, 86.3), turned to 168 degrees
- moved C5 50.0 mm to (78.7, 99.2)
- moved J5 49.4 mm to (55.9, 105.9), turned to -60 degrees
- moved C3 48.1 mm to (88.4, 84.6), turned to 180 degrees
- moved U2 46.4 mm to (75.3, 101.7), turned to 180 degrees
- moved U1 44.4 mm to (100.1, 91.5), turned to 0 degrees
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Connections:
- U1 pad 8: TX_FU2 -> unconnected-(U1-Pad8)
- U1 pad 9: RX_FU2 -> unconnected-(U1-Pad9)
Routing:
- net +12V: track 0.00 -> 257.8 mm
- net VBUS: track 0.00 -> 143.8 mm
- net +5V: track 0.00 -> 128.0 mm, vias 0 -> 1
- net D+: track 0.00 -> 95.6 mm, vias 0 -> 1
- net GND: track 0.00 -> 89.1 mm, vias 0 -> 6
- net D-: track 0.00 -> 89.0 mm, vias 0 -> 1
- net +3.3V: track 0.00 -> 85.9 mm, vias 0 -> 3
- net TX_FU4: track 0.00 -> 53.6 mm, vias 0 -> 1
- net RX_FU4: track 0.00 -> 52.6 mm, vias 0 -> 1
- net RX_FU3: track 0.00 -> 43.1 mm, vias 0 -> 1
- net TX_FU3: track 0.00 -> 39.0 mm, vias 0 -> 1
- net RESET: track 0.00 -> 38.1 mm, vias 0 -> 2
- net RX_FU2: track 0.00 -> 36.0 mm, vias 0 -> 1
- net RX_FU: track 0.00 -> 34.5 mm, vias 0 -> 1
- net TX_FU2: track 0.00 -> 31.6 mm, vias 0 -> 1
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- added copper zone on B.Cu, net GND
Other:
- board size 104.2 x 154 mm -> 118 x 78.6 mm
- board text added: "+"
- board text added: "-"
- board text added: "5V OUT"
- board text added: "Future 1"
- board text added: "Future 2"
- board text added: "Future 3"
- board text added: "Future 4"
- board text added: "G"
- board text added: "Rx"
- board text added: "SERIAL"
- board text added: "Tx"
- board text added: "UNREGULATED OUT"
- board text added: "Uppity Spinner"

Commit message: Added a lot since last check in
Parts:
- J4: value SERIAL_RS -> SERIAL_US
Connections:
- J13 pad 20: VBUS -> unconnected-(J13-Pad20)
- J13 pad 21: D- -> unconnected-(J13-Pad21)
- J13 pad 8: GND -> unconnected-(J13-Pad8)
- J13 pad 9: D+ -> unconnected-(J13-Pad9)
Routing:
- net +12V: track 257.8 -> 510.7 mm
- net unconnected-(J2-Pad0): track 0.00 -> 53.2 mm
- net unconnected-(J13-Pad0): track 0.00 -> 51.6 mm
- net D+: track 95.6 -> 77.8 mm
- net VBUS: track 143.8 -> 131.8 mm
- net D-: track 89.0 -> 76.9 mm

Commit message: added LED PCBs
Changed lines of the file:
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@@
       (drillshape 0)
       (scaleselection 1)
-      (outputdirectory "Gerber/Dome_ControllerV2.0/")
+      (outputdirectory "BOM and CPL/")
     )
   )
@@
     (fp_line (start -1.27 -0.5) (end -0.562893 0) (layer "F.Fab") (width 0.1))
     (fp_line (start -1.27 2.88) (end 6.35 2.88) (layer "F.Fab") (width 0.1))
-    (pad "1" thru_hole roundrect locked (at 0 0 90) (size 1.74 2.19) (drill 1.19) (layers *.Cu *.Mask) (roundrect_rratio 0.143678)
+    (pad "1" thru_hole roundrect locked (at 0 0 90) (size 1.74 2.19) (drill 1.19) (layers *.Cu *.Mask) (roundrect_rratio 0.1436781609)
       (net 2 "GND") (pinfunction "Pin_1") (pintype "passive"))
     (pad "2" thru_hole oval locked (at 2.54 0 90) (size 1.74 2.19) (drill 1.19) (layers *.Cu *.Mask)
@@
     (fp_line (start 6.35 -2.92) (end -1.27 -2.92) (layer "F.Fab") (width 0.1))
     (fp_line (start 6.35 2.88) (end 6.35 -2.92) (layer "F.Fab") (width 0.1))
-    (pad "1" thru_hole roundrect locked (at 0 0 90) (size 1.74 2.19) (drill 1.19) (layers *.Cu *.Mask) (roundrect_rratio 0.143678)
+    (pad "1" thru_hole roundrect locked (at 0 0 90) (size 1.74 2.19) (drill 1.19) (layers *.Cu *.Mask) (roundrect_rratio 0.1436781609)
       (net 2 "GND") (pinfunction "Pin_1") (pintype "passive"))
     (pad "2" thru_hole oval locked (at 2.54 0 90) (size 1.74 2.19) (drill 1.19) (layers *.Cu *.Mask)
@@
     (fp_line (start -1.27 -2.92) (end -1.27 2.88) (layer "F.Fab") (width 0.1))
     (fp_line (start 6.35 -2.92) (end -1.27 -2.92) (layer "F.Fab") (width 0.1))
-    (pad "1" thru_hole roundrect locked (at 0 0 90) (size 1.74 2.19) (drill 1.19) (layers *.Cu *.Mask) (roundrect_rratio 0.143678)
+    (pad "1" thru_hole roundrect locked (at 0 0 90) (size 1.74 2.19) (drill 1.19) (layers *.Cu *.Mask) (roundrect_rratio 0.1436781609)
       (net 2 "GND") (pinfunction "Pin_1") (pintype "passive"))
     (pad "2" thru_hole oval locked (at 2.54 0 90) (size 1.74 2.19) (drill 1.19) (layers *.Cu *.Mask)
@@
     (fp_line (start 6.35 2.88) (end 6.35 -2.92) (layer "F.Fab") (width 0.1))
     (fp_line (start -1.27 -2.92) (end -1.27 2.88) (layer "F.Fab") (width 0.1))
-    (pad "1" thru_hole roundrect locked (at 0 0 90) (size 1.74 2.19) (drill 1.19) (layers *.Cu *.Mask) (roundrect_rratio 0.143678)
+    (pad "1" thru_hole roundrect locked (at 0 0 90) (size 1.74 2.19) (drill 1.19) (layers *.Cu *.Mask) (roundrect_rratio 0.1436781609)
       (net 2 "GND") (pinfunction "Pin_1") (pintype "passive"))
     (pad "2" thru_hole oval locked (at 2.54 0 90) (size 1.74 2.19) (drill 1.19) (layers *.Cu *.Mask)
@@
     (fp_line (start -1.27 -0.5) (end -0.562893 0) (layer "F.Fab") (width 0.1))
     (fp_line (start -1.27 2.88) (end 6.35 2.88) (layer "F.Fab") (width 0.1))
-    (pad "1" thru_hole roundrect locked (at 0 0 90) (size 1.74 2.19) (drill 1.19) (layers *.Cu *.Mask) (roundrect_rratio 0.143678)
+    (pad "1" thru_hole roundrect locked (at 0 0 90) (size 1.74 2.19) (drill 1.19) (layers *.Cu *.Mask) (roundrect_rratio 0.1436781609)
       (net 2 "GND") (pinfunction "Pin_1") (pintype "passive"))
     (pad "2" thru_hole oval locked (at 2.54 0 90) (size 1.74 2.19) (drill 1.19) (layers *.Cu *.Mask)
