File: Body_LED_Controller_V2/Body_LED_Controller_V2.kicad_sch (KiCad schematic)
At the start: 92 parts, among them J1 Body Servos, J10 USB_B_Micro, J11 USB_B_Micro, J12 UnSW_BATT_IN, J13 Batt Level LEDS, J14 DomeControllerUSB, J15 DomePlateControllerUSB, J16 UnSW_BATT_PASS, J17 RADH_POW, J18 RASP_POW, J19 5V_OUT_3, J2 Body Servos, J20 ICSP, J21 DomeElectronicsPowerIn, J22 DB25_Male_MountingHoles, J23 Amplifier_POW, J24 Future, J25 Stealth, J26 RADH, J27 VU Data Panel, J3 Conn_02x10_Odd_Even, J4 LDP, J5 Coin Slots, J6 Batt Level LEDS, J7 Data Panel/ CBI, J8 Spectrum Analyzer, J9 Maintenance, SW1 SW_Push, SW2 SW_Push, U1 ATMEGA256016AU, U14 D36V50F5-STEPDOWN, U2 CH340C, U3 CJ2301_S1, U4 ESP32-WROOM-32D_16MB_, U5 CH340C, U6 UMH3N, U7 ME6211C33M5G, U8 CJ2301_S1, Y1 16MHz

Commit message: Added custom libraries and updated the Kill Switch (Remote)
Connections:
- net +5V_BL: now also C5.1, U2.4 (V3)
Changed lines of the file:
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@@
   (junction (at 275.59 194.31) (diameter 0) (color 0 0 0 0)
   )
+  (junction (at 222.25 24.13) (diameter 0) (color 0 0 0 0)
+  )
   (junction (at 250.19 54.61) (diameter 0) (color 0 0 0 0)
   )
@@
   )
   (junction (at 267.97 204.47) (diameter 0) (color 0 0 0 0)
+  )
+  (junction (at 222.25 26.67) (diameter 0) (color 0 0 0 0)
   )
   (no_connect (at 44.45 226.06))
@@
     (stroke (width 0) (type default) (color 0 0 0 0))
   )
+  (wire (pts (xy 222.25 24.13) (xy 218.44 24.13))
+    (stroke (width 0) (type default) (color 0 0 0 0))
+  )
   (wire (pts (xy 262.89 256.54) (xy 267.97 256.54))
     (stroke (width 0) (type default) (color 0 0 0 0))
@@
     (stroke (width 0) (type default) (color 0 0 0 0))
   )
+  (wire (pts (xy 222.25 24.13) (xy 222.25 26.67))
+    (stroke (width 0) (type default) (color 0 0 0 0))
+  )
   (wire (pts (xy 24.13 246.38) (xy 24.13 248.92))
     (stroke (width 0) (type default) (color 0 0 0 0))
@@
     (stroke (width 0) (type default) (color 0 0 0 0))
   )
-  (wire (pts (xy 218.44 26.67) (xy 228.6 26.67))
+  (wire (pts (xy 218.44 26.67) (xy 222.25 26.67))
     (stroke (width 0) (type default) (color 0 0 0 0))
   )
@@
     (stroke (width 0) (type default) (color 0 0 0 0))
   )
+  (wire (pts (xy 222.25 26.67) (xy 228.6 26.67))
+    (stroke (width 0) (type default) (color 0 0 0 0))
+  )
   (wire (pts (xy 405.13 24.13) (xy 405.13 26.67))
     (stroke (width 0) (type default) (color 0 0 0 0))
@@
     (stroke (width 0) (type default) (color 0 0 0 0))
   )
+  (wire (pts (xy 224.79 24.13) (xy 222.25 24.13))
+    (stroke (width 0) (type default) (color 0 0 0 0))
+  )
   (polyline (pts (xy 199.39 264.16) (xy 106.68 264.16))
     (stroke (width 0.5) (type default) (color 255 0 255 1))
@@
     )
   )
-  (global_label "+5V_BL" (shape input) (at 218.44 24.13 0) (fields_autoplaced)
-    (effects (font (size 1.27 1.27)) (justify left))
-    (property "Intersheet References" "${INTERSHEET_REFS}" (id 0) (at 227.9004 24.0506 0)
-      (effects (font (size 1.27 1.27)) (justify left) hide)
-    )
+  (global_label "+5V_BL" (shape input) (at 224.79 24.13 0) (fields_autoplaced)
+    (effects (font (size 1.27 1.27)) (justify left))
+    (property "Intersheet References" "${INTERSHEET_REFS}" (id 0) (at 234.2504 24.0506 0)
+      (effects (font (size 1.27 1.27)) (justify left) hide)
+    )

Commit message: Working on boards
Connections:
- net +5V_BL: no longer C5.1, U2.4 (V3)
- new net: C5.1, U2.4 (V3)
Changed lines of the file:
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@@
   (junction (at 275.59 194.31) (diameter 0) (color 0 0 0 0)
   )
-  (junction (at 222.25 24.13) (diameter 0) (color 0 0 0 0)
-  )
   (junction (at 250.19 54.61) (diameter 0) (color 0 0 0 0)
   )
@@
   )
   (junction (at 267.97 204.47) (diameter 0) (color 0 0 0 0)
-  )
-  (junction (at 222.25 26.67) (diameter 0) (color 0 0 0 0)
   )
   (no_connect (at 44.45 226.06))
@@
     (stroke (width 0) (type default) (color 0 0 0 0))
   )
-  (wire (pts (xy 222.25 24.13) (xy 218.44 24.13))
+  (wire (pts (xy 218.44 24.13) (xy 224.79 24.13))
     (stroke (width 0) (type default) (color 0 0 0 0))
   )
@@
     (stroke (width 0) (type default) (color 0 0 0 0))
   )
-  (wire (pts (xy 222.25 24.13) (xy 222.25 26.67))
-    (stroke (width 0) (type default) (color 0 0 0 0))
-  )
   (wire (pts (xy 24.13 246.38) (xy 24.13 248.92))
     (stroke (width 0) (type default) (color 0 0 0 0))
@@
     (stroke (width 0) (type default) (color 0 0 0 0))
   )
-  (wire (pts (xy 218.44 26.67) (xy 222.25 26.67))
+  (wire (pts (xy 218.44 26.67) (xy 228.6 26.67))
     (stroke (width 0) (type default) (color 0 0 0 0))
   )
@@
     (stroke (width 0) (type default) (color 0 0 0 0))
   )
-  (wire (pts (xy 222.25 26.67) (xy 228.6 26.67))
-    (stroke (width 0) (type default) (color 0 0 0 0))
-  )
   (wire (pts (xy 405.13 24.13) (xy 405.13 26.67))
     (stroke (width 0) (type default) (color 0 0 0 0))
@@
     (stroke (width 0) (type default) (color 0 0 0 0))
   )
-  (wire (pts (xy 224.79 24.13) (xy 222.25 24.13))
-    (stroke (width 0) (type default) (color 0 0 0 0))
-  )
