File: In Progress/Kill_Switch_Remote/Kill_Switch_Remote.kicad_sch (KiCad schematic)
At the start: 51 parts, among them J1 USB_B_Micro, J2 S2B-PH-K-S(LF)(SN), J3 U.FL-R-SMT-1(10), Q2 UMH3N, SW4 AS11CH, U1 ESP32-PICO-MINI-02, U2 CP2102N-A02-GQFN28, U3 LP5912-3.3DRV, U4 MCP73871-2CC-Custom, U5 RFM95W-915S2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

Commit message: Working on boards
Parts:
- D4: Digikey Part Number 754-1356-1-ND -> 160-1423-1-ND; LCSC ------ -> C913075; Manufacturers Name Kingbright -> Lite-On Inc.; Manufacturers Part Number APG1608ZGC -> LTST-C171GKT; Mouser Part Number 604-APG1608ZGC -> 859-LTST-C171GKT
- D5: Digikey Part Number 160-1837-1-ND -> 160-1579-1-ND; LCSC C575417 -> C98222; Manufacturers Part Number LTST-C194TBKT -> LTST-C170TBKT; Mouser Part Number 859-LTST-C194TBKT -> 859-LTST-C170TBKT
- L1, L2, L3: value WS2812B-2020 -> WS2812B; Digikey Part Number 1528-4684-ND -> 1568-COM-16347CT-ND; LCSC C965555 -> C114586; Manufacturers Name Worldsemi/Adafruit -> SparkFun Electronics; Manufacturers Part Number WS2812B-2020/4684 -> COM-16347
- S2, S3: footprint Custom:KillSwiitch -> Custom:SW_TL3305BF260QG; Digikey Part Number EG2531CT-ND -> EG5355CT-ND; LCSC ------ -> C2886904; Manufacturers Part Number TL3342F160QG/TR -> TL3305CF260QG; Mouser Part Number ------ -> 612-TL3305CF260QG
Other:
- note removed: "Update: Blue Discrete LED - PN's Green Discrete LED - PN's SW2 and SW3 - PN's L1,L2,L3 - PN's"
