File: In Progress/Kill_Switch_Remote/_autosave-Kill_Switch_Remote.kicad_sch (KiCad schematic)
At the start: 36 parts, among them J1 USB_B_Micro, J3 U.FL-R-SMT-1(10), Q2 UMH3N, U1 ESP32-PICO-MINI-02, U2 CP2102N-A02-GQFN28, U3 LP5912-3.3DRV, U5 RFM95W-915S2, U6 LS18-S(Debouce)

Commit message: Working on boards
Parts:
- removed J?: Screw_Terminal_01x02, symbol Connector:Screw_Terminal_01x02
- removed U?: D24V550F5_Step_Down_Regulator, symbol Pololu:D24V550F5_Step_Down_Regulator
- added C8: 10uF, Capacitor_SMD:C_0805_2012Metric, symbol Device:C_Small
- added C9: 4.7uF, Capacitor_SMD:C_0603_1608Metric, symbol Device:C_Small
- added D3: SMAJ5.0, Custom:SMAJ5.0_DIOM4325X250N, symbol Custom:SMAJ5.0
- added D4: Green, LED_SMD:LED_0805_2012Metric_Pad1.15x1.40mm_HandSolder, symbol Device:LED
- added D5: BLUE, LED_SMD:LED_0805_2012Metric_Pad1.15x1.40mm_HandSolder, symbol Device:LED
- added D6: Red, LED_SMD:LED_0805_2012Metric_Pad1.15x1.40mm_HandSolder, symbol Device:LED
- added J2: S2B-PH-K-S(LF)(SN), Custom:JST_S2B-PH-K-S(LF)(SN), symbol Custom:S2B-PH-K-S(LF)(SN)
- added R10: 10K, Resistor_SMD:R_0402_1005Metric, symbol Device:R_Small
- added R11, R12, R13: 100K, Resistor_SMD:R_0402_1005Metric, symbol Device:R_Small
- added R7, R8: 82, Resistor_SMD:R_0402_1005Metric, symbol Device:R_Small
- added R9: 150, Resistor_SMD:R_0402_1005Metric, symbol Device:R_Small
- added SW4: AS11CH, Custom:AS11CH, symbol Custom:AS11CH
- added TH1: 10K, Capacitor_SMD:C_0603_1608Metric, symbol Device:Thermistor_NTC
- added U4: MCP73871-2CC-Custom, Package_DFN_QFN:QFN-20-1EP_4x4mm_P0.5mm_EP2.7x2.7mm_ThermalVias, symbol Custom:MCP73871-2CC-Custom
- L1, L2, L3: value WS2812B-2020 -> WS2812B; Digikey Part Number 1528-4684-ND -> 1568-COM-16347CT-ND; LCSC C965555 -> C114586; Manufacturers Name Worldsemi/Adafruit -> SparkFun Electronics; Manufacturers Part Number WS2812B-2020/4684 -> COM-16347
- S2, S3: footprint Custom:KillSwiitch -> Custom:SW_TL3305BF260QG; Digikey Part Number EG2531CT-ND -> EG5355CT-ND; LCSC ------ -> C2886904; Manufacturers Part Number TL3342F160QG/TR -> TL3305CF260QG; Mouser Part Number ------ -> 612-TL3305CF260QG
Connections:
- net GND: now also C8.2, C9.2, D3.A, J2.2, R10.2, R11.2, R13.1, TH1.2, U4.10 (GND), U4.11 (GND), U4.3 (SEL), U4.4 (PROG2), U4.9 (TE)
- net VBUS: now also C8.1, D3.C, D4.2 (A), D5.2 (A), D6.2 (A), U4.17 (CE), U4.18 (IN), U4.19 (IN), U4.2 (VPCC)
- net at C6.2, U3.4 (EN), U3.6 (IN): now also U4.1 (OUT), U4.20 (OUT)
- new net: J2.1, SW4.3
- new net: R9.1, U4.8 (STAT1/LBO)
- new net: D6.1 (K), R9.2
- new net: D4.1 (K), R7.2
- new net: R7.1, U4.6 (PG)
- new net: R11.1, U4.12 (PROG3)
- new net: R10.1, U4.13 (PROG1)
- new net: C9.1, R12.2, SW4.1, U4.14 (VBAT), U4.15 (VBAT), U4.16 (VBAT)
- new net: TH1.1, U4.5 (THERM)
- new net: R8.1, U4.7 (STAT2)
- new net: D5.1 (K), R8.2
- new net BATT_LEVEL: R12.1, R13.2
Other:
- note added: "Power/Battery Charging"
- note removed: "Power"
- note removed: "Update: Blue Discrete LED - PN's Green Discrete LED - PN's SW2 and SW3 - PN's L1,L2,L3 - PN's"
- moved on the sheet: C6, C7, U3
