File: In Progress/Kill_Switch_Droid/Kill_Switch_Droid.kicad_pcb (KiCad board)
At the start: 4 copper layers, 65 x 27 mm, 58 parts, among them J1 USB_B_Micro, J2 S2B-PH-K-S(LF)(SN), J3 U.FL-R-SMT-1(10), Q2 UMH3N, SW4 AS11CH, U1 ESP32-PICO-MINI-02, U2 CP2102N-A02-GQFN28, U3 LP5912-3.3DRV, U4 MCP73871-2CC-Custom, U5 RFM95W-915S2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

Commit message: Working on boards
Parts:
- removed D3: SMAJ5.0, Custom:SMAJ5.0_DIOM4325X250N
- removed D4: Green, LED_SMD:LED_0805_2012Metric_Pad1.15x1.40mm_HandSolder
- removed D5: BLUE, LED_SMD:LED_0805_2012Metric_Pad1.15x1.40mm_HandSolder
- removed D6: Red, LED_SMD:LED_0805_2012Metric_Pad1.15x1.40mm_HandSolder
- removed the G*** at (110.7, 87.2)
- removed R11, R12, R13: 100K, Resistor_SMD:R_0402_1005Metric
- removed REF** (x3): MountingHole_2.1mm, MountingHole:MountingHole_2.1mm
- removed SW4: AS11CH, Custom:AS11CH
- removed TH1: 10K, Capacitor_SMD:C_0603_1608Metric
- added C12: .1uF, Capacitor_SMD:C_0603_1608Metric, F.Cu at (91.1, 73.1)
- added G***: LOGO, Logos:DroidKillSwitchLogo, F.Cu at (108.7, 83.3)
- added J4: Conn_01x02, Connector_Molex:Molex_KK-254_AE-6410-02A_1x02_P2.54mm_Vertical, F.Cu at (77.8, 59.9)
- added J5: Screw_Terminal_01x02, TerminalBlock:TerminalBlock_bornier-2_P5.08mm, F.Cu at (94.6, 60.5)
- added Q3: BSS138, Package_TO_SOT_SMD:SOT-23, F.Cu at (93.0, 66.7)
- added U7: D24V550F5_Step_Down_Regulator, Pololu:VoltageREG_2851, F.Cu at (68.5, 74.2)
- C9: value 4.7uF -> .1uF
- J2: value S2B-PH-K-S(LF)(SN) -> Screw_Terminal_01x02; footprint Custom:JST_S2B-PH-K-S(LF)(SN) -> TerminalBlock:TerminalBlock_bornier-2_P5.08mm
- L1, L2, L3: footprint LED_SMD:LED_WS2812B_PLCC4_5.0x5.0mm_P3.2mm -> Custom:WS2812B-2020; moved to F.Cu
- R10: value 10K -> 400
- R7, R8: value 82 -> 10K
- R9: value 150 -> 400
- S2, S3: value TL3342F160QG -> TL3305CF260QG; footprint Custom:KillSwiitch -> Custom:TL3305CF260QG; moved to F.Cu
- U4: value MCP73871-2CC-Custom -> TPS2115APW; footprint Package_DFN_QFN:QFN-20-1EP_4x4mm_P0.5mm_EP2.7x2.7mm_ThermalVias -> Package_SO:TSSOP-8_4.4x3mm_P0.65mm
- U6: value LS18-S(Debouce) -> LS18-S
- moved L3 86.8 mm to (63.4, 58.7)
- moved R16 84.3 mm to (36.5, 85.7), turned to 0 degrees
- moved R17 80.5 mm to (63.3, 62.0), turned to 0 degrees
- moved L2 79.6 mm to (36.5, 83.2), turned to 90 degrees
- moved S3 78.9 mm to (55.6, 58.8), turned to 0 degrees
- moved U1 77.4 mm to (43.1, 60.3), turned to 90 degrees
- moved S1 69.5 mm to (36.2, 75.1), turned to 90 degrees
- moved C1 68.6 mm to (38.9, 69.1), turned to 180 degrees
- moved C2 66.8 mm to (42.5, 68.5), turned to 0 degrees
- moved C3 58.6 mm to (46.1, 74.1)
- moved Q2 58.0 mm to (49.4, 75.8), turned to -90 degrees
- moved R1 56.5 mm to (46.7, 76.7), turned to 90 degrees
- moved R3 55.3 mm to (51.1, 63.0), turned to 180 degrees
- moved R2 52.6 mm to (51.1, 64.7), turned to 180 degrees
- moved S2 51.2 mm to (70.4, 58.8), turned to 0 degrees
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Connections:
- net BATSTAT_LED_DATA renamed RELAY_LED_DATA
- C8 pad 1: VBUS -> GND
- C8 pad 2: GND -> Net-(C6-Pad2)
- C9 pad 1: Net-(C9-Pad1) -> +5V
- J2 pad 1: Net-(J2-Pad1) -> GND
- J2 pad 2: GND -> VIN
- R10 pad 1: Net-(R10-Pad1) -> Net-(C6-Pad2)
- R7 pad 1: Net-(R7-Pad1) -> +3V3
- R7 pad 2: Net-(D4-Pad1) -> RELAY_CONTROL
- R8 pad 1: Net-(R8-Pad1) -> +5V
- R9 pad 2: Net-(R9-Pad2) -> GND
- U1 pad 24: unconnected-(U1-Pad24) -> EXT_SW_OUT
- U2 pad 28: DTS -> DTR
- U4 pad 1: Net-(C6-Pad2) -> unconnected-(U4-Pad1)
- U4 pad 2: VBUS -> GND
- U4 pad 3: GND -> +5V
- U4 pad 4: GND -> Net-(R9-Pad1)
- U4 pad 5: Net-(TH1-Pad1) -> GND
- U4 pad 6: Net-(R7-Pad1) -> VBUS
- U4 pad 7: Net-(R8-Pad1) -> Net-(C6-Pad2)
- U4 pad 8: Net-(R9-Pad1) -> +5V
- U6 pad 3: unconnected-(U6-Pad3) -> EXT_Switch
- U6 pad 6: unconnected-(U6-Pad6) -> EXT_SW_OUT
Routing:
- net EXT_SW_OUT: track 0.00 -> 47.5 mm, vias 0 -> 2
- net Net-(C9-Pad1): track 46.7 -> 0.00 mm, vias 1 -> 0
- net Net-(R7-Pad1): track 38.1 -> 0.00 mm, vias 2 -> 0
- net STATUS_LED_DATA: track 1.97 -> 39.4 mm, vias 0 -> 2
- net OFF_SW_OUT: track 19.7 -> 56.7 mm
- net LORA_LED_DATA: track 21.0 -> 56.9 mm
- net Net-(R8-Pad1): track 35.5 -> 0.00 mm, vias 2 -> 0
- net Net-(R9-Pad1): track 36.6 -> 2.25 mm, vias 2 -> 0
- net USB_DN: track 18.1 -> 51.9 mm, vias 0 -> 2
- net SCK_LORA: track 41.6 -> 75.0 mm
- net RESET_LORA: track 45.2 -> 78.5 mm
- net ON_SW_OUT: track 16.1 -> 49.3 mm
- net MOSI_LORA: track 40.7 -> 72.6 mm
- net +5V: track 0.00 -> 30.3 mm
- net NSS_LORA: track 46.0 -> 75.9 mm
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Other:
- board size 65 x 27 mm -> 88 x 36 mm
- board text added: "+"
- board text added: "-"
- board text added: "6V-36V In"
- board text added: "External Switch"
- board text added: "LoRa Antenna"
- board text added: "Relay OFF"
- board text added: "Relay ON"
- board text added: "Relay Status"
- board text added: "Reset"
- board text added: "To Relay"

Commit message: A lot of updates.  Too much to describe
Parts:
- removed the G*** at (89.2, 125.5)
- removed the G*** at (119.6, 125.5)
- added C13: .1uF, Capacitor_SMD:C_0603_1608Metric, F.Cu at (84.6, 59.7)
- added U8: MAX6816, Package_TO_SOT_SMD:SOT-143, F.Cu at (84.4, 63.3)
- J2: value Screw_Terminal_01x02 -> Power In
- J4: value Conn_01x02 -> External Switch In
- J5: value Screw_Terminal_01x02 -> Output
- U6: value LS18-S -> MAX6817EUT+T; footprint Custom:SOIC127P600X175-8N -> Custom:SOT95P280X145-6N
- moved G*** 6.60 mm to (102.1, 83.3)
- moved G*** 6.04 mm to (97.3, 77.7)
- moved C11 4.10 mm to (79.9, 64.5)
- moved U6 3.52 mm to (80.5, 66.9)
- moved S1 1.78 mm to (36.2, 76.9)
Connections:
- C11 pad 1: +3V3 -> GND
- C11 pad 2: GND -> +3V3
- J4 pad 1: EXT_Switch -> Net-(J4-Pad1)
- U6 pad 1: +3V3 -> Net-(S2-Pad1)
- U6 pad 2: Net-(S2-Pad1) -> GND
- U6 pad 3: EXT_Switch -> Net-(S3-Pad1)
- U6 pad 4: Net-(S3-Pad1) -> OFF_SW_OUT
- U6 pad 5: OFF_SW_OUT -> +3V3
- U6 pad 6: EXT_SW_OUT -> ON_SW_OUT
Routing:
- net +3V3: track 37.7 -> 51.3 mm
- net EXT_Switch: track 10.6 -> 0.00 mm
- net GND: track 166.2 -> 175.2 mm, vias 20 -> 21
- net Net-(S2-Pad1): track 27.3 -> 18.3 mm
- net Net-(J4-Pad1): track 0.00 -> 8.00 mm
- net EXT_SW_OUT: track 47.5 -> 49.7 mm
- net ON_SW_OUT: track 49.3 -> 51.2 mm
- net OFF_SW_OUT: track 56.7 -> 58.2 mm
- net Net-(S3-Pad1): track 38.0 -> 37.4 mm
Other:
- board text removed: "Battery Status"
- board text removed: "Board Status"
- board text removed: "Charging (Blue)"
- board text removed: "Low Batt (Red)"
- board text removed: "OFF"
- board text removed: "ON"
- board text removed: "USB Power (Green)"
