File: In Progress/Kill_Switch_Droid/Kill_Switch_Droid.kicad_sch (KiCad schematic)
At the start: 34 parts, among them J1 USB_B_Micro, J3 U.FL-R-SMT-1(10), Q2 UMH3N, U1 ESP32-PICO-MINI-02, U2 CP2102N-A02-GQFN28, U3 LP5912-3.3DRV, U5 RFM95W-915S2, U6 LS18-S(Debouce)

Commit message: Working on boards
Parts:
- added C12, C9: .1uF, Capacitor_SMD:C_0603_1608Metric, symbol Device:C_Small
- added C8: 10uF, Capacitor_SMD:C_0805_2012Metric, symbol Device:C_Small
- added J2, J5: Screw_Terminal_01x02, TerminalBlock:TerminalBlock_bornier-2_P5.08mm, symbol Connector:Screw_Terminal_01x02
- added J4: Conn_01x02, Connector_Molex:Molex_KK-254_AE-6410-02A_1x02_P2.54mm_Vertical, symbol Connector_Generic:Conn_01x02
- added Q3: BSS138, Package_TO_SOT_SMD:SOT-23, symbol Transistor_FET:BSS138
- added R10, R9: 400, Resistor_SMD:R_0402_1005Metric, symbol Device:R_Small
- added R7, R8: 10K, Resistor_SMD:R_0402_1005Metric, symbol Device:R_Small
- added U4: TPS2115APW, Package_SO:TSSOP-8_4.4x3mm_P0.65mm, symbol Custom:TPS2115APW
- added U7: D24V550F5_Step_Down_Regulator, Pololu:VoltageREG_2851, symbol Pololu:D24V550F5_Step_Down_Regulator
- L1, L2, L3: footprint LED_SMD:LED_WS2812B_PLCC4_5.0x5.0mm_P3.2mm -> Custom:WS2812B-2020
- S2, S3: value TL3342F160QG -> TL3305CF260QG; footprint Custom:KillSwiitch -> Custom:TL3305CF260QG; Digikey Part Number EG2531CT-ND -> EG5355CT-ND; LCSC ------ -> C2886904; Manufacturers Part Number TL3342F160QG/TR -> TL3305CF260QG; Mouser Part Number ------ -> 612-TL3305CF260QG
- U6: value LS18-S(Debouce) -> LS18-S
Connections:
- net DTS is gone; now on net DTR: U2.28 (DTR)
- net +3V3: now also Q3.1 (G), R7.1
- net GND: now also C12.2, C8.1, C9.2, J2.1 (Pin_1), J4.2 (Pin_2), J5.1 (Pin_1), R10.2, R9.2, U4.2 (D0), U4.5 (GND), U7.2 (GND), U7.4 (GND)
- net VBUS: now also C12.1, U4.6 (IN2)
- net at C6.2, U3.4 (EN), U3.6 (IN): now also C8.2, R10.1, U4.7 (OUT)
- net EXT_Switch: now reaches U6.3 (SW1)
- net EXT_Switch: now also J4.1 (Pin_1)
- net EXT_SW_OUT: now reaches U6.6 (OUT1)
- net EXT_SW_OUT: now also U1.24 (IO4)
- net BATSTAT_LED_DATA renamed RELAY_LED_DATA
- new net: R9.1, U4.4 (ILIM)
- new net: J5.2 (Pin_2), Q3.3 (D), R8.2
- new net +5V: C9.1, R8.1, U4.3 (D1), U4.8 (IN1), U7.5 (VOut)
- new net RELAY_CONTROL: Q3.2 (S), R7.2
- new net VIN: J2.2 (Pin_2), U7.1 (VIN)
- no-connect marks 41 -> 40
Other:
- note added: "Power Source Selection IC"
- note added: "Relay Control Output"
- moved on the sheet: C10, C6, C7, J3, L1, L2, L3, R14, R16, R17, S3, U3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

Commit message: A lot of updates.  Too much to describe
Parts:
- removed U6: LS18-S, Custom:SOIC127P600X175-8N, symbol Custom:LS18-S(Debouce)
- added C13: .1uF, Capacitor_SMD:C_0603_1608Metric, symbol Device:C_Small
- added U6: MAX6817EUT+T, SOT95P280X145-6N, symbol Custom:MAX6817EUT+T
- added U8: MAX6816, Package_TO_SOT_SMD:SOT-143, symbol Interface:MAX6816
- J2: value Screw_Terminal_01x02 -> Power In
- J4: value Conn_01x02 -> External Switch In
- J5: value Screw_Terminal_01x02 -> Output
Connections:
- net +3V3: now also C11.2, C13.2, U6.5 (VCC), U8.4 (VCC); no longer C11.1
- net EXT_SW_OUT: now also U8.3 (OUT)
- net GND: now also C11.1, C13.1, U6.2 (GND), U8.1 (GND); no longer C11.2
- net OFF_SW_OUT: now also U6.4 (OUT2)
- net ON_SW_OUT: now also U6.6 (OUT1)
- net at S3.1, S3.2: now also U6.3 (IN2)
- net at S2.1, S2.2: now also U6.1 (IN1)
- net EXT_Switch: no longer names the net of J4.1 (Pin_1)
- net EXT_Switch: now also U8.2 (IN)
Other:
- note added: "Debouce IC (1 Channel)"
- note added: "Debouce IC (2 Channel)"
- note added: "Used with TPS2115APW"
- note removed: "Update: Blue Discrete LED - PN's Green Discrete LED - PN's SW2 and SW3 - PN's L1,L2,L3 - PN's"
- moved on the sheet: C11, C12, J2, J4, J5, L1, L2, Q3, R14, R16, R7, R8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
