File: Body_Servos/Body_Servos.kicad_sch (KiCad schematic)
At the start: 30 parts, among them J1 USB_B_Micro, J12 SERIAL_FU, J2 AUX3, J3 AUX1, J4 AUX2, J5 12OUT, J6 12VOUT, J7 5V OUT, J8 5V Out 2, SW1 SW_Push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

Commit message: Updated the servo controller to adjust for the 4 pin molex header's alignment pin
Parts:
- J2, J3, J4: footprint Connector_Molex:Molex_KK-254_AE-6410-04A_1x04_P2.54mm_Vertical -> Custom:470531000
Changed lines of the file:
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@@
       (effects (font (size 1.27 1.27)) (justify left))
     )
-    (property "Footprint" "Connector_Molex:Molex_KK-254_AE-6410-04A_1x04_P2.54mm_Vertical" (id 2) (at 267.97 41.91 0)
+    (property "Footprint" "Custom:470531000" (id 2) (at 267.97 41.91 0)
       (effects (font (size 1.27 1.27)) hide)
     )
@@
       (effects (font (size 1.27 1.27)) (justify left))
     )
-    (property "Footprint" "Connector_Molex:Molex_KK-254_AE-6410-04A_1x04_P2.54mm_Vertical" (id 2) (at 237.49 41.91 0)
+    (property "Footprint" "Custom:470531000" (id 2) (at 237.49 41.91 0)
       (effects (font (size 1.27 1.27)) hide)
     )
@@
       (effects (font (size 1.27 1.27)) (justify left))
     )
-    (property "Footprint" "Connector_Molex:Molex_KK-254_AE-6410-04A_1x04_P2.54mm_Vertical" (id 2) (at 237.49 26.67 0)
+    (property "Footprint" "Custom:470531000" (id 2) (at 237.49 26.67 0)
       (effects (font (size 1.27 1.27)) hide)
     )
@@
     )
     (path "/a9448de9-7beb-45d2-bf6e-71f8cedebf98"
-      (reference "J2") (unit 1) (value "AUX3") (footprint "Connector_Molex:Molex_KK-254_AE-6410-04A_1x04_P2.54mm_Vertical")
+      (reference "J2") (unit 1) (value "AUX3") (footprint "Custom:470531000")
     )
     (path "/9cdb5bde-d012-4dfd-bd3c-8364dcaa5312"
-      (reference "J3") (unit 1) (value "AUX1") (footprint "Connector_Molex:Molex_KK-254_AE-6410-04A_1x04_P2.54mm_Vertical")
+      (reference "J3") (unit 1) (value "AUX1") (footprint "Custom:470531000")
     )
     (path "/4d78864d-566d-466b-be26-3a572d3eb5eb"
-      (reference "J4") (unit 1) (value "AUX2") (footprint "Connector_Molex:Molex_KK-254_AE-6410-04A_1x04_P2.54mm_Vertical")
+      (reference "J4") (unit 1) (value "AUX2") (footprint "Custom:470531000")
     )
     (path "/1a1346f9-ba9f-4c77-90ee-18d527b20ae9"
