File: Body_LED_Controller_V1.1/Body_LED_Controller_V1.kicad_pcb (KiCad board)
At the start: 4 copper layers, 123 x 78 mm, 104 parts, among them J1 Ext Mic, J10 2560 USB, J11 ESP USB, J12 UnSW_BATT_IN, J13 Sound Board, J14 Dome Controller USB, J15 Dome Plate Controller USB, J16 UnSW_BATT_PASS, J17 RADH_POW, J18 RASP_POW, J19 5V_OUT_3, J20 ICSP, J21 Dome Electronics Power In, J22 DB25_Male_MountingHoles, J23 Amplifier_POW, J24 AUX1, J25 Stealth, J26 RADH, J27 Vu Data Panel, J3 Conn_02x10_Odd_Even, J37 AUX2, J4 LDP, J5 Coin Slots, J6 CBI Batt LEDS, J7 Data Panel/ CBI, J8 Spectrum Analyzer, J9 Maintenance, SW1 2560 Reset, SW2 SW_Push, U1 ATMEGA256016AU, U14 D36V50F5-STEPDOWN, U2 CH340C, U3 TPS2115APW, U4 ESP32-WROOM-32D_16MB_, U5 CH340C, U6 UMH3N, U7 LP5912-3.3DRV, Y1 16MHz

Commit message: some minor updates
Changed lines of the file:
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@@
       (effects (font (size 0.25 0.25) (thickness 0.15)))
     )
+    (fp_line (start 12.7 12.7) (end -12.7 12.7) (layer "F.SilkS") (width 0.12))
+    (fp_line (start 12.7 -12.7) (end -12.7 -12.7) (layer "F.SilkS") (width 0.12))
+    (fp_line (start 12.7 -12.7) (end 12.7 12.7) (layer "F.SilkS") (width 0.12))
     (fp_line (start -12.7 12.7) (end -12.7 -12.7) (layer "F.SilkS") (width 0.12))
-    (fp_line (start 12.7 -12.7) (end 12.7 12.7) (layer "F.SilkS") (width 0.12))
-    (fp_line (start 12.7 -12.7) (end -12.7 -12.7) (layer "F.SilkS") (width 0.12))
-    (fp_line (start 12.7 12.7) (end -12.7 12.7) (layer "F.SilkS") (width 0.12))
-    (pad "1" thru_hole circle (at -6.35 11.43) (size 1.524 1.524) (drill 0.762) (layers *.Cu *.Mask)
+    (pad "1" thru_hole circle (at -6.35 11.43) (size 1.7 1.7) (drill 1) (layers *.Cu *.Mask)
       (net 3 "+5V") (pinfunction "VOUT") (pintype "bidirectional"))
-    (pad "2" thru_hole circle (at -3.81 11.43) (size 1.524 1.524) (drill 0.762) (layers *.Cu *.Mask)
+    (pad "2" thru_hole circle (at -3.81 11.43) (size 1.7 1.7) (drill 1) (layers *.Cu *.Mask)
       (net 2 "GND") (pinfunction "GND") (pintype "bidirectional"))
-    (pad "3" thru_hole circle (at -1.27 11.43) (size 1.524 1.524) (drill 0.762) (layers *.Cu *.Mask)
+    (pad "3" thru_hole circle (at -1.27 11.43) (size 1.7 1.7) (drill 1) (layers *.Cu *.Mask)
       (net 2 "GND") (pinfunction "GND") (pintype "bidirectional"))
-    (pad "4" thru_hole circle (at 1.27 11.43) (size 1.524 1.524) (drill 0.762) (layers *.Cu *.Mask)
+    (pad "4" thru_hole circle (at 1.27 11.43) (size 1.7 1.7) (drill 1) (layers *.Cu *.Mask)
       (net 1 "+12V") (pinfunction "VIN") (pintype "bidirectional"))
-    (pad "5" thru_hole circle (at 3.81 11.43) (size 1.524 1.524) (drill 0.762) (layers *.Cu *.Mask)
+    (pad "5" thru_hole circle (at 3.81 11.43) (size 1.7 1.7) (drill 1) (layers *.Cu *.Mask)
       (net 159 "unconnected-(U14-Pad5)") (pinfunction "VRP") (pintype "bidirectional+no_connect"))
-    (pad "6" thru_hole circle (at 6.35 11.43) (size 1.524 1.524) (drill 0.762) (layers *.Cu *.Mask)
+    (pad "6" thru_hole circle (at 6.35 11.43) (size 1.7 1.7) (drill 1) (layers *.Cu *.Mask)
       (net 160 "unconnected-(U14-Pad6)") (pinfunction "EN") (pintype "bidirectional+no_connect"))
-    (pad "7" thru_hole circle (at 6.35 8.89) (size 1.524 1.524) (drill 0.762) (layers *.Cu *.Mask)
+    (pad "7" thru_hole circle (at 6.35 8.89) (size 1.7 1.7) (drill 1) (layers *.Cu *.Mask)
       (net 161 "unconnected-(U14-Pad7)") (pinfunction "PG") (pintype "bidirectional+no_connect"))
-    (pad "8" thru_hole circle (at 3.81 8.89) (size 1.524 1.524) (drill 0.762) (layers *.Cu *.Mask)
+    (pad "8" thru_hole circle (at 3.81 8.89) (size 1.7 1.7) (drill 1) (layers *.Cu *.Mask)
       (net 162 "unconnected-(U14-Pad8)") (pinfunction "VRP") (pintype "bidirectional+no_connect"))
-    (pad "9" thru_hole circle (at 1.27 8.89) (size 1.524 1.524) (drill 0.762) (layers *.Cu *.Mask)
+    (pad "9" thru_hole circle (at 1.27 8.89) (size 1.7 1.7) (drill 1) (layers *.Cu *.Mask)
       (net 1 "+12V") (pinfunction "VIN") (pintype "bidirectional"))
-    (pad "10" thru_hole circle (at -1.27 8.89) (size 1.524 1.524) (drill 0.762) (layers *.Cu *.Mask)
+    (pad "10" thru_hole circle (at -1.27 8.89) (size 1.7 1.7) (drill 1) (layers *.Cu *.Mask)
       (net 2 "GND") (pinfunction "GND") (pintype "bidirectional"))
-    (pad "11" thru_hole circle (at -3.81 8.89) (size 1.524 1.524) (drill 0.762) (layers *.Cu *.Mask)
+    (pad "11" thru_hole circle (at -3.81 8.89) (size 1.7 1.7) (drill 1) (layers *.Cu *.Mask)
       (net 2 "GND") (pinfunction "GND") (pintype "bidirectional"))
-    (pad "12" thru_hole circle (at -6.35 8.89) (size 1.524 1.524) (drill 0.762) (layers *.Cu *.Mask)
+    (pad "12" thru_hole circle (at -6.35 8.89) (size 1.7 1.7) (drill 1) (layers *.Cu *.Mask)
       (net 3 "+5V") (pinfunction "VOUT") (pintype "bidirectional"))
     (pad "13" thru_hole circle (at -10.6 10.5) (size 2.3 2.3) (drill 2.2) (layers *.Cu *.Mask))
