File: Body_Controller_V1.2/Body_Controller_V1.kicad_pcb (KiCad board)
At the start: 4 copper layers, 123 x 78 mm, 104 parts, among them J1 Ext Mic, J10 2560 USB, J11 ESP USB, J12 UnSW_BATT_IN, J13 Sound Board, J14 Dome Controller USB, J15 Dome Plate Controller USB, J16 UnSW_BATT_PASS, J17 RADH_POW, J18 RASP_POW, J19 5V_OUT_3, J20 ICSP, J21 Dome Electronics Power In, J22 DB25_Male_MountingHoles, J23 Amplifier_POW, J24 AUX1, J25 Stealth, J26 RADH, J27 Vu Data Panel, J3 Conn_02x10_Odd_Even, J37 AUX2, J4 LDP, J5 Coin Slots, J6 CBI Batt LEDS, J7 Data Panel/ CBI, J8 Spectrum Analyzer, J9 Maintenance, SW1 2560 Reset, SW2 SW_Push, U1 ATMEGA256016AU, U14 D36V50F5-STEPDOWN, U2 CH340C, U3 TPS2115APW, U4 ESP32-WROOM-32D_16MB_, U5 CH340C, U6 UMH3N, U7 LP5912-3.3DRV, Y1 16MHz

Commit message: Lots of changes
Parts:
- removed the G*** at (151.1, 90.4)
- added G***: LOGO, Logos:R2DroidGatewayV1.2, F.Cu at (151.9, 89.7)
- J10: value 2560 USB -> MICROXNJ; footprint Connector_USB:USB_Micro-B_Amphenol_10118194_Horizontal -> Custom:SHOUHAN_MICROXNJ
- J11: value ESP USB -> MICROXNJ; footprint Connector_USB:USB_Micro-B_Amphenol_10118194_Horizontal -> Custom:SHOUHAN_MICROXNJ
- J14: value Dome Controller USB -> MICROXNJ; footprint Connector_USB:USB_Micro-B_Amphenol_10118194_Horizontal -> Custom:SHOUHAN_MICROXNJ
- J15: value Dome Plate Controller USB -> MICROXNJ; footprint Connector_USB:USB_Micro-B_Amphenol_10118194_Horizontal -> Custom:SHOUHAN_MICROXNJ
- R18: renamed from R2; value 57K -> 60K
- SW1, SW2: footprint Custom:GT-TC057A-H050-L1 -> Custom:TS-1101-C-W
- moved J11 2.78 mm to (110.0, 119.9), turned to 180 degrees
- moved J10 2.75 mm to (121.0, 119.9), turned to 180 degrees
- moved J15 2.65 mm to (88.1, 119.9), turned to 180 degrees
- moved J14 2.62 mm to (99.3, 119.9), turned to 180 degrees
- moved C5 0.51 mm to (105.3, 85.8)
- turned SW1 to 180 degrees
- turned SW2 to 180 degrees
- renumbered R1 to R19
Routing:
- net unconnected-(J10-PadS1): track 0.00 -> 14.3 mm
- net unconnected-(J14-Pad6): track 13.9 -> 0.00 mm
- net unconnected-(J14-PadS1): track 0.00 -> 13.9 mm
- net unconnected-(J11-PadS1): track 0.00 -> 13.6 mm
- net unconnected-(J15-PadS1): track 0.00 -> 13.6 mm
- net unconnected-(J15-Pad6): track 13.4 -> 0.00 mm
- net unconnected-(J10-Pad6): track 13.3 -> 0.00 mm
- net unconnected-(J11-Pad6): track 12.8 -> 0.00 mm
- net D+_ESP: track 22.4 -> 24.6 mm
- net +5V_IC: track 54.6 -> 56.2 mm
- net D-_ESP: track 20.2 -> 21.5 mm
- net GND_DP: track 78.8 -> 79.9 mm
- net RESET_ESP: track 74.0 -> 74.8 mm
Other:
- board text added: "R1"
- board text added: "R2"
