File: Body_Controller_V1.2/Body_Controller_V1.kicad_sch (KiCad schematic)
At the start: 95 parts, among them J1 Ext Mic, J10 2560 USB, J11 ESP USB, J12 UnSW_BATT_IN, J13 Sound Board, J14 Dome Controller USB, J15 Dome Plate Controller USB, J16 UnSW_BATT_PASS, J17 RADH_POW, J18 RASP_POW, J19 5V_OUT_3, J20 ICSP, J21 Dome Electronics Power In, J22 DB25_Male_MountingHoles, J23 Amplifier_POW, J24 AUX1, J25 Stealth, J26 RADH, J27 Vu Data Panel, J3 Conn_02x10_Odd_Even, J37 AUX2, J4 LDP, J5 Coin Slots, J6 CBI Batt LEDS, J7 Data Panel/ CBI, J8 Spectrum Analyzer, J9 Maintenance, SW1 2560 Reset, SW2 SW_Push, U1 ATMEGA256016AU, U14 D36V50F5-STEPDOWN, U2 CH340C, U3 TPS2115APW, U4 ESP32-WROOM-32D_16MB_, U5 CH340C, U6 UMH3N, U7 LP5912-3.3DRV, Y1 16MHz

Commit message: Lots of changes
Parts:
- removed J10: 2560 USB, Connector_USB:USB_Micro-B_Amphenol_10118194_Horizontal, symbol Connector:USB_B_Micro
- removed J11: ESP USB, Connector_USB:USB_Micro-B_Amphenol_10118194_Horizontal, symbol Connector:USB_B_Micro
- removed J14: Dome Controller USB, Connector_USB:USB_Micro-B_Amphenol_10118194_Horizontal, symbol Connector:USB_B_Micro
- removed J15: Dome Plate Controller USB, Connector_USB:USB_Micro-B_Amphenol_10118194_Horizontal, symbol Connector:USB_B_Micro
- added J10, J11, J14, J15: MICROXNJ, Custom:SHOUHAN_MICROXNJ, symbol Custom:MICROXNJ
- D2, D3, D4: footprint SOD3716X135N -> Custom:SOD3716X135N
- L2, L3: footprint WS2812B-2020 -> Custom:WS2812B-2020
- R18: value 57K -> 60K; Digikey Part Number 311-57.6KHRCT-ND -> (none); LCSC C245983 -> (none); Manufacturer's Part Number RC0603FR-0757K6L -> (none); Mouser Part Number 603-RC0603FR-0757K6L -> (none)
- R19: Digikey Part Number RMCF0603FG22K0CT-ND -> (none); LCSC C325646 -> (none); Manufacturer Stackpole Electronics Inc -> (none); Manufacturer's Part Number RMCF0603FG22K0 -> (none); Mouser Part Number 708-RMCF0603FG22K0 -> (none)
- SW1, SW2: footprint Custom:GT-TC057A-H050-L1 -> Custom:TS-1101-C-W; Digikey Part Number EG2529CT-ND -> (none); LCSC C2886915 -> C318938; Manufacturer E-Switch -> XKB Connectivity; Manufacturer's Part Number TL3302BF180QG/TR -> TS-1101-C-W
Connections:
- net D+_2560: now also J10.3 (D+)
- net D+_DC: now also J14.3 (D+)
- net D+_DP: now also J15.3 (D+)
- net D+_ESP: now also J11.3 (D+)
- net D-_2560: now also J10.2 (D-)
- net D-_DC: now also J14.2 (D-)
- net D-_DP: now also J15.2 (D-)
- net D-_ESP: now also J11.2 (D-)
- net GND: now also J10.5 (GND), J11.5 (GND)
- net GND_DC: now also J14.5 (GND)
- net GND_DP: now also J15.5 (GND)
- net VBUS_DC: now also J14.1 (VBUS)
- net VBUS_DP: now also J15.1 (VBUS)
- net at F1.1: now also J10.1 (VBUS)
- net at D2.A: now also J11.1 (VBUS)
- new net: J10.S1 (SHIELD), J10.S2 (SHIELD), J10.S3 (SHIELD), J10.S4 (SHIELD), J10.S5 (SHIELD), J10.S6 (SHIELD)
- new net: J14.S1 (SHIELD), J14.S2 (SHIELD), J14.S3 (SHIELD), J14.S4 (SHIELD), J14.S5 (SHIELD), J14.S6 (SHIELD)
- new net: J15.S1 (SHIELD), J15.S2 (SHIELD), J15.S3 (SHIELD), J15.S4 (SHIELD), J15.S5 (SHIELD), J15.S6 (SHIELD)
- new net: J11.S1 (SHIELD), J11.S2 (SHIELD), J11.S3 (SHIELD), J11.S4 (SHIELD), J11.S5 (SHIELD), J11.S6 (SHIELD)
Other:
- note added: "G"
- note removed: "C"
- moved on the sheet: C3, C4, D2, SW2
