File: Pancake_Servo_Slip_Ring/R2_Art/R2_Art.kicad_pcb (KiCad board)
At the start: 2 copper layers, 60.7 x 82.3 mm, 2 parts

Commit message: Updated C3P0 Controller
Parts:
- removed the G*** at (153.4, 64.0)
- removed the G*** at (221.0, 62.7)
- added G***: LOGO, 02-Logos:R2BW147-3, F.Cu at (86.9, 95.0)
- added G***: LOGO, 02-Logos:qrcode3, B.Cu at (90.9, 99.1)
- added G***: LOGO, 02-Logos:R2logo30mm, B.Cu at (87.9, 62.0)
- added REF**: dome, 01-Custom:dome, F.Cu at (87.1, 54.9)
Other:
- board size 60.7 x 82.3 mm -> 70 x 100.5 mm
- board text added: "R2D2 Builder: Greg Hulette"
