File: Wireless3.0/Wireless3.0.kicad_pcb (KiCad board)
At the start: 2 copper layers, 57.5 x 71.5 mm, 14 parts, among them J1 Serial 1, J2 Serial 2, J3 Serial 3, J4 Serial 4, J5 Serial 5, J6 Power, U1 ESP32-S3-DEVKITC-1-N8R2

Commit message: added files.
Connections:
- U1 pad J1_1: GND -> Net-(U1-3V3-PadJ1_1)
- U1 pad J1_2: GND -> Net-(U1-3V3-PadJ1_1)
Routing:
- net Net-(U1-3V3-PadJ1_1): track 0.00 -> 2.54 mm
Other:
- board text added: "wireless communication board (wcb) ver: 3.1 date: 8/jul/2025 created by: greg hulette"
- board text removed: "wireless communication board (wcb) ver: 3.0 date: 2/jul/2025 created by: greg hulette"
