File: Sabe-FullSized/Sabe-FullSized.kicad_sch (KiCad schematic)
At the start: 23 parts, among them J1 Roboteq, J2 Conn_01x04, J3 Conn_01x04, J4 Conn_01x04, J5 5V, J6 6-36V, U2 D24V550F5_Step_Down_Regulator, U3 MCP1700x-330xxTO, U5 ESP32-S3-DEVKITC-1-N8R2

Commit message: sabe
Parts:
- removed D2, D3: D_Schottky, Diode_THT:D_DO-201AD_P12.70mm_Horizontal, symbol Device:D_Schottky
- removed U3: MCP1700x-330xxTO, Package_TO_SOT_THT:TO-92_Inline, symbol Regulator_Linear:MCP1700x-330xxTO
- added J10: Misc 4, Connector_PinHeader_2.54mm:PinHeader_1x04_P2.54mm_Vertical, symbol Connector_Generic:Conn_01x04
- added J7: Misc 1, Connector_PinHeader_2.54mm:PinHeader_1x04_P2.54mm_Vertical, symbol Connector_Generic:Conn_01x04
- added J8: Misc 2, Connector_PinHeader_2.54mm:PinHeader_1x04_P2.54mm_Vertical, symbol Connector_Generic:Conn_01x04
- added J9: Misc 3, Connector_PinHeader_2.54mm:PinHeader_1x04_P2.54mm_Vertical, symbol Connector_Generic:Conn_01x04
- added R2, R3: 100, Resistor_THT:R_Axial_DIN0207_L6.3mm_D2.5mm_P10.16mm_Horizontal, symbol Device:R_Small
- added U1: LM2937xT, Package_TO_SOT_THT:TO-220-3_Vertical, symbol Regulator_Linear:LM2937xT
- added U3, U6: LM66100DCK, Package_TO_SOT_SMD:SOT-363_SC-70-6, symbol Power_Management:LM66100DCK
- C2: value 1uf -> 10uf; footprint Capacitor_THT:C_Disc_D7.5mm_W4.4mm_P5.00mm -> Capacitor_THT:CP_Radial_D5.0mm_P2.00mm; symbol Device:C -> Device:C_Polarized_US
- C4, C6: symbol Device:C_Polarized_US -> Device:C
- J2: value Conn_01x04 -> Serial 1
- J3: value Conn_01x04 -> Serial 2
- J4: value Conn_01x04 -> Serial 3
Connections:
- net 3.3V: now also C3.1, C4.1, R1.2, U4.1 (VCC), U1.3 (VO)
- net 5V: now also J1.2 (Pin_2), J2.2 (Pin_2), J3.2 (Pin_2), J4.2 (Pin_2), J10.2 (Pin_2), J7.2 (Pin_2), J8.2 (Pin_2), J9.2 (Pin_2), R2.1, R3.1, U1.1 (VI), U3.6 (VOUT), U6.6 (VOUT); no longer C1.2, C2.2, C6.2, C7.2, J5.1 (Pin_1), J6.1 (Pin_1), U2.2 (GND), U2.3 (GND)
- net at J6.2 (Pin_2), U2.1 (VIN): now also U2.0 (En)
- net xbee_din: now reaches U5.J1_10 (GPIO17)
- net xbee_din: now also U4.3 (DIN)
- net xbee_dout: now reaches U5.J1_11 (GPIO18)
- net xbee_dout: now also U4.2 (DOUT)
- net S2_RX: now reaches U5.J1_12 (GPIO8)
- net S2_RX: now also J3.4 (Pin_4)
- net xbee_rst: now reaches U5.J1_15 (GPIO9)
- net xbee_rst: now also R1.1, U4.5 (~{RESET})
- net Misc1_G10: now reaches U5.J1_16 (GPIO10)
- net Misc1_G10: now also J10.3 (Pin_3)
- net Misc1_G11: now reaches U5.J1_17 (GPIO11)
- net Misc1_G11: now also J10.4 (Pin_4)
- net S3_TX: now reaches U5.J1_19 (GPIO13)
- net S3_TX: now also J4.3 (Pin_3)
- net S3_RX: now reaches U5.J1_20 (GPIO14)
- net S3_RX: now also J4.4 (Pin_4)
- net GND: now reaches U5.J1_22 (GND), U5.J3_1 (GND), U5.J3_21 (GND), U5.J3_22 (GND)
- net GND: now also C1.2, C2.2, C3.2, C4.2, C6.2, C7.2, J1.1 (Pin_1), J2.1 (Pin_1), J3.1 (Pin_1), J4.1 (Pin_1), J5.1 (Pin_1), J6.1 (Pin_1), U2.2 (GND), U2.3 (GND), U4.10 (GND), J10.1 (Pin_1), J7.1 (Pin_1), J8.1 (Pin_1), J9.1 (Pin_1), U1.2 (GND), U3.2 (GND), U6.2 (GND)
- net RBTQ_1: now reaches U5.J1_4 (GPIO4)
- net RBTQ_1: now also J1.3 (Pin_3)
- net RBTQ_2: now reaches U5.J1_5 (GPIO5)
- net RBTQ_2: now also J1.4 (Pin_4)
- net Misc1_G6: now reaches U5.J1_6 (GPIO6)
- net Misc1_G6: now also J7.3 (Pin_3)
- net Misc1_G7: now reaches U5.J1_7 (GPIO7)
- net Misc1_G7: now also J8.3 (Pin_3)
- net Misc1_G15: now reaches U5.J1_8 (GPIO15)
- net Misc1_G15: now also J8.4 (Pin_4)
- net S2_TX: now reaches U5.J1_9 (GPIO16)
- net S2_TX: now also J3.3 (Pin_3)
- net S1_RX: now reaches U5.J3_16 (GPIO48)
- net S1_RX: now also J2.4 (Pin_4)
- net S1_TX: now reaches U5.J3_17 (GPIO47)
- net S1_TX: now also J2.3 (Pin_3)
- net Misc1_G21: now reaches U5.J3_18 (GPIO21)
- net Misc1_G21: now also J7.4 (Pin_4)
- net Misc1_G1: now reaches U5.J3_4 (GPIO1)
- net Misc1_G1: now also J9.3 (Pin_3)
- net Misc1_G2: now reaches U5.J3_5 (GPIO2)
- net Misc1_G2: now also J9.4 (Pin_4)
- net at U2.4 (VOut): now also U6.1 (VIN)
- net at J5.2 (Pin_2): now also U3.1 (VIN)
- new net: R2.2, U3.3 (~{CE})
- new net: R3.2, U6.3 (~{CE})
- no-connect marks 4 -> 38
Other:
- moved on the sheet: C1, C3, C7, H1, H2, H3, H4, J1, J2, J3, J4, J5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
