File: Sabe-FullSized/Sabe-FullSized.kicad_sch (KiCad schematic)
At the start: 24 parts, among them J1 Roboteq, J10 Misc 4, J2 Serial 1, J3 Serial 2, J4 Serial 3, J5 5V, J7 Misc 1, J8 Misc 2, J9 Misc 3, U1 LM2937xT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

Commit message: updates
Parts:
- added J11, J6: Conn_01x02, Connector_PinHeader_2.54mm:PinHeader_1x02_P2.54mm_Vertical, symbol Connector_Generic:Conn_01x02
- added R2, R3: 470, Resistor_THT:R_Axial_DIN0207_L6.3mm_D2.5mm_P10.16mm_Horizontal, symbol Device:R_Small
Connections:
- net RST: now reaches U5.J1_3 (RST)
- net RST: now also U7.2 (D1)
- net GPIO_0: now reaches U5.J3_14 (GPIO0)
- net GPIO_0: now also U7.3 (D2)
- net S6TX_C6RX: now reaches U5.J3_2 (U0TXD/GPIO43)
- net S6TX_C6RX: now also R2.1
- net S6RX_C6TX: now reaches U5.J3_3 (U0RXD/GPIO44)
- net S6RX_C6TX: now also R3.1
- net at U7.10 (D9): now also R3.2
- net at U7.9 (D8): now also R2.2
- no-connect marks 34 -> 30
Other:
- moved on the sheet: U7

Commit message: sabe
Parts:
- removed J10: Misc 4, Connector_PinHeader_2.54mm:PinHeader_1x04_P2.54mm_Vertical, symbol Connector_Generic:Conn_01x04
- J6: value Conn_01x02 -> Dome PWM
Connections:
- net Misc1_G10 is gone; now on net ESTOP: U5.J1_16 (GPIO10)
- net Misc1_G11 is gone; now on net S1_RX: U5.J1_17 (GPIO11)
- net 5V: now also U7.14 (VUSB)
- net GND: now also J11.1 (Pin_1), J6.1 (Pin_1), U7.13 (GND)
- net Misc1_G1: now also J7.3 (Pin_3); no longer J9.3 (Pin_3)
- net Misc1_G2: now also J7.4 (Pin_4); no longer J9.4 (Pin_4)
- net RBTQ_1: now also U5.J1_7 (GPIO7); no longer U5.J1_4 (GPIO4)
- net RBTQ_2: now also U5.J1_12 (GPIO8); no longer U5.J1_5 (GPIO5)
- net S1_RX: no longer U5.J3_16 (GPIO48)
- net S1_TX: now also U5.J1_18 (GPIO12); no longer U5.J3_17 (GPIO47)
- net S2_RX: now also U5.J1_19 (GPIO13); no longer U5.J1_12 (GPIO8)
- net S2_TX: now also U5.J1_20 (GPIO14); no longer U5.J1_9 (GPIO16)
- net S3_RX: now also J4.3 (Pin_3), U5.J1_8 (GPIO15); no longer J4.4 (Pin_4), U5.J1_20 (GPIO14)
- net S3_TX: now also J4.4 (Pin_4), U5.J1_9 (GPIO16); no longer J4.3 (Pin_3), U5.J1_19 (GPIO13)
- net xbee_din: now also U5.J1_5 (GPIO5); no longer U5.J1_10 (GPIO17)
- net xbee_dout: now also U5.J1_4 (GPIO4); no longer U5.J1_11 (GPIO18)
- net xbee_rst: now also U5.J1_6 (GPIO6); no longer U5.J1_15 (GPIO9)
- net ESTOP: now reaches J11.2 (Pin_2)
- net Dome_PWM: now reaches J6.2 (Pin_2)
- net Dome_PWM: now also U5.J1_15 (GPIO9)
- net Misc1_G15 renamed Misc2_G18
- net Misc2_G18: no longer U5.J1_8 (GPIO15)
- net Misc1_G21: no longer names the net of U5.J3_18 (GPIO21)
- net Misc1_G21: no longer J7.4 (Pin_4)
- removed net Misc1_G6: J7.3 (Pin_3), U5.J1_6 (GPIO6)
- net Misc1_G7 renamed Misc2_G17
- net Misc2_G17: no longer U5.J1_7 (GPIO7)
- new net Misc3_G47: J9.3 (Pin_3), U5.J3_17 (GPIO47)
- new net Misc3_G48: J9.4 (Pin_4), U5.J3_16 (GPIO48)
- no-connect marks 30 -> 38
Other:
- moved on the sheet: J11, J6
