File: Sabe-FullSized/Sabe-FullSized.kicad_pcb (KiCad board)
At the start: 2 copper layers, 67.9 x 86.3 mm, 29 parts, among them J1 Roboteq, J2 Conn_01x04, J3 Conn_01x04, J4 Conn_01x04, J5 5V, J6 6-36V, U2 D24V550F5_Step_Down_Regulator, U3 MCP1700x-330xxTO, U5 ESP32-S3-DEVKITC-1-N8R2

Commit message: sabe
Parts:
- removed D2, D3: D_Schottky, Diode_THT:D_DO-201AD_P12.70mm_Horizontal
- removed the J1 at (207.4, 127.7)
- removed the J2 at (207.4, 124.1)
- removed the J3 at (207.4, 120.5)
- removed the J3 at (207.4, 113.2)
- removed the J4 at (207.4, 116.8)
- removed the J4 at (207.4, 109.5)
- added G***: LOGO, 01-Custom:SABEQR_20, F.Cu at (140.1, 66.4)
- added G***: LOGO, 01-Custom:SabeLogo25W, F.Cu at (168.0, 52.5)
- added G***: LOGO, 01-Custom:R2_Logo_V2, F.Cu at (181.3, 61.4)
- added G***: LOGO, 01-Custom:SABEQR_20, B.Cu at (168.2, 76.3)
- added G***: LOGO, 01-Custom:BB_Logo, B.Cu at (140.2, 67.3)
- added J10: Misc 4, Connector_PinHeader_2.54mm:PinHeader_1x04_P2.54mm_Vertical, F.Cu at (139.5, 85.0)
- added J7: Misc 1, Connector_PinHeader_2.54mm:PinHeader_1x04_P2.54mm_Vertical, F.Cu at (139.5, 101.9)
- added J8: Misc 2, Connector_PinHeader_2.54mm:PinHeader_1x04_P2.54mm_Vertical, F.Cu at (139.5, 96.3)
- added J9: Misc 3, Connector_PinHeader_2.54mm:PinHeader_1x04_P2.54mm_Vertical, F.Cu at (139.5, 90.7)
- added R2: 100, Resistor_THT:R_Axial_DIN0207_L6.3mm_D2.5mm_P10.16mm_Horizontal, F.Cu at (160.5, 105.4)
- added R3: 100, Resistor_THT:R_Axial_DIN0207_L6.3mm_D2.5mm_P10.16mm_Horizontal, F.Cu at (139.6, 118.6)
- added U1: LM2937xT, Package_TO_SOT_THT:TO-220-3_Vertical, F.Cu at (166.8, 87.4)
- added U6: LM66100DCK, Package_TO_SOT_SMD:SOT-363_SC-70-6, F.Cu at (141.9, 112.2)
- C2: value 1uf -> 10uf; footprint Capacitor_THT:C_Disc_D7.5mm_W4.4mm_P5.00mm -> Capacitor_THT:CP_Radial_D5.0mm_P2.00mm
- J2: value Conn_01x04 -> Serial 1
- J3: value Conn_01x04 -> Serial 2
- J4: value Conn_01x04 -> Serial 3
- U3: value MCP1700x-330xxTO -> LM66100DCK; footprint Package_TO_SOT_THT:TO-92_Inline -> Package_TO_SOT_SMD:SOT-363_SC-70-6
- moved J5 77.4 mm to (127.9, 120.2), turned to 0 degrees
- moved U3 73.9 mm to (170.5, 110.2)
- moved J1 72.4 mm to (127.2, 96.8)
- moved J2 72.4 mm to (127.2, 93.1)
- moved J3 72.4 mm to (127.2, 89.4)
- moved J4 72.4 mm to (127.2, 85.7)
- moved U2 72.0 mm to (146.0, 117.2)
- moved C1 69.5 mm to (163.5, 93.6)
- moved C2 69.5 mm to (168.6, 96.3)
- moved U5 69.1 mm to (168.4, 95.4)
- moved H1 69.0 mm to (170.4, 47.7)
- moved H3 69.0 mm to (170.4, 126.2)
- moved H4 69.0 mm to (120.9, 126.3)
- moved U4 69.0 mm to (140.1, 66.1)
- moved C3 69.0 mm to (123.7, 65.0)
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Connections:
- C1 pad 2: 5V -> GND
- C2 pad 2: 5V -> GND
- C3 pad 1: unconnected-(C3-Pad1) -> 3.3V
- C3 pad 2: unconnected-(C3-Pad2) -> GND
- C4 pad 1: unconnected-(C4-Pad1) -> 3.3V
- C4 pad 2: unconnected-(C4-Pad2) -> GND
- C6 pad 2: 5V -> GND
- C7 pad 2: 5V -> GND
- J1 pad 1: unconnected-(J1-Pin_1-Pad1) -> GND
- J1 pad 2: unconnected-(J1-Pin_2-Pad2) -> 5V
- J1 pad 3: unconnected-(J1-Pin_3-Pad3) -> RBTQ_1
- J1 pad 4: unconnected-(J1-Pin_4-Pad4) -> RBTQ_2
- J2 pad 1: unconnected-(J2-Pin_1-Pad1) -> GND
- J2 pad 2: unconnected-(J2-Pin_2-Pad2) -> 5V
- J2 pad 3: unconnected-(J2-Pin_3-Pad3) -> S1_TX
- J2 pad 4: unconnected-(J2-Pin_4-Pad4) -> S1_RX
- J3 pad 1: unconnected-(J3-Pin_1-Pad1) -> GND
- J3 pad 2: unconnected-(J3-Pin_2-Pad2) -> 5V
- J3 pad 3: unconnected-(J3-Pin_3-Pad3) -> S2_TX
- J3 pad 4: unconnected-(J3-Pin_4-Pad4) -> S2_RX
- J4 pad 1: unconnected-(J4-Pin_1-Pad1) -> GND
- J4 pad 2: unconnected-(J4-Pin_2-Pad2) -> 5V
- J4 pad 3: unconnected-(J4-Pin_3-Pad3) -> S3_TX
- J4 pad 4: unconnected-(J4-Pin_4-Pad4) -> S3_RX
- J5 pad 1: 5V -> GND
- J5 pad 2: Net-(D2-K) -> Net-(J5-Pin_2)
- J6 pad 1: 5V -> GND
- R1 pad 1: unconnected-(R1-Pad1) -> xbee_rst
- R1 pad 2: unconnected-(R1-Pad2) -> 3.3V
- U2 pad 0: unconnected-(U2-En-Pad0) -> Net-(J6-Pin_2)
- U2 pad 2: 5V -> GND
- U2 pad 3: 5V -> GND
- U3 pad 1: 3.3V -> Net-(J5-Pin_2)
- U3 pad 2: 5V -> GND
- U3 pad 3: 5V -> Net-(U3-~{CE})
- U4 pad 1: unconnected-(U4-VCC-Pad1) -> 3.3V
- U4 pad 10: unconnected-(U4-GND-Pad10) -> GND
- U4 pad 2: unconnected-(U4-DOUT-Pad2) -> xbee_dout
- U4 pad 3: unconnected-(U4-DIN-Pad3) -> xbee_din
- U4 pad 5: unconnected-(U4-~{RESET}-Pad5) -> xbee_rst
- U5 pad J1_1: Net-(U5-3V3-PadJ1_1) -> unconnected-(U5-3V3-PadJ1_1)_1
- U5 pad J1_10: unconnected-(U5-GPIO17-PadJ1_10) -> xbee_din
- U5 pad J1_11: unconnected-(U5-GPIO18-PadJ1_11) -> xbee_dout
- U5 pad J1_12: unconnected-(U5-GPIO8-PadJ1_12) -> S2_RX
- U5 pad J1_15: unconnected-(U5-GPIO9-PadJ1_15) -> xbee_rst
- U5 pad J1_16: unconnected-(U5-GPIO10-PadJ1_16) -> Misc1_G10
- U5 pad J1_17: unconnected-(U5-GPIO11-PadJ1_17) -> Misc1_G11
- U5 pad J1_19: unconnected-(U5-GPIO13-PadJ1_19) -> S3_TX
- U5 pad J1_2: Net-(U5-3V3-PadJ1_1) -> unconnected-(U5-3V3-PadJ1_1)
- U5 pad J1_20: unconnected-(U5-GPIO14-PadJ1_20) -> S3_RX
- U5 pad J1_22: Net-(U5-GND-PadJ1_22) -> GND
- U5 pad J1_4: unconnected-(U5-GPIO4-PadJ1_4) -> RBTQ_1
- U5 pad J1_5: unconnected-(U5-GPIO5-PadJ1_5) -> RBTQ_2
- U5 pad J1_6: unconnected-(U5-GPIO6-PadJ1_6) -> Misc1_G6
- U5 pad J1_7: unconnected-(U5-GPIO7-PadJ1_7) -> Misc1_G7
- U5 pad J1_8: unconnected-(U5-GPIO15-PadJ1_8) -> Misc1_G15
- U5 pad J1_9: unconnected-(U5-GPIO16-PadJ1_9) -> S2_TX
- U5 pad J3_1: Net-(U5-GND-PadJ1_22) -> GND
- U5 pad J3_16: unconnected-(U5-GPIO48-PadJ3_16) -> S1_RX
- U5 pad J3_17: unconnected-(U5-GPIO47-PadJ3_17) -> S1_TX
- U5 pad J3_18: unconnected-(U5-GPIO21-PadJ3_18) -> Misc1_G21
- U5 pad J3_21: Net-(U5-GND-PadJ1_22) -> GND
- U5 pad J3_22: Net-(U5-GND-PadJ1_22) -> GND
- U5 pad J3_4: unconnected-(U5-GPIO1-PadJ3_4) -> Misc1_G1
- U5 pad J3_5: unconnected-(U5-GPIO2-PadJ3_5) -> Misc1_G2
Routing:
- net xbee_rst: track 0.00 -> 65.7 mm
- net S1_TX: track 0.00 -> 55.6 mm
- net RBTQ_1: track 0.00 -> 55.6 mm
- net RBTQ_2: track 0.00 -> 55.4 mm
- net Misc1_G1: track 0.00 -> 54.8 mm
- net S1_RX: track 0.00 -> 51.9 mm
- net Misc1_G2: track 0.00 -> 49.6 mm
- net xbee_din: track 0.00 -> 49.4 mm
- net S3_TX: track 0.00 -> 47.1 mm
- net Net-(J5-Pin_2): track 0.00 -> 46.6 mm
- net xbee_dout: track 0.00 -> 44.6 mm
- net S3_RX: track 0.00 -> 43.6 mm
- net Misc1_G21: track 0.00 -> 38.0 mm
- net Misc1_G6: track 0.00 -> 33.7 mm
- net Misc1_G10: track 0.00 -> 29.5 mm
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- added copper zone on In1.Cu, net 3.3V
- added copper zone on F.Cu, net 5V
- added copper zone on B.Cu, net GND
Other:
- copper layers 2 -> 4
- board text added: "1"
- board text added: "10"
- board text added: "11"
- board text added: "15"
- board text added: "2"
- board text added: "21"
- board text added: "6"
- board text added: "7"
- board text added: "Misc 1"
- board text added: "Misc 2"
- board text added: "Misc 3"
- board text added: "Misc 4"
- board text added: "Ver: 1.1 DATE: 28 MAY 26"
- board text removed: "sabé ver: 1.0 date: 21 may 26"

Commit message: updates
Parts:
- removed U2: D24V550F5_Step_Down_Regulator, custom:D24V50F5_Step_Down_Regulator
- removed U3, U6: LM66100DCK, Package_TO_SOT_SMD:SOT-363_SC-70-6
- added J11: Conn_01x02, Connector_PinHeader_2.54mm:PinHeader_1x02_P2.54mm_Vertical, F.Cu at (127.7, 106.3)
- added U7: XIAO_ESP32C3, 01-Custom:MODULE_XIAO_ESP32C3, F.Cu at (144.7, 115.3)
- J6: value 6-36V -> Conn_01x02; footprint TerminalBlock_Phoenix:TerminalBlock_Phoenix_MKDS-1,5-2-5.08_1x02_P5.08mm_Horizontal -> Connector_PinHeader_2.54mm:PinHeader_1x02_P2.54mm_Vertical
- R2, R3: value 100 -> 470
- moved R3 56.3 mm to (173.7, 73.7), turned to 180 degrees
- moved R2 38.0 mm to (173.6, 69.8), turned to 180 degrees
- moved J6 5.42 mm to (127.5, 101.0), turned to 90 degrees
- moved J5 3.11 mm to (126.4, 117.5)
- moved J1 0.38 mm to (126.9, 96.5)
- moved J2 0.38 mm to (126.9, 92.8)
- moved J3 0.38 mm to (126.9, 89.1)
- moved J4 0.38 mm to (126.9, 85.4)
Connections:
- J5 pad 2: Net-(J5-Pin_2) -> 5V
- J6 pad 1: GND -> unconnected-(J6-Pin_1-Pad1)
- J6 pad 2: Net-(J6-Pin_2) -> unconnected-(J6-Pin_2-Pad2)
- R2 pad 1: 5V -> S6TX_C6RX
- R3 pad 1: 5V -> S6RX_C6TX
- U5 pad J1_3: unconnected-(U5-RST-PadJ1_3) -> RST
- U5 pad J3_14: unconnected-(U5-GPIO0-PadJ3_14)_1 -> GPIO_0
- U5 pad J3_2: unconnected-(U5-U0TXD/GPIO43-PadJ3_2) -> S6TX_C6RX
- U5 pad J3_3: unconnected-(U5-U0RXD/GPIO44-PadJ3_3) -> S6RX_C6TX
Routing:
- net Net-(J5-Pin_2): track 46.6 -> 0.00 mm
- net Net-(J6-Pin_2): track 22.5 -> 0.00 mm
- net GND: track 22.1 -> 5.08 mm, vias 2 -> 0
- net Net-(U7-D9): track 11.8 -> 0.00 mm
- net Net-(U7-D8): track 4.51 -> 0.00 mm
- net Net-(U2-VOut): track 4.05 -> 0.00 mm
Other:
- board text added: "Dome"
- board text added: "E-STOP"
- board text added: "S"
- board text added: "Ver: 1.2 DATE: 28 MAY 26"
- board text removed: "- 6-36V +"
- board text removed: "Ver: 1.1 DATE: 28 MAY 26"

Commit message: sabe
Parts:
- removed J10: Misc 4, Connector_PinHeader_2.54mm:PinHeader_1x04_P2.54mm_Vertical
- J6: value Conn_01x02 -> Dome PWM
- moved R2 46.2 mm to (175.8, 116.0)
- moved R3 45.5 mm to (175.8, 119.1)
- moved G*** 17.2 mm to (167.9, 72.1)
- moved G*** 12.5 mm to (155.9, 49.2)
- moved J8 5.11 mm to (139.7, 91.2)
- moved J7 5.09 mm to (139.6, 96.8)
- moved J9 5.07 mm to (139.8, 85.6)
- moved H1 3.35 mm to (171.0, 51.0)
- moved H2 3.29 mm to (121.0, 51.0)
- moved R1 2.49 mm to (123.6, 80.9)
- moved C4 2.07 mm to (124.0, 57.5)
- moved J1 1.80 mm to (127.2, 98.3)
- moved J11 1.80 mm to (127.9, 108.1)
- moved J6 1.80 mm to (127.7, 102.8)
- moved U4 1.44 mm to (140.2, 64.7)
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Connections:
- J11 pad 1: unconnected-(J11-Pin_1-Pad1) -> GND
- J11 pad 2: unconnected-(J11-Pin_2-Pad2) -> ESTOP
- J4 pad 3: S3_TX -> S3_RX
- J4 pad 4: S3_RX -> S3_TX
- J6 pad 1: unconnected-(J6-Pin_1-Pad1) -> GND
- J6 pad 2: unconnected-(J6-Pin_2-Pad2) -> Dome_PWM
- J7 pad 3: Misc1_G6 -> Misc1_G1
- J7 pad 4: Misc1_G21 -> Misc1_G2
- J8 pad 3: Misc1_G7 -> Misc2_G17
- J8 pad 4: Misc1_G15 -> Misc2_G18
- J9 pad 3: Misc1_G1 -> Misc3_G47
- J9 pad 4: Misc1_G2 -> Misc3_G48
- U5 pad J1_10: xbee_din -> unconnected-(U5-GPIO17-PadJ1_10)
- U5 pad J1_11: xbee_dout -> unconnected-(U5-GPIO18-PadJ1_11)
- U5 pad J1_12: S2_RX -> RBTQ_2
- U5 pad J1_15: xbee_rst -> Dome_PWM
- U5 pad J1_16: Misc1_G10 -> ESTOP
- U5 pad J1_17: Misc1_G11 -> S1_RX
- U5 pad J1_18: unconnected-(U5-GPIO12-PadJ1_18) -> S1_TX
- U5 pad J1_19: S3_TX -> S2_RX
- U5 pad J1_20: S3_RX -> S2_TX
- U5 pad J1_4: RBTQ_1 -> xbee_dout
- U5 pad J1_5: RBTQ_2 -> xbee_din
- U5 pad J1_6: Misc1_G6 -> xbee_rst
- U5 pad J1_7: Misc1_G7 -> RBTQ_1
- U5 pad J1_8: Misc1_G15 -> S3_RX
- U5 pad J1_9: S2_TX -> S3_TX
- U5 pad J3_16: S1_RX -> Misc3_G48
- U5 pad J3_17: S1_TX -> Misc3_G47
- U5 pad J3_18: Misc1_G21 -> unconnected-(U5-GPIO21-PadJ3_18)
- U7 pad 13: unconnected-(U7-GND-Pad13) -> GND
- U7 pad 14: unconnected-(U7-VUSB-Pad14) -> 5V
Routing:
- net RST: track 0.00 -> 57.9 mm
- net S6TX_C6RX: track 0.00 -> 53.2 mm
- net S6RX_C6TX: track 0.00 -> 52.8 mm
- net Misc3_G47: track 0.00 -> 48.9 mm
- net Net-(U7-D8): track 0.00 -> 44.9 mm
- net Misc3_G48: track 0.00 -> 43.6 mm
- net Net-(U7-D9): track 0.00 -> 40.8 mm
- net GPIO_0: track 0.00 -> 38.1 mm
- net Misc1_G21: track 38.0 -> 0.00 mm
- net Misc1_G6: track 33.7 -> 0.00 mm
- net RBTQ_2: track 55.4 -> 24.4 mm
- net Misc1_G10: track 29.5 -> 0.00 mm
- net ESTOP: track 0.00 -> 28.8 mm
- net Dome_PWM: track 0.00 -> 27.5 mm
- net Misc1_G11: track 26.3 -> 0.00 mm
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Other:
- board text added: "17"
- board text added: "18"
- board text added: "47"
- board text added: "48"
- board text added: "P1"
- board text added: "P2"
- board text added: "Ver: 1.4 DATE: 26 JUNE 26"
- board text removed: "10"
- board text removed: "11"
- board text removed: "15"
- board text removed: "21"
- board text removed: "6"
- board text removed: "7"
- board text removed: "Misc 4"
- board text removed: "Ver: 1.2 DATE: 28 MAY 26"

Commit message: updates
Routing:
- net unconnected-(U5-USB_D-/GPIO19-PadJ3_20)_1: track 0.00 -> 2.54 mm
- net unconnected-(U5-USB_D+/GPIO20-PadJ3_19)_1: track 0.00 -> 2.54 mm
- net unconnected-(U5-MTMS/GPIO42-PadJ3_6): track 0.00 -> 2.54 mm
- net unconnected-(U5-MTDO/GPIO40-PadJ3_8): track 0.00 -> 2.54 mm
- net unconnected-(U5-MTDI/GPIO41-PadJ3_7): track 0.00 -> 2.54 mm
- net unconnected-(U5-MTCK/GPIO39-PadJ3_9)_1: track 0.00 -> 2.54 mm
- net unconnected-(U5-GPIO45-PadJ3_15): track 0.00 -> 2.54 mm
- net unconnected-(U5-GPIO38-PadJ3_10): track 0.00 -> 2.54 mm
- net unconnected-(U5-GPIO37-PadJ3_11)_1: track 0.00 -> 2.54 mm
- net unconnected-(U5-GPIO36-PadJ3_12): track 0.00 -> 2.54 mm
- net unconnected-(U5-GPIO35-PadJ3_13): track 0.00 -> 2.54 mm
- net unconnected-(U5-GPIO21-PadJ3_18): track 0.00 -> 2.54 mm
Changed lines of the file:
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@@
 			(outputformat 1)
 			(mirror no)
-			(drillshape 1)
+			(drillshape 0)
 			(scaleselection 1)
-			(outputdirectory "")
+			(outputdirectory "Gerbers/Sabe_V1.4_271448RJUN26/")
 		)
 	)
@@
 	)
 	(segment
+		(start 179.86 80.67)
+		(end 182.4 80.67)
+		(width 0.2)
+		(layer "F.Cu")
+		(net 3)
+	)
+	(segment
+		(start 179.86 78.13)
+		(end 182.4 78.13)
+		(width 0.2)
+		(layer "F.Cu")
+		(net 4)
+	)
+	(segment
+		(start 179.86 88.29)
+		(end 182.4 88.29)
+		(width 0.2)
+		(layer "F.Cu")
+		(net 5)
+	)
+	(segment
+		(start 182.4 83.21)
+		(end 179.86 83.21)
+		(width 0.2)
+		(layer "F.Cu")
+		(net 6)
+	)
+	(segment
 		(start 157 80.67)
 		(end 153.595 80.67)
@@
 	)
 	(segment
+		(start 182.4 100.99)
+		(end 179.86 100.99)
+		(width 0.2)
+		(layer "F.Cu")
+		(net 23)
+	)
+	(segment
 		(start 153.125 55.149136)
 		(end 152.17598 54.200116)
@@
 	)
 	(segment
+		(start 182.4 95.91)
+		(end 179.86 95.91)
+		(width 0.2)
+		(layer "F.Cu")
+		(net 41)
+	)
+	(segment
+		(start 179.86 93.37)
+		(end 182.4 93.37)
+		(width 0.2)
+		(layer "F.Cu")
+		(net 43)
+	)
+	(segment
+		(start 182.4 90.83)
+		(end 179.86 90.83)
+		(width 0.2)
+		(layer "F.Cu")
+		(net 44)
+	)
+	(segment
+		(start 182.4 111.15)
+		(end 179.86 111.15)
+		(width 0.2)
+		(layer "F.Cu")
+		(net 45)
+	)
+	(segment
+		(start 179.86 85.75)
+		(end 182.4 85.75)
+		(width 0.2)
+		(layer "F.Cu")
+		(net 46)
+	)
+	(segment
+		(start 179.86 113.69)
+		(end 182.4 113.69)
+		(width 0.2)
+		(layer "F.Cu")
+		(net 48)
+	)
+	(segment
 		(start 176.875 114.855)
 		(end 176.875 69.375)
@@
 		(end 182.4 98.45)
 		(width 0.25)
-		(layer "B.Cu")
+		(layer "F.Cu")
 		(net 63)
 	)
@@
 	)
 	(segment
+		(start 179.86 108.61)
+		(end 182.4 108.61)
+		(width 0.2)
+		(layer "F.Cu")
+		(net 65)
+	)
+	(segment
 		(start 182.4 106.07)
 		(end 179.86 106.07)
@@
 	)
 	(segment
-		(start 182.4 103.53)
-		(end 179.86 103.53)
+		(start 179.86 103.53)
+		(end 182.4 103.53)
 		(width 0.25)
-		(layer "In1.Cu")
+		(layer "F.Cu")
 		(net 67)
 	)
