File: R2_HH_Controllers/R2_HH_Controllers.kicad_sch (KiCad schematic)
At the start: 27 parts, among them IC1 E22-900M22S, J1 U.FL-R-SMT-1_10_, J2 USB4105-GF-A, J3 S2B-PH-SM4-TB_LF__SN_, SW1 SW_Push, SW10 SW_Push, SW11 SW_Push, SW2 Reset, SW3 Boot, SW4 SW_Push, SW5 PCM12SMTR, SW6 SW_Push, SW7 SW_Push, SW8 SW_Push, SW9 SW_Push, U1 ESP32-S3-WROOM-1, U2 USBLC6-2SC6, U3 BQ24074RGT

Commit message: hh
Parts:
- removed J1: U.FL-R-SMT-1_10_, custom:HRS_U.FL-R-SMT-1_10_, symbol 01-Custom:U.FL-R-SMT-1_10_
- added C10: 22uf, Capacitor_SMD:C_0201_0603Metric, symbol Device:C
- added C11, C4: .1uf, Capacitor_SMD:C_0201_0603Metric, symbol Device:C
- added C5, C7, C8, C9: 1uf, Capacitor_SMD:C_0201_0603Metric, symbol Device:C
- added C6: 10uf, Capacitor_SMD:C_0201_0603Metric, symbol Device:C
- added R10: 17.8K, Resistor_SMD:R_0201_0603Metric, symbol Device:R
- added R3, R4: 5.1K, Resistor_SMD:R_0201_0603Metric, symbol Device:R
- added R5, R6, R7: 10K, Resistor_SMD:R_0201_0603Metric, symbol Device:R
- added R8: 1.8K, Resistor_SMD:R_0201_0603Metric, symbol Device:R
- added R9: 1.62K, Resistor_SMD:R_0201_0603Metric, symbol Device:R
- added U5: AP2112K-3.3, Package_TO_SOT_SMD:SOT-23-5, symbol Regulator_Linear:AP2112K-3.3
Connections:
- net BAT+ is gone; now on net CHARGER_OUT: SW5.1
- net SHELL_GND is gone; now on net GND: J2.SH1 (SHELL_GND), J2.SH2 (SHELL_GND), J2.SH3 (SHELL_GND), J2.SH4 (SHELL_GND)
- net 3.3V_REG: now also U2.5 (VBUS), U3.6 (EN1), C10.2, C11.2, C9.2, R6.2, U5.5 (VOUT)
- net BAT+_SWITCHED: now also C8.2, U5.1 (VIN), U5.3 (EN)
- net D+: now also J2.A6 (DP1), J2.B6 (DP2), U2.6 (I/O1); no longer U1.14 (USB_D+)
- net D-: now also J2.A7 (DN1), J2.B7 (DN2), U2.4 (I/O2); no longer U1.13 (USB_D-)
- net GND: now also E1.2, J3.2, J3.S1 (SHIELD), J3.S2 (SHIELD), SW3.2, U2.2 (GND), U3.17 (VSS), U3.4 (~{CE}), U3.5 (EN2), U3.8 (VSS), C10.1, C11.1, C4.1, C5.1, C6.1, C7.1, C8.1, C9.1, R10.1, R3.2, R4.1, R7.1, R8.1, R9.1, U5.2 (GND)
- net VBUS: now also U3.13 (IN), C5.2
- net at U3.1 (TS): now also R5.1, R7.2
- net CHARGER_OUT: now reaches U3.10 (OUT), U3.11 (OUT)
- net CHARGER_OUT: now also C7.2
- net at U3.12 (ILIM): now also R9.2
- net at U3.14 (TMR): now also C4.2
- net at U3.15 (ITERM): now also R10.2
- net at U3.16 (ISET): now also R8.2
- net JST_BAT+: now reaches U3.2 (BAT), U3.3 (BAT)
- net JST_BAT+: now also J3.1, C6.2, R5.2
- net at C1.1, R2.1, U1.3 (EN): now also SW2.2
- net at J2.A5 (CC1): now also R3.1
- net at J2.B5 (CC2): now also R4.2
- net BUSY: now reaches IC1.14 (BUSY)
- net BUSY: now also U1.8 (IO15)
- net RST: now reaches IC1.15 (NRST)
- net RST: now also U1.22 (IO14)
- net MISO: now reaches IC1.16 (MISO)
- net MISO: now also U1.21 (IO13)
- net MOSI: now reaches IC1.17 (MOSI)
- net MOSI: now also U1.19 (IO11)
- net SCK: now reaches IC1.18 (SCK)
- net SCK: now also U1.20 (IO12)
- net NSS: now reaches IC1.19 (NSS)
- net NSS: now also U1.18 (IO10)
- net at IC1.21 (ANT): now also E1.1
- net at SW3.1: now also U1.27 (IO0), R6.1
- net D+_ESP: now reaches U2.1 (I/O1)
- net D+_ESP: now also U1.14 (USB_D+)
- net D-_ESP: now reaches U2.3 (I/O2)
- net D-_ESP: now also U1.13 (USB_D-)
- net DIO1: now reaches U1.9 (IO16)
- no-connect marks 1 -> 5
Other:
- moved on the sheet: C1, D1, E1, IC1, J3, R1, R2, SW1, SW10, SW11, SW2, SW3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

Commit message: hh
Parts:
- removed U4: ~, 01-Custom:A24AH, symbol 01-Custom:A24AH
- removed VR1: RKJXV1224005, 01-Custom:RKJXV1224005, symbol 01-Custom:RKJXV1224005
- added C12, C13, C14, C15, C16: 100nf, Capacitor_SMD:C_0201_0603Metric, symbol Device:C
- added R11: 10K, Resistor_SMD:R_0201_0603Metric, symbol Device:R
- added R15: 330, Resistor_SMD:R_0201_0603Metric, symbol Device:R
- added S1: RKJXV122400R, 01-Custom:RKJXV122400R, symbol 01-Custom:RKJXV122400R
- renumbered SW2 to SW10, SW3 to SW12, SW4 to SW2, SW6 to SW3, SW7 to SW4, SW11 to SW5, SW10 to SW6, SW9 to SW7, SW5 to SW9
Connections:
- net 3.3V_REG: now also R1.1, C16.2, R11.2, S1.A13, S1.B13
- net GND: now also C1.1, R1.3, SW1.2, SW2.2, SW3.2, SW4.2, SW5.2, SW6.2, SW7.2, SW8.2, C12.1, C13.1, C14.1, C15.1, C16.1, S1.A11, S1.B1, S1.B11, S1.D1, S1.MH1, S1.MH2, S1.MH3, S1.MH4, S1.MH5, S1.MH6; no longer C1.2
- net BTN_8: now reaches SW8.1
- net BTN_8: now also U1.34 (IO41)
- net BTN_6: now reaches SW6.1
- net BTN_6: now also U1.32 (IO39)
- net at R2.1, U1.3 (EN): now also C1.2; no longer C1.1, SW10.2
- net BOOT: now reaches R6.1, SW12.1, U1.27 (IO0)
- net at D1.3 (DIN): now also R15.1
- net BTN_2: now reaches SW2.1
- net BTN_2: now also U1.10 (IO17)
- net POT_1: now reaches R1.2
- net POT_1: now also C15.2
- net BTN_5: now reaches SW5.1
- net BTN_5: now also U1.31 (IO38)
- net BTN_3: now reaches SW3.1
- net BTN_3: now also U1.11 (IO18)
- net BTN_7: now reaches SW7.1
- net BTN_7: now also U1.33 (IO40)
- net BTN_4: now reaches SW4.1
- net BTN_4: now also U1.23 (IO21)
- net BTN_1: now reaches SW1.1
- net BTN_1: now also U1.17 (IO9)
- net NEOPIXEL: now reaches U1.12 (IO8)
- net NEOPIXEL: now also R15.2
- net JOY_SWITCH: now reaches U1.15 (IO3)
- net JOY_SWITCH: now also C14.2, R11.1, S1.A1, S1.C1
- net JOY_Y: now reaches U1.38 (IO2)
- net JOY_Y: now also C13.2, S1.B12
- net JOY_X: now reaches U1.39 (IO1)
- net JOY_X: now also C12.2, S1.A12
- net MODE_1: now reaches U1.4 (IO4)
- net MODE_2: now reaches U1.5 (IO5)
- net MODE_3: now reaches U1.6 (IO6)
- net VOL_POT: now reaches U1.7 (IO7)
- new net EN: SW10.2
Other:
- moved on the sheet: E1, IC1, R1, R2, R6, SW1, SW10, SW12, SW2, SW3, SW4, SW5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

Commit message: hh
Parts:
- added C17, C18: 100nf, Capacitor_SMD:C_0603_1608Metric, symbol Device:C
- added D2, D3: WS2812B-2020, LED_SMD:LED_WS2812B-2020_PLCC4_2.0x2.0mm, symbol LED:WS2812B-2020
- added R12, R13: 330, Resistor_SMD:R_0603_1608Metric, symbol Device:R
- C1, C12, C13, C14, C15, C16, C2, C3, C4, C5, C6, C7, C8, C9: footprint Capacitor_SMD:C_0201_0603Metric -> Capacitor_SMD:C_0603_1608Metric
- C10, C11: footprint Capacitor_SMD:C_0201_0603Metric -> Capacitor_SMD:C_0805_2012Metric_Pad1.18x1.45mm_HandSolder
- R10, R11, R15, R2, R3, R4, R5, R6, R7, R8, R9: footprint Resistor_SMD:R_0201_0603Metric -> Resistor_SMD:R_0603_1608Metric
Connections:
- net 3.3V_REG: now also C17.2, C18.2, D2.4 (VDD), D3.4 (VDD)
- net GND: now also C17.1, C18.1, D2.2 (VSS), D3.2 (VSS)
- net at D1.1 (DOUT): now also R12.2
- new net: D3.3 (DIN), R13.1
- new net: D2.3 (DIN), R12.1
- new net: D2.1 (DOUT), R13.2

Commit message: updates
Parts:
- removed U1: ESP32-S3-WROOM-1, RF_Module:ESP32-S3-WROOM-1, symbol RF_Module:ESP32-S3-WROOM-1
- added R14: DNP, Resistor_SMD:R_0805_2012Metric_Pad1.20x1.40mm_HandSolder, symbol Device:R
- added U4: ESP32-S3-MINI-1, RF_Module:ESP32-S2-MINI-1, symbol RF_Module:ESP32-S3-MINI-1
Connections:
- net 3.3V_REG: now also U4.3 (3V3)
- net BOOT: now also U4.4 (IO0)
- net BTN_1: now also U4.13 (IO9)
- net BTN_2: now also U4.8 (IO4)
- net BTN_3: now also U4.9 (IO5)
- net BTN_4: now also U4.10 (IO6)
- net BTN_5: now also U4.21 (IO17)
- net BTN_6: now also U4.22 (IO18)
- net BTN_7: now also U4.25 (IO21)
- net BTN_8: now also U4.28 (IO33)
- net BUSY: now also U4.19 (IO15)
- net D+_ESP: now also U4.24 (USB_D+)
- net D-_ESP: now also U4.23 (USB_D-)
- net DIO1: now also U4.20 (IO16)
- net JOY_SWITCH: now also U4.7 (IO3)
- net JOY_X: now also U4.5 (IO1)
- net JOY_Y: now also U4.6 (IO2)
- net MISO: now also U4.17 (IO13)
- net MOSI: now also U4.15 (IO11)
- net NEOPIXEL: now also U4.12 (IO8)
- net NSS: now also U4.14 (IO10)
- net RST: now also U4.18 (IO14)
- net SCK: now also U4.16 (IO12)
- net VOL_POT: now also U4.11 (IO7)
- net at C1.2, R2.1: now also U4.45 (EN)
- net at IC1.21 (ANT): now also R14.2; no longer E1.1
- new net: U4.1 (GND), U4.2 (GND), U4.42 (GND), U4.43 (GND), U4.46 (GND), U4.47 (GND), U4.48 (GND), U4.49 (GND), U4.50 (GND), U4.51 (GND), U4.52 (GND), U4.53 (GND), U4.54 (GND), U4.55 (GND), U4.56 (GND), U4.57 (GND), U4.58 (GND), U4.59 (GND), U4.60 (GND), U4.61 (GND), U4.62 (GND), U4.63 (GND), U4.64 (GND), U4.65 (GND)
- new net: E1.1, R14.1
Other:
- moved on the sheet: E1

Commit message: updates
Parts:
- removed C1, C5, C7, C8, C9: 1uf, Capacitor_SMD:C_0603_1608Metric, symbol Device:C
- removed C10: 22uf, Capacitor_SMD:C_0805_2012Metric_Pad1.18x1.45mm_HandSolder, symbol Device:C
- removed C11: .1uf, Capacitor_SMD:C_0805_2012Metric_Pad1.18x1.45mm_HandSolder, symbol Device:C
- removed C12, C13, C14, C15, C16, C17, C18: 100nf, Capacitor_SMD:C_0603_1608Metric, symbol Device:C
- removed C2: 22uf, Capacitor_SMD:C_0603_1608Metric, symbol Device:C
- removed C3, C4: .1uf, Capacitor_SMD:C_0603_1608Metric, symbol Device:C
- removed C6: 10uf, Capacitor_SMD:C_0603_1608Metric, symbol Device:C
- removed D1, D2, D3: WS2812B-2020, LED_SMD:LED_WS2812B-2020_PLCC4_2.0x2.0mm, symbol LED:WS2812B-2020
- removed E1: ANT-915-USP410, custom:XDCR_ANT-915-USP410, symbol 01-Custom:ANT-915-USP410
- removed IC1: E22-900M22S, custom:E22-900M22S, symbol 01-Custom:E22-900M22S
- removed J2: USB4105-GF-A, 01-Custom:GCT_USB4105-GF-A, symbol 01-Custom:USB4105-GF-A
- removed J3: S2B-PH-SM4-TB_LF__SN_, 01-Custom:JST_S2B-PH-SM4-TB_LF__SN_, symbol 01-Custom:S2B-PH-SM4-TB_LF__SN_
- removed R1: 3352T-1-103LF, 01-Custom:TRIM_3352T-1-103LF, symbol 01-Custom:3352T-1-103LF
- removed R10: 17.8K, Resistor_SMD:R_0603_1608Metric, symbol Device:R
- removed R11, R2, R5, R6, R7: 10K, Resistor_SMD:R_0603_1608Metric, symbol Device:R
- removed R12, R13, R15: 330, Resistor_SMD:R_0603_1608Metric, symbol Device:R
- removed R14: DNP, Resistor_SMD:R_0805_2012Metric_Pad1.20x1.40mm_HandSolder, symbol Device:R
- removed R3, R4: 5.1K, Resistor_SMD:R_0603_1608Metric, symbol Device:R
- removed R8: 1.8K, Resistor_SMD:R_0603_1608Metric, symbol Device:R
- removed R9: 1.62K, Resistor_SMD:R_0603_1608Metric, symbol Device:R
- removed S1: RKJXV122400R, 01-Custom:RKJXV122400R, symbol 01-Custom:RKJXV122400R
- removed SW1, SW2, SW3, SW4, SW5, SW6, SW7, SW8: SW_Push, 01-Custom:TL3360CF185Q, symbol Switch:SW_Push
- removed SW10: Reset, Button_Switch_SMD:SW_SPST_TL3342, symbol Switch:SW_Push
- removed SW12: Boot, Button_Switch_SMD:SW_SPST_TL3342, symbol Switch:SW_Push
- removed SW9: PCM12SMTR, 01-Custom:SW_PCM12SMTR, symbol 01-Custom:PCM12SMTR
- removed U2: USBLC6-2SC6, Package_TO_SOT_SMD:SOT-23-6, symbol Power_Protection:USBLC6-2SC6
- removed U3: BQ24074RGT, Package_DFN_QFN:VQFN-16-1EP_3x3mm_P0.5mm_EP1.6x1.6mm, symbol Battery_Management:BQ24074RGT
- removed U4: ESP32-S3-MINI-1, RF_Module:ESP32-S2-MINI-1, symbol RF_Module:ESP32-S3-MINI-1
- removed U5: AP2112K-3.3, Package_TO_SOT_SMD:SOT-23-5, symbol Regulator_Linear:AP2112K-3.3
Connections:
- no-connect marks 5 -> 0
Other:
- added sheet Remote_Left_Hand (Navicore_Remote.kicad_sch)
- added sheet Remote_Right_Hand (Navicore_Remote.kicad_sch)
