File: R2_HH_Controllers/R2_HH_Controllers.kicad_sch (KiCad schematic)
At the start: 0 parts

Commit message: update
Parts:
- added U10, U12, U14, U16, U18, U20, U22, U24, U26, U28: ~, 01-Custom:mouse-bite-2.54mm-slot, symbol 01-Custom:mousebites
Other:
- note added: "Mousebites for board panelization"

Commit message: updates
Parts:
- U10, U12, U14, U16, U18, U20, U22, U24, U26, U28: value ~ -> (none)
