File: R2_HH_Controllers/Navicore_Remote.kicad_sch (KiCad schematic)
At the start: 56 parts, among them IC1 E22-900M22S, J1 USB4105-GF-A, J2 S2B-PH-SM4-TB_LF__SN_, SW1 SW_Push, SW10 Boot, SW11 PCM12SMTR, SW2 SW_Push, SW3 SW_Push, SW4 SW_Push, SW5 SW_Push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

Commit message: updates
Changed lines of the file:
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@@
 	(paper "A4")
 	(junction
-		(at 200.66 152.4)
-		(diameter 0)
-		(color 0 0 0 0)
-	)
-	(junction
 		(at 25.4 87.63)
 		(diameter 0)
@@
 	(wire
 		(pts
-			(xy 157.48 134.62) (xy 160.02 134.62)
-		)
-		(stroke
-			(width 0)
-			(type default)
-		)
-	)
-	(wire
-		(pts
 			(xy 156.21 172.72) (xy 168.91 172.72)
 		)
@@
 	(wire
 		(pts
-			(xy 200.66 152.4) (xy 196.85 152.4)
-		)
-		(stroke
-			(width 0)
-			(type default)
-		)
-	)
-	(wire
-		(pts
 			(xy 207.01 128.27) (xy 201.93 128.27)
 		)
@@
 	(wire
 		(pts
-			(xy 204.47 152.4) (xy 200.66 152.4)
-		)
-		(stroke
-			(width 0)
-			(type default)
-		)
-	)
-	(wire
-		(pts
 			(xy 146.05 22.86) (xy 146.05 27.94)
 		)
@@
 	(wire
 		(pts
-			(xy 157.48 130.81) (xy 157.48 134.62)
+			(xy 160.02 130.81) (xy 160.02 134.62)
 		)
 		(stroke
@@
 	(wire
 		(pts
-			(xy 157.48 123.19) (xy 157.48 121.92)
+			(xy 160.02 123.19) (xy 157.48 121.92)
 		)
 		(stroke
@@
 	(global_label "BAT+_SWITCHED"
 		(shape input)
-		(at 204.47 152.4 0)
+		(at 200.66 152.4 0)
 		(fields_autoplaced yes)
 		(effects
@@
 		)
 		(property "Intersheetrefs" "${INTERSHEET_REFS}"
-			(at 222.5742 152.4 0)
+			(at 218.7642 152.4 0)
 			(effects
 				(font
@@
 		(dnp no)
 		(property "Reference" "D1"
-			(at 118.364 135.128 0)
+			(at 110.49 137.16 0)
 			(effects
 				(font
@@
 	(symbol
 		(lib_id "Device:C")
-		(at 157.48 127 180)
+		(at 160.02 127 180)
 		(unit 1)
 		(exclude_from_sim no)
@@
 		(dnp no)
 		(property "Reference" "C13"
-			(at 153.67 128.2701 0)
+			(at 156.21 128.2701 0)
 			(effects
 				(font
@@
 		)
 		(property "Value" "1uf"
-			(at 159.004 129.54 0)
+			(at 161.544 129.54 0)
 			(effects
 				(font
@@
 		)
 		(property "Footprint" "Capacitor_SMD:C_0603_1608Metric"
-			(at 156.5148 123.19 0)
+			(at 159.0548 123.19 0)
 			(effects
 				(font
@@
 		)
 		(property "Datasheet" "~"
-			(at 157.48 127 0)
+			(at 160.02 127 0)
 			(effects
 				(font
@@
 		)
 		(property "Description" "Unpolarized capacitor"
-			(at 157.48 127 0)
+			(at 160.02 127 0)
 			(effects
 				(font
