File: R2_HH_Controllers/Navicore_Remote.kicad_sch (KiCad schematic)
At the start: 56 parts, among them IC1 E22-900M22S, J1 USB4105-GF-A, J2 S2B-PH-SM4-TB_LF__SN_, SW1 SW_Push, SW10 Boot, SW11 PCM12SMTR, SW2 SW_Push, SW3 SW_Push, SW4 SW_Push, SW5 SW_Push, SW6 SW_Push, SW7 SW_Push, SW8 SW_Push, SW9 Reset, U1 AP2112K-3.3, U2 ESP32-S3-MINI-1, U3 BQ24074RGT, U4 USBLC6-2SC6

Commit message: updates
Parts:
- removed C11, C13: 1uf, Capacitor_SMD:C_0603_1608Metric, symbol Device:C
- removed C15: .1uf, Capacitor_SMD:C_0603_1608Metric, symbol Device:C
- removed U1: AP2112K-3.3, Package_TO_SOT_SMD:SOT-23-5, symbol Regulator_Linear:AP2112K-3.3
- removed U2: ESP32-S3-MINI-1, 01-Custom:ESP32-S2-MINI-1, symbol RF_Module:ESP32-S3-MINI-1
- added C33: 220nf, Capacitor_SMD:C_0603_1608Metric, symbol Device:C
- added C37: 1uf, Capacitor_SMD:C_0805_2012Metric_Pad1.18x1.45mm_HandSolder, symbol Device:C
- added C40: 22uf, Capacitor_SMD:C_0603_1608Metric, symbol Device:C
- added C42: 10uf, Capacitor_SMD:C_0603_1608Metric, symbol Device:C
- added L1: .47uH, Inductor_SMD:L_0603_1608Metric, symbol Device:L
- added R28, R32: 470K, Resistor_SMD:R_0805_2012Metric_Pad1.20x1.40mm_HandSolder, symbol Device:R
- added R35, R41: 100K, Resistor_SMD:R_0603_1608Metric, symbol Device:R
- added R37: 511K, Resistor_SMD:R_0603_1608Metric, symbol Device:R
- added R39: 91K, Resistor_SMD:R_0603_1608Metric, symbol Device:R
- added U2: TPS63802DLAR, 01-Custom:VREG_TPS63802DLAR, symbol 01-Custom:TPS63802DLAR
- added U9: ESP32-S3-MINI-1-N8, 01-Custom:XCVR_ESP32-S3-MINI-1-N8, symbol 01-Custom:ESP32-S3-MINI-1-N8
- D1, D2, D3: footprint LED_SMD:LED_WS2812B-2020_PLCC4_2.0x2.0mm -> 01-Custom:LED_WS2812B-2020_PLCC4_2.0x2.0mm
- E1: footprint custom:XDCR_ANT-915-USP410 -> 01-Custom:XDCR_ANT-915-USP410
- IC1: footprint custom:E22-900M22S -> 01-Custom:E22-900M22S
- R13: value 10K -> 200K
- R9: value 17.8K -> 3K
- SW1, SW2, SW3, SW4, SW5, SW6, SW7, SW8: footprint 01-Custom:TL3360CF185Q -> 01-Custom:SW_TL3360AF185Q
Connections:
- net 3.3V_REG: now also C40.2, R37.2, R41.1, U2.6 (VOUT), U9.3 (3V3); no longer U3.6 (EN1)
- net BAT+_SWITCHED: now also R13.2, C42.2, U2.10 (VIN)
- net BOOT: now also U9.4 (IO0)
- net BTN_1: now also U9.31 (IO35)
- net BTN_2: now also U9.8 (IO4)
- net BTN_3: now also U9.9 (IO5)
- net BTN_4: now also U9.10 (IO6)
- net BTN_5: now also U9.21 (IO17)
- net BTN_6: now also U9.22 (IO18)
- net BTN_7: now also U9.25 (IO21)
- net BTN_8: now also U9.28 (IO33)
- net BUSY: now also U9.19 (IO15)
- net CHARGER_OUT: now also U3.5 (EN2)
- net D+_ESP: now also U9.24 (IO20)
- net D-_ESP: now also U9.23 (IO19)
- net DIO1: now also U9.20 (IO16)
- net EN: now also U9.45 (EN)
- net GND: now also U3.6 (EN1), C33.1, C37.1, C40.1, C42.1, R28.1, R35.1, R39.1, U2.2 (MODE), U2.3 (AGND), U2.8 (GND), U9.1 (GND), U9.2 (GND), U9.42 (GND), U9.43 (GND), U9.46 (GND), U9.47 (GND), U9.48 (GND), U9.49 (GND), U9.50 (GND), U9.51 (GND), U9.52 (GND), U9.53 (GND), U9.54 (GND), U9.55 (GND), U9.56 (GND), U9.57 (GND), U9.58 (GND), U9.59 (GND), U9.60 (GND), U9.61 (GND), U9.61_1 (GND), U9.61_2 (GND), U9.61_3 (GND), U9.61_4 (GND), U9.61_5 (GND), U9.61_6 (GND), U9.61_7 (GND), U9.61_8 (GND), U9.62 (GND), U9.63 (GND), U9.64 (GND), U9.65 (GND); no longer U3.5 (EN2)
- net JOY_SWITCH: now also U9.7 (IO3)
- net JOY_X: now also U9.5 (IO1)
- net JOY_Y: now also U9.6 (IO2)
- net JST_BAT+: now also R32.2; no longer R13.2
- net MISO: now also U9.17 (IO13)
- net MOSI: now also U9.15 (IO11)
- net NEOPIXEL: now also U9.12 (IO8)
- net NSS: now also U9.14 (IO10)
- net RST: now also U9.18 (IO14)
- net RX_EN: now also U9.29 (IO34)
- net SCK: now also U9.16 (IO12)
- net TX_EN: now also U9.34 (IO38)
- net VOL_POT: now also U9.11 (IO7)
- net at R14.2, U3.1 (TS): no longer R13.1
- net PWR_GOOD: now reaches U3.7 (~{PGOOD})
- net PWR_GOOD: now also U9.33 (IO37)
- net CHG_STAT: now reaches U3.9 (~{CHG})
- net CHG_STAT: now also U9.32 (IO36)
- new net: C33.2, R13.1, R35.2, U2.1 (EN)
- new net: R41.2, U2.5 (PG)
- new net: R37.1, R39.2, U2.4 (FB)
- new net: L1.1, U2.7 (L2)
- new net: L1.2, U2.9 (L1)
- new net VBAT_SENSE: C37.2, R28.2, R32.1, U9.13 (IO9)
- no-connect marks 5 -> 17
Other:
- moved on the sheet: D1, D2, D3, J2, R10, R11, R14, R3, R6, R7, R9, U3
