File: R2_HH_Controllers/R2_HH_Controllers.kicad_pcb (KiCad board)
At the start: 2 copper layers, 33.5 x 112.9 mm, 26 parts, among them IC1 E22-900M22S, J1 U.FL-R-SMT-1_10_, J2 USB4105-GF-A, J3 S2B-PH-SM4-TB_LF__SN_, SW1 SW_Push, SW10 SW_Push, SW11 SW_Push, SW2 Reset, SW3 Boot, SW4 SW_Push, SW5 PCM12SMTR, SW6 SW_Push, SW7 SW_Push, SW8 SW_Push, SW9 SW_Push, U1 ESP32-S3-WROOM-1, U2 USBLC6-2SC6, U3 BQ24074RGT

Commit message: hh
Parts:
- removed J1: U.FL-R-SMT-1_10_, custom:HRS_U.FL-R-SMT-1_10_
- removed SW11: SW_Push, 01-Custom:TL3360CF185Q
- removed U4: ~, 01-Custom:A24AH
- removed VR1: RKJXV1224005, 01-Custom:RKJXV1224005
- added C10: 22uf, Capacitor_SMD:C_0201_0603Metric, F.Cu at (189.8, 88.9)
- added C11: .1uf, Capacitor_SMD:C_0201_0603Metric, F.Cu at (189.9, 90.7)
- added C12: 100nf, Capacitor_SMD:C_0201_0603Metric, F.Cu at (189.9, 92.3)
- added C13: 100nf, Capacitor_SMD:C_0201_0603Metric, F.Cu at (189.9, 93.8)
- added C14: 100nf, Capacitor_SMD:C_0201_0603Metric, F.Cu at (189.9, 95.6)
- added C15: 100nf, Capacitor_SMD:C_0201_0603Metric, F.Cu at (189.9, 97.2)
- added C16: 100nf, Capacitor_SMD:C_0201_0603Metric, F.Cu at (190.0, 98.8)
- added C3: .1uf, Capacitor_SMD:C_0201_0603Metric, F.Cu at (207.3, 89.1)
- added C4: .1uf, Capacitor_SMD:C_0201_0603Metric, F.Cu at (189.9, 79.2)
- added C5: 1uf, Capacitor_SMD:C_0201_0603Metric, F.Cu at (190.0, 80.9)
- added C6: 10uf, Capacitor_SMD:C_0201_0603Metric, F.Cu at (190.0, 82.5)
- added C7: 1uf, Capacitor_SMD:C_0201_0603Metric, F.Cu at (189.8, 84.0)
- added C8: 1uf, Capacitor_SMD:C_0201_0603Metric, F.Cu at (189.9, 85.6)
- added C9: 1uf, Capacitor_SMD:C_0201_0603Metric, F.Cu at (189.8, 87.1)
- added R10: 17.8K, Resistor_SMD:R_0201_0603Metric, F.Cu at (207.4, 37.9)
- added R11: 10K, Resistor_SMD:R_0201_0603Metric, F.Cu at (207.4, 39.8)
- added R15: 330, Resistor_SMD:R_0201_0603Metric, F.Cu at (205.1, 100.6)
- added R3: 5.1K, Resistor_SMD:R_0201_0603Metric, F.Cu at (205.1, 30.8)
- added R4: 5.1K, Resistor_SMD:R_0201_0603Metric, F.Cu at (205.1, 32.5)
- added R5: 10K, Resistor_SMD:R_0201_0603Metric, F.Cu at (207.6, 30.5)
- added R6: 10K, Resistor_SMD:R_0201_0603Metric, F.Cu at (187.3, 95.7)
- added R7: 10K, Resistor_SMD:R_0201_0603Metric, F.Cu at (207.6, 32.5)
- added R8: 1.8K, Resistor_SMD:R_0201_0603Metric, F.Cu at (207.6, 34.5)
- added R9: 1.62K, Resistor_SMD:R_0201_0603Metric, F.Cu at (207.4, 36.1)
- added S1: RKJXV122400R, 01-Custom:RKJXV122400R, F.Cu at (203.6, 48.5)
- added SW12: Boot, Button_Switch_SMD:SW_SPST_TL3342, F.Cu at (184.1, 98.5)
- added U5: AP2112K-3.3, Package_TO_SOT_SMD:SOT-23-5, F.Cu at (204.1, 57.7)
- C1: value C -> 1uf
- C2: value C -> 22uf
- E1, IC1, SW6, SW7: moved to B.Cu
- R2: value R -> 10K
- SW10: value SW_Push -> Reset; footprint 01-Custom:TL3360CF185Q -> Button_Switch_SMD:SW_SPST_TL3342; moved to F.Cu
- SW2: value Reset -> SW_Push; footprint Button_Switch_SMD:SW_SPST_TL3342 -> 01-Custom:TL3360CF185Q
- SW3: value Boot -> SW_Push; footprint Button_Switch_SMD:SW_SPST_TL3342 -> 01-Custom:TL3360CF185Q
- SW5: value PCM12SMTR -> SW_Push; footprint 01-Custom:SW_PCM12SMTR -> 01-Custom:TL3360CF185Q; moved to B.Cu
- SW9: value SW_Push -> PCM12SMTR; footprint 01-Custom:TL3360CF185Q -> 01-Custom:SW_PCM12SMTR; moved to F.Cu
- moved SW5 75.9 mm to (179.7, 60.8), turned to -90 degrees
- moved U2 64.3 mm to (189.7, 65.8)
- moved SW9 46.2 mm to (203.8, 110.0), turned to 0 degrees
- moved SW2 42.5 mm to (179.7, 66.4), turned to 90 degrees
- moved SW3 41.9 mm to (179.7, 77.8), turned to 90 degrees
- moved SW8 37.5 mm to (179.7, 95.5)
- moved U1 34.4 mm to (196.7, 81.1)
- moved D1 33.9 mm to (200.8, 101.1)
- moved J2 26.7 mm to (193.8, 109.2)
- moved SW4 25.3 mm to (179.7, 89.5)
- moved J3 23.7 mm to (184.0, 31.7)
- moved SW10 21.0 mm to (184.1, 106.3), turned to 0 degrees
- moved R2 20.9 mm to (207.3, 86.1)
- moved C1 19.8 mm to (207.3, 84.6), turned to 180 degrees
- moved E1 19.6 mm to (201.8, 90.5), turned to 90 degrees
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Connections:
- C1 pad 1: unconnected-(C1-Pad1) -> GND
- C1 pad 2: unconnected-(C1-Pad2) -> Net-(U1-EN)
- C2 pad 1: Net-(C2-Pad1) -> GND
- C2 pad 2: unconnected-(C2-Pad2) -> 3.3V_REG
- D1 pad 2: unconnected-(D1-VSS-Pad2) -> GND
- D1 pad 3: unconnected-(D1-DIN-Pad3) -> Net-(D1-DIN)
- D1 pad 4: unconnected-(D1-VDD-Pad4) -> 3.3V_REG
- E1 pad 1: unconnected-(E1-Pad1) -> Net-(IC1-ANT)
- E1 pad 2: unconnected-(E1-Pad2) -> GND
- IC1 pad 14: unconnected-(IC1-BUSY-Pad14) -> BUSY
- IC1 pad 15: unconnected-(IC1-NRST-Pad15) -> RST
- IC1 pad 16: unconnected-(IC1-MISO-Pad16) -> MISO
- IC1 pad 17: unconnected-(IC1-MOSI-Pad17) -> MOSI
- IC1 pad 18: unconnected-(IC1-SCK-Pad18) -> SCK
- IC1 pad 19: unconnected-(IC1-NSS-Pad19) -> NSS
- IC1 pad 21: unconnected-(IC1-ANT-Pad21) -> Net-(IC1-ANT)
- IC1 pad 9: unconnected-(IC1-VCC-Pad9) -> 3.3V_REG
- J2 pad A4_B9: VBUS -> USB_VCC
- J2 pad A5: unconnected-(J2-CC1-PadA5) -> Net-(J2-CC1)
- J2 pad A6: unconnected-(J2-DP1-PadA6) -> D+
- J2 pad A7: unconnected-(J2-DN1-PadA7) -> D-
- J2 pad B4_A9: VBUS -> USB_VCC
- J2 pad B5: unconnected-(J2-CC2-PadB5) -> Net-(J2-CC2)
- J2 pad B6: unconnected-(J2-DP2-PadB6) -> D+
- J2 pad B7: unconnected-(J2-DN2-PadB7) -> D-
- J2 pad SH1: SHELL_GND -> GND
- J2 pad SH2: SHELL_GND -> GND
- J2 pad SH3: SHELL_GND -> GND
- J2 pad SH4: SHELL_GND -> GND
- J3 pad 1: unconnected-(J3-Pad1) -> JST_BAT+
- J3 pad 2: unconnected-(J3-Pad2) -> GND
- J3 pad S1: Net-(J3-SHIELD-PadS1) -> GND
- J3 pad S2: Net-(J3-SHIELD-PadS1) -> GND
- R1 pad 1: unconnected-(R1-Pad1) -> 3.3V_REG
- R1 pad 2: unconnected-(R1-Pad2) -> POT_1
- R1 pad 3: unconnected-(R1-Pad3) -> GND
- R2 pad 1: Net-(R2-Pad1) -> Net-(U1-EN)
- R2 pad 2: Net-(U1-IO0) -> 3.3V_REG
- SW1 pad 1: unconnected-(SW1-Pad1) -> BTN_1
- SW1 pad 2: unconnected-(SW1-Pad2) -> GND
- SW10 pad 1: unconnected-(SW10-Pad1) -> GND
- SW10 pad 2: unconnected-(SW10-Pad2) -> EN
- SW2 pad 1: Net-(C2-Pad1) -> BTN_2
- SW2 pad 2: Net-(R2-Pad1) -> GND
- SW3 pad 1: unconnected-(SW3-Pad1) -> BTN_3
- SW3 pad 2: unconnected-(SW3-Pad2) -> GND
- SW4 pad 1: unconnected-(SW4-Pad1) -> BTN_4
- SW4 pad 2: unconnected-(SW4-Pad2) -> GND
- SW5 pad 1: BAT+ -> BTN_5
- SW5 pad 2: BAT+_SWITCHED -> GND
- SW6 pad 1: unconnected-(SW6-Pad1) -> BTN_6
- SW6 pad 2: unconnected-(SW6-Pad2) -> GND
- SW7 pad 1: unconnected-(SW7-Pad1) -> BTN_7
- SW7 pad 2: unconnected-(SW7-Pad2) -> GND
- SW8 pad 1: unconnected-(SW8-Pad1) -> BTN_8
- SW8 pad 2: unconnected-(SW8-Pad2) -> GND
- SW9 pad 1: unconnected-(SW9-Pad1) -> CHARGER_OUT
- SW9 pad 2: unconnected-(SW9-Pad2) -> BAT+_SWITCHED
- U1 pad 1: Net-(U1-GND-Pad1) -> GND
- U1 pad 10: unconnected-(U1-IO17-Pad10) -> BTN_2
- U1 pad 11: unconnected-(U1-IO18-Pad11) -> BTN_3
- U1 pad 12: unconnected-(U1-IO8-Pad12) -> NEOPIXEL
- U1 pad 13: unconnected-(U1-USB_D--Pad13) -> D-_ESP
- U1 pad 14: unconnected-(U1-USB_D+-Pad14) -> D+_ESP
- U1 pad 15: unconnected-(U1-IO3-Pad15) -> JOY_SWITCH
- U1 pad 17: unconnected-(U1-IO9-Pad17) -> BTN_1
- U1 pad 18: unconnected-(U1-IO10-Pad18) -> NSS
- U1 pad 19: unconnected-(U1-IO11-Pad19) -> MOSI
- U1 pad 2: unconnected-(U1-3V3-Pad2) -> 3.3V_REG
- U1 pad 20: unconnected-(U1-IO12-Pad20) -> SCK
- U1 pad 21: unconnected-(U1-IO13-Pad21) -> MISO
- U1 pad 22: unconnected-(U1-IO14-Pad22) -> RST
- U1 pad 23: unconnected-(U1-IO21-Pad23) -> BTN_4
- U1 pad 27: Net-(U1-IO0) -> BOOT
- U1 pad 3: unconnected-(U1-EN-Pad3) -> Net-(U1-EN)
- U1 pad 31: unconnected-(U1-IO38-Pad31) -> BTN_5
- U1 pad 32: unconnected-(U1-IO39-Pad32) -> BTN_6
- U1 pad 33: unconnected-(U1-IO40-Pad33) -> BTN_7
- U1 pad 34: unconnected-(U1-IO41-Pad34) -> BTN_8
- U1 pad 38: unconnected-(U1-IO2-Pad38) -> JOY_Y
- U1 pad 39: unconnected-(U1-IO1-Pad39) -> JOY_X
- U1 pad 4: unconnected-(U1-IO4-Pad4) -> MODE_1
- U1 pad 40: Net-(U1-GND-Pad1) -> GND
- U1 pad 41: Net-(U1-GND-Pad1) -> GND
- U1 pad 5: unconnected-(U1-IO5-Pad5) -> MODE_2
- U1 pad 6: unconnected-(U1-IO6-Pad6) -> MODE_3
- U1 pad 7: unconnected-(U1-IO7-Pad7) -> VOL_POT
- U1 pad 8: unconnected-(U1-IO15-Pad8) -> BUSY
- U1 pad 9: unconnected-(U1-IO16-Pad9) -> DIO1
- U2 pad 1: unconnected-(U2-I/O1-Pad1) -> D+_ESP
- U2 pad 2: unconnected-(U2-GND-Pad2) -> GND
- U2 pad 3: unconnected-(U2-I/O2-Pad3) -> D-_ESP
- U2 pad 4: unconnected-(U2-I/O2-Pad4) -> D-
- U2 pad 5: unconnected-(U2-VBUS-Pad5) -> 3.3V_REG
- U2 pad 6: unconnected-(U2-I/O1-Pad6) -> D+
- U3 pad 1: unconnected-(U3-TS-Pad1) -> Net-(U3-TS)
- U3 pad 10: Net-(U3-OUT-Pad10) -> CHARGER_OUT
- U3 pad 11: Net-(U3-OUT-Pad10) -> CHARGER_OUT
- U3 pad 12: unconnected-(U3-ILIM-Pad12) -> Net-(U3-ILIM)
- U3 pad 13: unconnected-(U3-IN-Pad13) -> USB_VCC
- U3 pad 14: unconnected-(U3-TMR-Pad14) -> Net-(U3-TMR)
- U3 pad 15: unconnected-(U3-ITERM-Pad15) -> Net-(U3-ITERM)
- U3 pad 16: unconnected-(U3-ISET-Pad16) -> Net-(U3-ISET)
- U3 pad 17: Net-(U3-VSS-Pad17) -> GND
- U3 pad 2: Net-(U3-BAT-Pad2) -> JST_BAT+
- U3 pad 3: Net-(U3-BAT-Pad2) -> JST_BAT+
- U3 pad 4: unconnected-(U3-~{CE}-Pad4) -> GND
- U3 pad 5: unconnected-(U3-EN2-Pad5) -> GND
- U3 pad 6: unconnected-(U3-EN1-Pad6) -> 3.3V_REG
- U3 pad 8: Net-(U3-VSS-Pad17) -> GND
Other:
- board size 33.5 x 112.9 mm -> 29.3 x 82.4 mm
- copper layers 2 -> 4

Commit message: hh
Parts:
- added C17: 100nf, Capacitor_SMD:C_0603_1608Metric, F.Cu at (184.7, 31.1)
- added C18: 100nf, Capacitor_SMD:C_0603_1608Metric, F.Cu at (184.7, 32.8)
- added D2: WS2812B-2020, LED_SMD:LED_WS2812B-2020_PLCC4_2.0x2.0mm, F.Cu at (181.4, 31.9)
- added D3: WS2812B-2020, LED_SMD:LED_WS2812B-2020_PLCC4_2.0x2.0mm, F.Cu at (204.5, 32.0)
- added R12: 330, Resistor_SMD:R_0603_1608Metric, F.Cu at (207.9, 31.0)
- added R13: 330, Resistor_SMD:R_0603_1608Metric, F.Cu at (207.9, 32.8)
- C1, C12, C13, C14, C15, C16, C2, C3, C4, C5, C6, C7, C8, C9: footprint Capacitor_SMD:C_0201_0603Metric -> Capacitor_SMD:C_0603_1608Metric
- C10, C11: footprint Capacitor_SMD:C_0201_0603Metric -> Capacitor_SMD:C_0805_2012Metric_Pad1.18x1.45mm_HandSolder; moved to B.Cu
- R10, R11, R15, R2, R3, R4, R5, R6, R7, R8, R9: footprint Resistor_SMD:R_0201_0603Metric -> Resistor_SMD:R_0603_1608Metric
- moved R3 73.5 mm to (189.9, 102.8)
- moved R4 72.8 mm to (200.5, 105.1)
- moved C15 63.9 mm to (201.2, 34.3)
- moved C13 59.7 mm to (188.6, 34.1)
- moved C12 48.0 mm to (208.8, 48.2), turned to 90 degrees
- moved C14 45.4 mm to (208.8, 54.3), turned to 90 degrees
- moved R5 41.7 mm to (187.3, 66.9)
- moved R7 37.9 mm to (187.3, 64.6), turned to 180 degrees
- moved U2 36.6 mm to (197.8, 101.5), turned to 180 degrees
- moved R8 33.5 mm to (188.7, 62.2), turned to -90 degrees
- moved R9 32.7 mm to (195.0, 66.3), turned to 180 degrees
- moved R10 30.5 mm to (190.4, 63.2), turned to -90 degrees
- moved C9 28.8 mm to (198.0, 59.6)
- moved C8 26.4 mm to (194.2, 59.6)
- moved E1 26.0 mm to (203.9, 64.6)
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Connections:
- D1 pad 1: unconnected-(D1-DOUT-Pad1) -> Net-(D1-DOUT)
Routing:
- added copper zone on In1.Cu, net GND
Other:
- board size 29.3 x 82.4 mm -> 30.4 x 82.4 mm

Commit message: updates
Parts:
- removed U1: ESP32-S3-WROOM-1, RF_Module:ESP32-S3-WROOM-1
- added R14: DNP, Resistor_SMD:R_0805_2012Metric_Pad1.20x1.40mm_HandSolder, B.Cu at (190.5, 60.8)
- added U4: ESP32-S3-MINI-1, RF_Module:ESP32-S2-MINI-1, F.Cu at (199.4, 68.4)
- R1: moved to B.Cu
- moved R1 79.0 mm to (183.2, 107.3), turned to -90 degrees
- moved J3 74.3 mm to (203.9, 103.3), turned to 0 degrees
- moved E1 35.9 mm to (194.3, 29.9), turned to 180 degrees
- moved C3 32.9 mm to (190.5, 64.2), turned to -90 degrees
- moved C2 29.2 mm to (190.4, 67.2), turned to 90 degrees
- moved C11 26.9 mm to (206.8, 77.3), turned to -90 degrees
- moved C8 25.9 mm to (204.5, 83.4), turned to 180 degrees
- moved C10 25.8 mm to (206.8, 81.7), turned to 90 degrees
- moved R2 25.6 mm to (190.4, 70.5), turned to -90 degrees
- moved U5 24.7 mm to (203.2, 86.0), turned to 180 degrees
- moved C9 24.0 mm to (200.6, 83.4), turned to 180 degrees
- moved SW10 22.7 mm to (202.7, 96.2), turned to 0 degrees
- moved C1 22.6 mm to (190.3, 73.5), turned to 90 degrees
- moved C4 21.4 mm to (195.2, 83.4)
- moved C6 21.4 mm to (190.4, 90.2)
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Connections:
- E1 pad 1: Net-(IC1-ANT) -> Net-(E1-Pad1)
Other:
- board size 30.4 x 82.4 mm -> 26.5 x 87 mm

Commit message: sabe
Parts:
- moved J2 24.6 mm to (195.7, 133.7)
- moved R1 14.7 mm to (183.1, 122.0)
- moved D1 14.0 mm to (204.2, 118.7)
- moved R4 14.0 mm to (200.2, 119.2)
- moved SW9 14.0 mm to (203.4, 124.0)
- moved U2 14.0 mm to (197.5, 115.6)
- moved C16 14.0 mm to (204.3, 115.9)
- moved R15 14.0 mm to (206.5, 119.0)
- moved SW12 12.7 mm to (194.3, 108.7)
- moved SW10 12.7 mm to (203.6, 108.9)
- moved SW8 9.30 mm to (182.4, 102.3)
- moved SW4 8.73 mm to (182.3, 107.3)
- moved C5 8.54 mm to (197.6, 93.5)
- moved C6 8.54 mm to (191.1, 98.7)
- moved C8 8.54 mm to (205.2, 91.9)
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Other:
- board size 26.5 x 87 mm -> 26.5 x 111.3 mm
Changed lines of the file:
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@@
 	(footprint "Resistor_SMD:R_0603_1608Metric"
 		(layer "F.Cu")
-		(at 206.85 104.95 90)
+		(at 206.51 118.99 90)
 		(descr "Resistor SMD 0603 (1608 Metric), square (rectangular) end terminal, IPC-7351 nominal, (Body size source: IPC-SM-782 page 72, https://www.pcb-3d.com/wordpress/wp-content/uploads/ipc-sm-782a_amendment_1_and_2.pdf), generated with kicad-footprint-generator")
 		(tags "resistor")
@@
 	(footprint "Capacitor_SMD:C_0603_1608Metric"
 		(layer "F.Cu")
-		(at 204.62 101.87)
+		(at 204.28 115.91)
 		(descr "Capacitor SMD 0603 (1608 Metric), square (rectangular) end terminal, IPC-7351 nominal, (Body size source: IPC-SM-782 page 76, https://www.pcb-3d.com/wordpress/wp-content/uploads/ipc-sm-782a_amendment_1_and_2.pdf), generated with kicad-footprint-generator")
 		(tags "capacitor")
@@
 	(footprint "Capacitor_SMD:C_0603_1608Metric"
 		(layer "F.Cu")
-		(at 200.635 83.4275 180)
+		(at 201.315 91.94 180)
 		(descr "Capacitor SMD 0603 (1608 Metric), square (rectangular) end terminal, IPC-7351 nominal, (Body size source: IPC-SM-782 page 76, https://www.pcb-3d.com/wordpress/wp-content/uploads/ipc-sm-782a_amendment_1_and_2.pdf), generated with kicad-footprint-generator")
 		(tags "capacitor")
@@
 	(footprint "01-Custom:TL3360CF185Q"
 		(layer "F.Cu")
-		(at 182.59 98.616 90)
+		(at 182.35 107.34 90)
 		(property "Reference" "SW4"
 			(at 0 -3 90)
@@
 	(footprint "Button_Switch_SMD:SW_SPST_TL3342"
 		(layer "F.Cu")
-		(at 193.32 95.97 180)
+		(at 194.27 108.65 180)
 		(descr "Low-profile SMD Tactile Switch, https://www.e-switch.com/system/asset/product_line/data_sheet/165/TL3342.pdf")
 		(tags "SPST Tactile Switch")
@@
 	(footprint "01-Custom:GCT_USB4105-GF-A"
 		(layer "F.Cu")
-		(at 193.82 109.15)
+		(at 195.71 133.71)
 		(property "Reference" "J2"
 			(at -1.825 -8.635 0)
@@
 	(footprint "01-Custom:TL3360CF185Q"
 		(layer "F.Cu")
-		(at 182.59 75.523 90)
+		(at 182.2 83.06 90)
 		(property "Reference" "SW2"
 			(at 0 -3 90)
@@
 	(footprint "Capacitor_SMD:C_0603_1608Metric"
 		(layer "F.Cu")
-		(at 195.23 83.385 -90)
+		(at 195.91 91.8975 -90)
 		(descr "Capacitor SMD 0603 (1608 Metric), square (rectangular) end terminal, IPC-7351 nominal, (Body size source: IPC-SM-782 page 76, https://www.pcb-3d.com/wordpress/wp-content/uploads/ipc-sm-782a_amendment_1_and_2.pdf), generated with kicad-footprint-generator")
 		(tags "capacitor")
@@
 	(footprint "Package_TO_SOT_SMD:SOT-23-6"
 		(layer "F.Cu")
-		(at 197.83 101.52 180)
+		(at 197.49 115.56 180)
 		(descr "SOT, 6 Pin (JEDEC MO-178 Var AB https://www.jedec.org/document_search?search_api_views_fulltext=MO-178), generated with kicad-footprint-generator ipc_gullwing_generator.py")
 		(tags "SOT TO_SOT_SMD")
@@
 	(footprint "Capacitor_SMD:C_0603_1608Metric"
 		(layer "F.Cu")
-		(at 190.43 90.215)
+		(at 191.11 98.7275)
 		(descr "Capacitor SMD 0603 (1608 Metric), square (rectangular) end terminal, IPC-7351 nominal, (Body size source: IPC-SM-782 page 76, https://www.pcb-3d.com/wordpress/wp-content/uploads/ipc-sm-782a_amendment_1_and_2.pdf), generated with kicad-footprint-generator")
 		(tags "capacitor")
@@
 	(footprint "01-Custom:SW_PCM12SMTR"
 		(layer "F.Cu")
-		(at 203.79 109.99)
+		(at 203.45 124.03)
 		(property "Reference" "SW9"
 			(at -0.635 -4.699 0)
@@
 	(footprint "Capacitor_SMD:C_0603_1608Metric"
 		(layer "F.Cu")
-		(at 204.515 83.3875 180)
+		(at 205.195 91.9 180)
 		(descr "Capacitor SMD 0603 (1608 Metric), square (rectangular) end terminal, IPC-7351 nominal, (Body size source: IPC-SM-782 page 76, https://www.pcb-3d.com/wordpress/wp-content/uploads/ipc-sm-782a_amendment_1_and_2.pdf), generated with kicad-footprint-generator")
 		(tags "capacitor")
@@
 	(footprint "Resistor_SMD:R_0603_1608Metric"
 		(layer "F.Cu")
-		(at 193.56 84.405 -90)
+		(at 194.24 92.9175 -90)
 		(descr "Resistor SMD 0603 (1608 Metric), square (rectangular) end terminal, IPC-7351 nominal, (Body size source: IPC-SM-782 page 72, https://www.pcb-3d.com/wordpress/wp-content/uploads/ipc-sm-782a_amendment_1_and_2.pdf), generated with kicad-footprint-generator")
 		(tags "resistor")
@@
 	(footprint "Package_TO_SOT_SMD:SOT-23-5"
 		(layer "F.Cu")
-		(at 203.2125 86.0275 180)
+		(at 203.8925 94.54 180)
 		(descr "SOT, 5 Pin (JEDEC MO-178 Var AA https://www.jedec.org/document_search?search_api_views_fulltext=MO-178), generated with kicad-footprint-generator ipc_gullwing_generator.py")
 		(tags "SOT TO_SOT_SMD")
@@
 	(footprint "Resistor_SMD:R_0603_1608Metric"
 		(layer "F.Cu")
-		(at 190.46 88.025)
+		(at 191.14 96.5375)
 		(descr "Resistor SMD 0603 (1608 Metric), square (rectangular) end terminal, IPC-7351 nominal, (Body size source: IPC-SM-782 page 72, https://www.pcb-3d.com/wordpress/wp-content/uploads/ipc-sm-782a_amendment_1_and_2.pdf), generated with kicad-footprint-generator")
 		(tags "resistor")
@@
 	(footprint "LED_SMD:LED_WS2812B-2020_PLCC4_2.0x2.0mm"
 		(layer "F.Cu")
-		(at 204.5 104.66)
+		(at 204.16 118.7)
 		(descr "2.0mm x 2.0mm Addressable RGB LED NeoPixel Nano, 12 mA, https://cdn-shop.adafruit.com/product-files/4684/4684_WS2812B-2020_V1.3_EN.pdf")
 		(tags "LED RGB NeoPixel Nano PLCC-4 2020")
@@
 	(footprint "Button_Switch_SMD:SW_SPST_TL3342"
 		(layer "F.Cu")
-		(at 202.66 96.23)
+		(at 203.61 108.91)
 		(descr "Low-profile SMD Tactile Switch, https://www.e-switch.com/system/asset/product_line/data_sheet/165/TL3342.pdf")
 		(tags "SPST Tactile Switch")
@@
 	(footprint "Resistor_SMD:R_0603_1608Metric"
 		(layer "F.Cu")
-		(at 200.53 105.13)
+		(at 200.19 119.17)
 		(descr "Resistor SMD 0603 (1608 Metric), square (rectangular) end terminal, IPC-7351 nominal, (Body size source: IPC-SM-782 page 72, https://www.pcb-3d.com/wordpress/wp-content/uploads/ipc-sm-782a_amendment_1_and_2.pdf), generated with kicad-footprint-generator")
 		(tags "resistor")
@@
 	(footprint "Capacitor_SMD:C_0603_1608Metric"
 		(layer "F.Cu")
-		(at 196.9 84.975 -90)
+		(at 197.58 93.4875 -90)
 		(descr "Capacitor SMD 0603 (1608 Metric), square (rectangular) end terminal, IPC-7351 nominal, (Body size source: IPC-SM-782 page 76, https://www.pcb-3d.com/wordpress/wp-content/uploads/ipc-sm-782a_amendment_1_and_2.pdf), generated with kicad-footprint-generator")
 		(tags "capacitor")
@@
 	(footprint "Package_DFN_QFN:VQFN-16-1EP_3x3mm_P0.5mm_EP1.6x1.6mm"
 		(layer "F.Cu")
-		(at 194.39 88.2975)
+		(at 195.07 96.81)
 		(descr "VQFN, 16 Pin (http://www.ti.com/lit/ds/symlink/cdclvp1102.pdf#page=28), generated with kicad-footprint-generator ipc_noLead_generator.py")
 		(tags "VQFN NoLead")
@@
 	(footprint "01-Custom:TL3360CF185Q"
 		(layer "F.Cu")
-		(at 182.59 86.933 90)
+		(at 182.42 95.27 90)
 		(property "Reference" "SW3"
 			(at 0 -3 90)
@@
 	(footprint "Capacitor_SMD:C_0603_1608Metric"
 		(layer "F.Cu")
-		(at 198.3 89.575 180)
+		(at 198.98 98.0875 180)
 		(descr "Capacitor SMD 0603 (1608 Metric), square (rectangular) end terminal, IPC-7351 nominal, (Body size source: IPC-SM-782 page 76, https://www.pcb-3d.com/wordpress/wp-content/uploads/ipc-sm-782a_amendment_1_and_2.pdf), generated with kicad-footprint-generator")
 		(tags "capacitor")
@@
 	(footprint "Resistor_SMD:R_0603_1608Metric"
 		(layer "F.Cu")
-		(at 198.11 87.475 180)
+		(at 198.79 95.9875 180)
 		(descr "Resistor SMD 0603 (1608 Metric), square (rectangular) end terminal, IPC-7351 nominal, (Body size source: IPC-SM-782 page 72, https://www.pcb-3d.com/wordpress/wp-content/uploads/ipc-sm-782a_amendment_1_and_2.pdf), generated with kicad-footprint-generator")
 		(tags "resistor")
@@
 	(footprint "Resistor_SMD:R_0603_1608Metric"
 		(layer "F.Cu")
-		(at 191.88 83.395 -90)
+		(at 192.56 91.9075 -90)
 		(descr "Resistor SMD 0603 (1608 Metric), square (rectangular) end terminal, IPC-7351 nominal, (Body size source: IPC-SM-782 page 72, https://www.pcb-3d.com/wordpress/wp-content/uploads/ipc-sm-782a_amendment_1_and_2.pdf), generated with kicad-footprint-generator")
 		(tags "resistor")
@@
 	(footprint "Resistor_SMD:R_0603_1608Metric"
 		(layer "F.Cu")
-		(at 190.43 85.745 180)
+		(at 191.11 94.2575 180)
 		(descr "Resistor SMD 0603 (1608 Metric), square (rectangular) end terminal, IPC-7351 nominal, (Body size source: IPC-SM-782 page 72, https://www.pcb-3d.com/wordpress/wp-content/uploads/ipc-sm-782a_amendment_1_and_2.pdf), generated with kicad-footprint-generator")
 		(tags "resistor")
@@
 	(footprint "01-Custom:TL3360CF185Q"
 		(layer "F.Cu")
-		(at 182.59 63.963 90)
+		(at 182.2 69.13 90)
 		(property "Reference" "SW1"
 			(at 0 -10.86625 270)
@@
 	(footprint "01-Custom:TL3360CF185Q"
 		(layer "B.Cu")
-		(at 182.15 69.66 -90)
+		(at 182.13 76.43 -90)
 		(property "Reference" "SW6"
 			(at 0 3 90)
@@
 	(footprint "01-Custom:TL3360CF185Q"
 		(layer "B.Cu")
-		(at 182.15 92.98 -90)
+		(at 182.42 102.28 -90)
 		(property "Reference" "SW8"
 			(at 0 3 90)
@@
 	(footprint "01-Custom:TL3360CF185Q"
 		(layer "B.Cu")
-		(at 182.15 58.32 -90)
+		(at 182.3 64.86 -90)
 		(property "Reference" "SW5"
 			(at 0 3 90)
@@
 	(footprint "01-Custom:TL3360CF185Q"
 		(layer "B.Cu")
-		(at 182.15 81.12 -90)
+		(at 182.2 89.02 -90)
 		(property "Reference" "SW7"
 			(at -0.64 -0.7 270)
@@
 	(footprint "01-Custom:TRIM_3352T-1-103LF"
 		(layer "B.Cu")
-		(at 183.18 107.32 -90)
+		(at 183.12 122.02 -90)
 		(property "Reference" "R1"
 			(at -0.625 5.435 90)
@@
 	(gr_rect
 		(start 181.735 24.95)
-		(end 208.245 111.93)
+		(end 208.245 136.25)
 		(stroke
 			(width 0.05)
@@
 		(min_thickness 0.25)
 		(filled_areas_thickness no)
-		(fill yes
+		(fill
 			(thermal_gap 0.5)
 			(thermal_bridge_width 0.5)
@@
 		(polygon
 			(pts
-				(xy 176.88 24.42) (xy 176.7 24.24) (xy 210.89 24.05) (xy 209.6 125.34) (xy 174.49 125.16)
+				(xy 176.88 24.42) (xy 176.7 24.24) (xy 210.89 24.05) (xy 209.05 137.36) (xy 177.98 137.74)
 			)
 		)
