File: R2_HH_Controllers/R2_HH_Controllers.kicad_pcb (KiCad board)
At the start: 4 copper layers, 26.5 x 111.3 mm, 56 parts, among them IC1 E22-900M22S, J2 USB4105-GF-A, J3 S2B-PH-SM4-TB_LF__SN_, SW1 SW_Push, SW10 Reset, SW12 Boot, SW2 SW_Push, SW3 SW_Push, SW4 SW_Push, SW5 SW_Push, SW6 SW_Push, SW7 SW_Push, SW8 SW_Push, SW9 PCM12SMTR, U2 USBLC6-2SC6, U3 BQ24074RGT, U4 ESP32-S3-MINI-1, U5 AP2112K-3.3

Commit message: updates
Parts:
- added C19: 100nf, Capacitor_SMD:C_0603_1608Metric, F.Cu at (129.9, 76.5)
- added C20: 22uf, Capacitor_SMD:C_0805_2012Metric_Pad1.18x1.45mm_HandSolder, F.Cu at (145.5, 96.0)
- added C21: 100nf, Capacitor_SMD:C_0603_1608Metric, F.Cu at (129.9, 79.0)
- added C22: .1uf, Capacitor_SMD:C_0805_2012Metric_Pad1.18x1.45mm_HandSolder, F.Cu at (145.5, 99.0)
- added C23: 100nf, Capacitor_SMD:C_0603_1608Metric, F.Cu at (139.8, 69.8)
- added C24: 100nf, Capacitor_SMD:C_0603_1608Metric, F.Cu at (159.1, 87.6)
- added C25: 100nf, Capacitor_SMD:C_0603_1608Metric, F.Cu at (129.9, 86.5)
- added C26: 22uf, Capacitor_SMD:C_0603_1608Metric, F.Cu at (129.9, 89.0)
- added C27: .1uf, Capacitor_SMD:C_0603_1608Metric, F.Cu at (129.9, 91.5)
- added C28: 1uf, Capacitor_SMD:C_0603_1608Metric, B.Cu at (153.8, 78.1)
- added C29: 1uf, Capacitor_SMD:C_0603_1608Metric, B.Cu at (153.9, 74.5)
- added C30: 100nf, Capacitor_SMD:C_0603_1608Metric, F.Cu at (133.9, 79.0)
- added C31: 1uf, Capacitor_SMD:C_0603_1608Metric, F.Cu at (133.9, 81.5)
- added C32: 100nf, Capacitor_SMD:C_0603_1608Metric, F.Cu at (133.9, 84.0)
- added C33: .1uf, Capacitor_SMD:C_0603_1608Metric, F.Cu at (133.9, 86.5)
- added C34: 1uf, Capacitor_SMD:C_0603_1608Metric, F.Cu at (133.9, 89.0)
- added C35: 1uf, Capacitor_SMD:C_0603_1608Metric, F.Cu at (133.9, 91.5)
- added C36: 10uf, Capacitor_SMD:C_0603_1608Metric, F.Cu at (133.9, 94.0)
- added D4: WS2812B-2020, LED_SMD:LED_WS2812B-2020_PLCC4_2.0x2.0mm, F.Cu at (168.5, 124.7)
- added D5: WS2812B-2020, LED_SMD:LED_WS2812B-2020_PLCC4_2.0x2.0mm, F.Cu at (155.6, 29.7)
- added D6: WS2812B-2020, LED_SMD:LED_WS2812B-2020_PLCC4_2.0x2.0mm, F.Cu at (175.9, 29.1)
- added E2: ANT-915-USP410, custom:XDCR_ANT-915-USP410, B.Cu at (166.4, 29.8)
- added IC2: E22-900M22S, custom:E22-900M22S, B.Cu at (163.3, 73.4)
- added J1: USB4105-GF-A, 01-Custom:GCT_USB4105-GF-A, F.Cu at (193.8, 133.9)
- added J4: S2B-PH-SM4-TB_LF__SN_, 01-Custom:JST_S2B-PH-SM4-TB_LF__SN_, B.Cu at (159.9, 122.0)
- added R16: DNP, Resistor_SMD:R_0805_2012Metric_Pad1.20x1.40mm_HandSolder, B.Cu at (156.3, 60.4)
- added R17: 10K, Resistor_SMD:R_0603_1608Metric, F.Cu at (137.9, 76.5)
- added R18: 330, Resistor_SMD:R_0603_1608Metric, F.Cu at (137.9, 79.0)
- added R19: 10K, Resistor_SMD:R_0603_1608Metric, F.Cu at (137.9, 81.5)
- added R20: 3352T-1-103LF, 01-Custom:TRIM_3352T-1-103LF, F.Cu at (152.6, 88.7)
- added R21: 330, Resistor_SMD:R_0603_1608Metric, F.Cu at (137.9, 84.0)
- added R22: 330, Resistor_SMD:R_0603_1608Metric, F.Cu at (137.9, 86.5)
- added R23: 10K, Resistor_SMD:R_0603_1608Metric, F.Cu at (137.9, 89.0)
- added R24: 17.8K, Resistor_SMD:R_0603_1608Metric, F.Cu at (137.9, 91.5)
- added R25: 1.62K, Resistor_SMD:R_0603_1608Metric, F.Cu at (137.9, 94.0)
- added R26: 1.8K, Resistor_SMD:R_0603_1608Metric, F.Cu at (141.9, 76.5)
- added R27: 5.1K, Resistor_SMD:R_0603_1608Metric, F.Cu at (141.9, 79.0)
- added R28: 10K, Resistor_SMD:R_0603_1608Metric, F.Cu at (141.9, 81.5)
- added R29: 10K, Resistor_SMD:R_0603_1608Metric, B.Cu at (159.5, 60.0)
- added R30: 5.1K, Resistor_SMD:R_0603_1608Metric, F.Cu at (141.9, 86.5)
- added S2: RKJXV122400R, 01-Custom:RKJXV122400R, F.Cu at (173.6, 48.1)
- added SW11: PCM12SMTR, 01-Custom:SW_PCM12SMTR, F.Cu at (206.0, 130.3)
- added SW13: SW_Push, 01-Custom:TL3360CF185Q, F.Cu at (178.7, 87.2)
- added SW14: SW_Push, 01-Custom:TL3360CF185Q, F.Cu at (178.5, 107.5)
- added SW15: SW_Push, 01-Custom:TL3360CF185Q, F.Cu at (178.7, 127.8)
- added SW16: SW_Push, 01-Custom:TL3360CF185Q, B.Cu at (178.5, 58.0)
- added SW17: SW_Push, 01-Custom:TL3360CF185Q, B.Cu at (178.9, 77.6)
- added SW18: SW_Push, 01-Custom:TL3360CF185Q, B.Cu at (178.4, 100.0)
- added SW19: SW_Push, 01-Custom:TL3360CF185Q, B.Cu at (178.8, 119.3)
- added SW20: Reset, Button_Switch_SMD:SW_SPST_TL3342, F.Cu at (166.6, 117.7)
- added SW21: Boot, Button_Switch_SMD:SW_SPST_TL3342, F.Cu at (157.5, 117.7)
- added SW22: PCM12SMTR, 01-Custom:SW_PCM12SMTR, F.Cu at (154.7, 130.4)
- added U1: AP2112K-3.3, Package_TO_SOT_SMD:SOT-23-5, F.Cu at (156.4, 99.0)
- added U6: ESP32-S3-MINI-1, 01-Custom:ESP32-S2-MINI-1, F.Cu at (162.7, 71.4)
- added U7: BQ24074RGT, Package_DFN_QFN:VQFN-16-1EP_3x3mm_P0.5mm_EP1.6x1.6mm, F.Cu at (164.2, 97.2)
- added U8: USBLC6-2SC6, Package_TO_SOT_SMD:SOT-23-6, F.Cu at (164.9, 107.0)
- added mouse-bite-2.54mm-slot: VAL**, 01-Custom:mouse-bite-2.54mm-slot, F.Cu at (180.4, 119.4)
- added mouse-bite-2.54mm-slot: VAL**, 01-Custom:mouse-bite-2.54mm-slot, F.Cu at (180.4, 99.2)
- added mouse-bite-2.54mm-slot: VAL**, 01-Custom:mouse-bite-2.54mm-slot, F.Cu at (180.4, 58.5)
- added mouse-bite-2.54mm-slot: VAL**, 01-Custom:mouse-bite-2.54mm-slot, F.Cu at (180.4, 107.6)
- added mouse-bite-2.54mm-slot: VAL**, 01-Custom:mouse-bite-2.54mm-slot, F.Cu at (180.4, 42.5)
- added mouse-bite-2.54mm-slot: VAL**, 01-Custom:mouse-bite-2.54mm-slot, F.Cu at (180.4, 87.2)
- added mouse-bite-2.54mm-slot: VAL**, 01-Custom:mouse-bite-2.54mm-slot, F.Cu at (180.4, 77.6)
- added mouse-bite-2.54mm-slot: VAL**, 01-Custom:mouse-bite-2.54mm-slot, F.Cu at (180.4, 128.2)
- added mouse-bite-2.54mm-slot: VAL**, 01-Custom:mouse-bite-2.54mm-slot, F.Cu at (180.4, 66.7)
- added mouse-bite-2.54mm-slot: VAL**, 01-Custom:mouse-bite-2.54mm-slot, F.Cu at (180.4, 29.6)
- C1, C5, C7: value 1uf -> 100nf
- C10: value 22uf -> 1uf; footprint Capacitor_SMD:C_0805_2012Metric_Pad1.18x1.45mm_HandSolder -> Capacitor_SMD:C_0603_1608Metric
- C11: value .1uf -> 1uf; footprint Capacitor_SMD:C_0805_2012Metric_Pad1.18x1.45mm_HandSolder -> Capacitor_SMD:C_0603_1608Metric
- C13, C16, C17: value 100nf -> 1uf
- C15: value 100nf -> .1uf
- C18: value 100nf -> 10uf
- C2, C4: footprint Capacitor_SMD:C_0603_1608Metric -> Capacitor_SMD:C_0805_2012Metric_Pad1.18x1.45mm_HandSolder
- C3: value .1uf -> 100nf
- C6: value 10uf -> 100nf
- C8: value 1uf -> 22uf
- C9: value 1uf -> .1uf
- J2: value USB4105-GF-A -> S2B-PH-SM4-TB_LF__SN_; footprint 01-Custom:GCT_USB4105-GF-A -> 01-Custom:JST_S2B-PH-SM4-TB_LF__SN_; moved to B.Cu
- J3: value S2B-PH-SM4-TB_LF__SN_ -> USB4105-GF-A; footprint 01-Custom:JST_S2B-PH-SM4-TB_LF__SN_ -> 01-Custom:GCT_USB4105-GF-A; moved to F.Cu
- R1: value 3352T-1-103LF -> DNP; footprint 01-Custom:TRIM_3352T-1-103LF -> Resistor_SMD:R_0805_2012Metric_Pad1.20x1.40mm_HandSolder
- R10: value 17.8K -> 1.62K
- R11: value 10K -> 1.8K
- R12, R15: value 330 -> 5.1K
- R13: value 330 -> 10K
- R14: value DNP -> 10K; footprint Resistor_SMD:R_0805_2012Metric_Pad1.20x1.40mm_HandSolder -> Resistor_SMD:R_0603_1608Metric
- R3: value 5.1K -> 330
- R4: value 5.1K -> 10K
- R5: value 10K -> 3352T-1-103LF; footprint Resistor_SMD:R_0603_1608Metric -> 01-Custom:TRIM_3352T-1-103LF
- R6, R7: value 10K -> 330
- R8: value 1.8K -> 10K
- R9: value 1.62K -> 17.8K
- SW10: value Reset -> Boot
- SW12: value Boot -> SW_Push; footprint Button_Switch_SMD:SW_SPST_TL3342 -> 01-Custom:TL3360CF185Q
- SW9: value PCM12SMTR -> Reset; footprint 01-Custom:SW_PCM12SMTR -> Button_Switch_SMD:SW_SPST_TL3342
- U2: value USBLC6-2SC6 -> ESP32-S3-MINI-1; footprint Package_TO_SOT_SMD:SOT-23-6 -> 01-Custom:ESP32-S2-MINI-1
- U4: value ESP32-S3-MINI-1 -> USBLC6-2SC6; footprint RF_Module:ESP32-S2-MINI-1 -> Package_TO_SOT_SMD:SOT-23-6
- moved R1 65.1 mm to (202.1, 59.7)
- moved J3 47.7 mm to (166.8, 133.2)
- moved SW12 44.7 mm to (178.7, 66.8), turned to -90 degrees
- moved U2 44.3 mm to (196.8, 71.3)
- moved U4 38.9 mm to (194.2, 106.9)
- moved C1 34.9 mm to (217.9, 94.9)
- moved C3 34.9 mm to (218.1, 85.6)
- moved C2 34.9 mm to (218.0, 88.6)
- moved R2 34.9 mm to (218.0, 91.9)
- moved C8 21.5 mm to (205.5, 70.4), turned to -90 degrees
- moved SW4 20.4 mm to (182.3, 127.7)
- moved C9 18.3 mm to (205.4, 74.2), turned to -90 degrees
- moved R5 18.1 mm to (207.6, 89.1), turned to -90 degrees
- moved SW8 17.0 mm to (182.2, 119.3)
- moved J2 15.2 mm to (202.9, 120.3)
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Connections:
- C1 pad 2: Net-(U4-EN) -> JOY_X
- C10 pad 2: 3.3V_REG -> Net-(U2-EN)
- C11 pad 2: 3.3V_REG -> BAT+_SWITCHED
- C12 pad 2: JOY_X -> 3.3V_REG
- C13 pad 2: JOY_Y -> 3.3V_REG
- C14 pad 2: JOY_SWITCH -> 3.3V_REG
- C15 pad 2: POT_1 -> Net-(U3-TMR)
- C16 pad 2: 3.3V_REG -> USB_VCC
- C17 pad 2: 3.3V_REG -> CHARGER_OUT
- C18 pad 2: 3.3V_REG -> JST_BAT+
- C3 pad 2: 3.3V_REG -> JOY_Y
- C4 pad 2: Net-(U3-TMR) -> 3.3V_REG
- C5 pad 2: USB_VCC -> JOY_SWITCH
- C6 pad 2: JST_BAT+ -> POT_1
- C7 pad 2: CHARGER_OUT -> 3.3V_REG
- C8 pad 2: BAT+_SWITCHED -> 3.3V_REG
- R1 pad 1: 3.3V_REG -> Net-(E1-Pad1)
- R1 pad 2: POT_1 -> Net-(IC1-ANT)
- R10 pad 2: Net-(U3-ITERM) -> Net-(U3-ILIM)
- R11 pad 1: JOY_SWITCH -> GND
- R11 pad 2: 3.3V_REG -> Net-(U3-ISET)
- R12 pad 1: Net-(D2-DIN) -> Net-(J1-CC1)
- R12 pad 2: Net-(D1-DOUT) -> GND
- R13 pad 1: Net-(D3-DIN) -> Net-(U3-TS)
- R13 pad 2: Net-(D2-DOUT) -> JST_BAT+
- R14 pad 1: Net-(E1-Pad1) -> GND
- R14 pad 2: Net-(IC1-ANT) -> Net-(U3-TS)
- R15 pad 1: Net-(D1-DIN) -> GND
- R15 pad 2: NEOPIXEL -> Net-(J1-CC2)
- R2 pad 1: Net-(U4-EN) -> JOY_SWITCH
- R3 pad 1: Net-(J2-CC1) -> Net-(D1-DIN)
- R3 pad 2: GND -> NEOPIXEL
- R4 pad 1: GND -> BOOT
- R4 pad 2: Net-(J2-CC2) -> 3.3V_REG
- R5 pad 1: Net-(U3-TS) -> 3.3V_REG
- R5 pad 2: JST_BAT+ -> POT_1
- R6 pad 1: BOOT -> Net-(D2-DIN)
- R6 pad 2: 3.3V_REG -> Net-(D1-DOUT)
- R7 pad 1: GND -> Net-(D3-DIN)
- R7 pad 2: Net-(U3-TS) -> Net-(D2-DOUT)
- R8 pad 1: GND -> Net-(U2-EN)
- R8 pad 2: Net-(U3-ISET) -> 3.3V_REG
- R9 pad 2: Net-(U3-ILIM) -> Net-(U3-ITERM)
- SW10 pad 1: GND -> BOOT
- SW10 pad 2: EN -> GND
- SW12 pad 1: BOOT -> BTN_1
- SW9 pad 1: CHARGER_OUT -> GND
- SW9 pad 2: BAT+_SWITCHED -> EN
- U2 pad 1: D+_ESP -> Net-(U2-GND-Pad1)
- U2 pad 2: GND -> Net-(U2-GND-Pad1)
- U2 pad 3: D-_ESP -> 3.3V_REG
- U2 pad 4: D- -> BOOT
- U2 pad 5: 3.3V_REG -> JOY_X
- U2 pad 6: D+ -> JOY_Y
- U4 pad 1: Net-(U4-GND-Pad1) -> D+_ESP
- U4 pad 2: Net-(U4-GND-Pad1) -> GND
- U4 pad 3: 3.3V_REG -> D-_ESP
- U4 pad 4: BOOT -> D-
- U4 pad 5: JOY_X -> 3.3V_REG
- U4 pad 6: JOY_Y -> D+
Other:
- board size 26.5 x 111.3 mm -> 55.6 x 111.3 mm

Commit message: updates
Parts:
- C10, C11, R14, R29: moved to F.Cu
- C2, C20, C22, C4: moved to B.Cu
- moved R12 120.3 mm to (132.5, 126.8), turned to 180 degrees
- moved R13 96.8 mm to (132.3, 97.1), turned to 180 degrees
- moved R11 89.0 mm to (133.5, 94.1), turned to -90 degrees
- moved C15 88.5 mm to (137.3, 92.3), turned to -90 degrees
- moved C13 88.2 mm to (140.1, 106.9), turned to 90 degrees
- moved C3 87.2 mm to (144.9, 38.2), turned to 180 degrees
- moved R6 86.7 mm to (126.4, 32.4), turned to 90 degrees
- moved C18 86.1 mm to (129.8, 97.9), turned to 90 degrees
- moved C1 85.6 mm to (147.0, 46.9)
- moved C17 82.0 mm to (141.5, 98.1), turned to 180 degrees
- moved R2 80.2 mm to (146.7, 55.0)
- moved C12 79.9 mm to (128.1, 32.4)
- moved C10 77.6 mm to (129.4, 76.6)
- moved R7 77.5 mm to (144.4, 32.4), turned to -90 degrees
- moved R14 77.3 mm to (132.3, 98.8)
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Routing:
- removed copper zone on In1.Cu, net GND
Other:
- board size 55.6 x 111.3 mm -> 56.5 x 111 mm
