File: R2_HH_Controllers/R2_HH_Controllers.kicad_pcb (KiCad board)
At the start: 4 copper layers, 56.5 x 111 mm, 122 parts, among them IC1 E22-900M22S, IC2 E22-900M22S, J1 USB4105-GF-A, J2 S2B-PH-SM4-TB_LF__SN_, J3 USB4105-GF-A, J4 S2B-PH-SM4-TB_LF__SN_, SW1 SW_Push, SW10 Boot, SW11 PCM12SMTR, SW12 SW_Push, SW13 SW_Push, SW14 SW_Push, SW15 SW_Push, SW16 SW_Push, SW17 SW_Push, SW18 SW_Push, SW19 SW_Push, SW2 SW_Push, SW20 Reset, SW21 Boot, SW22 PCM12SMTR, SW3 SW_Push, SW4 SW_Push, SW5 SW_Push, SW6 SW_Push, SW7 SW_Push, SW8 SW_Push, SW9 Reset, U1 AP2112K-3.3, U2 ESP32-S3-MINI-1, U3 BQ24074RGT, U4 USBLC6-2SC6, U5 AP2112K-3.3, U6 ESP32-S3-MINI-1, U7 BQ24074RGT, U8 USBLC6-2SC6

Commit message: updates
Parts:
- C28, C29: moved to F.Cu
- moved U4 32.2 mm to (168.2, 125.2), turned to 90 degrees
- moved U8 31.7 mm to (135.4, 125.3), turned to -90 degrees
- moved C29 29.1 mm to (160.0, 102.9)
- moved R23 21.6 mm to (156.3, 73.3), turned to 90 degrees
- moved R19 15.9 mm to (171.8, 108.8)
- moved SW21 10.2 mm to (168.5, 113.1)
- moved SW20 9.34 mm to (159.2, 113.1)
- moved D4 7.34 mm to (157.5, 128.9)
- moved D1 6.50 mm to (144.8, 128.8)
- moved C27 4.98 mm to (175.7, 73.5), turned to 180 degrees
- moved C13 4.63 mm to (139.1, 102.4), turned to -90 degrees
- moved C11 4.53 mm to (146.3, 102.4), turned to -90 degrees
- moved R8 4.45 mm to (128.4, 75.8), turned to 180 degrees
- moved C26 4.41 mm to (175.7, 75.3), turned to 180 degrees
- moved U1 3.75 mm to (163.7, 103.3)
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Other:
- board text added: "BOOT"
- board text added: "RESET"

Commit message: update
Parts:
- removed mouse-bite-2.54mm-slot (x10): VAL**, 01-Custom:mouse-bite-2.54mm-slot
- added U10: ~, 01-Custom:mouse-bite-2.54mm-slot, F.Cu at (151.7, 66.4)
- added U12: ~, 01-Custom:mouse-bite-2.54mm-slot, F.Cu at (151.7, 119.2)
- added U14: ~, 01-Custom:mouse-bite-2.54mm-slot, F.Cu at (151.7, 77.8)
- added U16: ~, 01-Custom:mouse-bite-2.54mm-slot, F.Cu at (151.7, 128.0)
- added U18: ~, 01-Custom:mouse-bite-2.54mm-slot, F.Cu at (151.7, 42.2)
- added U20: ~, 01-Custom:mouse-bite-2.54mm-slot, F.Cu at (151.7, 99.4)
- added U22: ~, 01-Custom:mouse-bite-2.54mm-slot, F.Cu at (151.7, 29.3)
- added U24: ~, 01-Custom:mouse-bite-2.54mm-slot, F.Cu at (151.7, 88.4)
- added U26: ~, 01-Custom:mouse-bite-2.54mm-slot, F.Cu at (151.7, 57.1)
- added U28: ~, 01-Custom:mouse-bite-2.54mm-slot, F.Cu at (151.7, 109.8)
- moved U4 32.9 mm to (135.3, 124.8), turned to -90 degrees
- moved U8 32.5 mm to (167.9, 124.8)
- moved U1 27.5 mm to (136.2, 103.0)
- moved U5 21.4 mm to (164.4, 103.0), turned to 0 degrees
- moved C11 13.9 mm to (132.5, 103.0)
- moved R4 2.14 mm to (145.0, 106.7), turned to 0 degrees
- moved R14 1.88 mm to (132.5, 97.0)
- moved R6 1.83 mm to (128.2, 32.4), turned to -90 degrees
- moved C12 1.80 mm to (126.3, 32.4)
- moved R28 1.76 mm to (159.7, 98.0), turned to 180 degrees
- moved C4 1.66 mm to (143.0, 60.1)
- moved R29 1.66 mm to (159.7, 96.3)
- moved R13 1.45 mm to (132.5, 98.6)
- moved C13 1.43 mm to (140.4, 103.0), turned to 90 degrees
- moved R16 1.24 mm to (161.4, 59.6), turned to 180 degrees
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Connections:
- net Net-(D1-DOUT) renamed /Remote_Right_Hand/D1-D2
- net Net-(D2-DOUT) renamed /Remote_Right_Hand/D2-D3
- net Net-(D4-DOUT) renamed /Remote_Left_Hand/D1-D2
- net Net-(D5-DOUT) renamed /Remote_Left_Hand/D2-D3
- net USB_VCC renamed VBUS
- C1 pad 2: JOY_X -> /Remote_Right_Hand/JOY_X
- C10 pad 2: Net-(U2-EN) -> /Remote_Right_Hand/EN
- C11 pad 2: BAT+_SWITCHED -> /Remote_Right_Hand/BAT+_SWITCHED
- C12 pad 2: 3.3V_REG -> /Remote_Right_Hand/3.3V_REG
- C13 pad 2: 3.3V_REG -> /Remote_Right_Hand/3.3V_REG
- C14 pad 2: 3.3V_REG -> /Remote_Right_Hand/3.3V_REG
- C17 pad 2: CHARGER_OUT -> /Remote_Right_Hand/CHARGER_OUT
- C18 pad 1: GND -> /Remote_Right_Hand/JST_BAT+
- C18 pad 2: JST_BAT+ -> GND
- C19 pad 2: JOY_X -> /Remote_Left_Hand/JOY_X
- C2 pad 2: 3.3V_REG -> /Remote_Right_Hand/3.3V_REG
- C20 pad 2: 3.3V_REG -> /Remote_Left_Hand/3.3V_REG
- C21 pad 2: JOY_Y -> /Remote_Left_Hand/JOY_Y
- C22 pad 2: 3.3V_REG -> /Remote_Left_Hand/3.3V_REG
- C23 pad 2: JOY_SWITCH -> /Remote_Left_Hand/JOY_SWITCH
- C24 pad 2: POT_1 -> /Remote_Left_Hand/VOL_POT
- C25 pad 2: 3.3V_REG -> /Remote_Left_Hand/3.3V_REG
- C26 pad 2: 3.3V_REG -> /Remote_Left_Hand/3.3V_REG
- C27 pad 2: 3.3V_REG -> /Remote_Left_Hand/3.3V_REG
- C28 pad 2: Net-(U6-EN) -> /Remote_Left_Hand/EN
- C29 pad 2: BAT+_SWITCHED -> /Remote_Left_Hand/BAT+_SWITCHED
- C3 pad 2: JOY_Y -> /Remote_Right_Hand/JOY_Y
- C30 pad 2: 3.3V_REG -> /Remote_Left_Hand/3.3V_REG
- C31 pad 2: 3.3V_REG -> /Remote_Left_Hand/3.3V_REG
- C32 pad 2: 3.3V_REG -> /Remote_Left_Hand/3.3V_REG
- C35 pad 2: CHARGER_OUT -> /Remote_Left_Hand/CHARGER_OUT
- C36 pad 1: GND -> /Remote_Left_Hand/JST_BAT+
- C36 pad 2: JST_BAT+ -> GND
- C4 pad 2: 3.3V_REG -> /Remote_Right_Hand/3.3V_REG
- C5 pad 2: JOY_SWITCH -> /Remote_Right_Hand/JOY_SWITCH
- C6 pad 2: POT_1 -> /Remote_Right_Hand/VOL_POT
- C7 pad 2: 3.3V_REG -> /Remote_Right_Hand/3.3V_REG
- C8 pad 2: 3.3V_REG -> /Remote_Right_Hand/3.3V_REG
- C9 pad 2: 3.3V_REG -> /Remote_Right_Hand/3.3V_REG
- D1 pad 4: 3.3V_REG -> /Remote_Right_Hand/3.3V_REG
- D2 pad 4: 3.3V_REG -> /Remote_Right_Hand/3.3V_REG
- D3 pad 4: 3.3V_REG -> /Remote_Right_Hand/3.3V_REG
- D4 pad 4: 3.3V_REG -> /Remote_Left_Hand/3.3V_REG
- D5 pad 4: 3.3V_REG -> /Remote_Left_Hand/3.3V_REG
- D6 pad 4: 3.3V_REG -> /Remote_Left_Hand/3.3V_REG
- IC1 pad 13: unconnected-(IC1-DIO1-Pad13) -> /Remote_Right_Hand/DIO1
- IC1 pad 14: BUSY -> /Remote_Right_Hand/BUSY
- IC1 pad 15: RST -> /Remote_Right_Hand/RST
- IC1 pad 16: MISO -> /Remote_Right_Hand/MISO
- IC1 pad 17: MOSI -> /Remote_Right_Hand/MOSI
- IC1 pad 18: SCK -> /Remote_Right_Hand/SCK
- IC1 pad 19: NSS -> /Remote_Right_Hand/NSS
- IC1 pad 6: unconnected-(IC1-RXEN-Pad6) -> /Remote_Right_Hand/RX_EN
- IC1 pad 7: unconnected-(IC1-TXEN-Pad7) -> /Remote_Right_Hand/TX_EN
- IC1 pad 9: 3.3V_REG -> /Remote_Right_Hand/3.3V_REG
- IC2 pad 13: unconnected-(IC2-DIO1-Pad13) -> /Remote_Left_Hand/DIO1
- IC2 pad 14: BUSY -> /Remote_Left_Hand/BUSY
- IC2 pad 15: RST -> /Remote_Left_Hand/RST
- IC2 pad 16: MISO -> /Remote_Left_Hand/MISO
- IC2 pad 17: MOSI -> /Remote_Left_Hand/MOSI
- IC2 pad 18: SCK -> /Remote_Left_Hand/SCK
- IC2 pad 19: NSS -> /Remote_Left_Hand/NSS
- IC2 pad 6: unconnected-(IC2-RXEN-Pad6) -> /Remote_Left_Hand/RX_EN
- IC2 pad 7: unconnected-(IC2-TXEN-Pad7) -> /Remote_Left_Hand/TX_EN
- IC2 pad 9: 3.3V_REG -> /Remote_Left_Hand/3.3V_REG
- J1 pad A6: D+ -> /Remote_Right_Hand/D+
- J1 pad A7: D- -> /Remote_Right_Hand/D-
- J1 pad B6: D+ -> /Remote_Right_Hand/D+
- J1 pad B7: D- -> /Remote_Right_Hand/D-
- J2 pad 1: JST_BAT+ -> /Remote_Right_Hand/JST_BAT+
- J3 pad A6: D+ -> /Remote_Left_Hand/D+
- J3 pad A7: D- -> /Remote_Left_Hand/D-
- J3 pad B6: D+ -> /Remote_Left_Hand/D+
- J3 pad B7: D- -> /Remote_Left_Hand/D-
- J4 pad 1: JST_BAT+ -> /Remote_Left_Hand/JST_BAT+
- R13 pad 2: JST_BAT+ -> /Remote_Right_Hand/JST_BAT+
- R17 pad 1: JOY_SWITCH -> /Remote_Left_Hand/JOY_SWITCH
- R17 pad 2: 3.3V_REG -> /Remote_Left_Hand/3.3V_REG
- R18 pad 2: NEOPIXEL -> /Remote_Left_Hand/NEOPIXEL
- R19 pad 1: BOOT -> /Remote_Left_Hand/BOOT
- R19 pad 2: 3.3V_REG -> /Remote_Left_Hand/3.3V_REG
- R2 pad 1: JOY_SWITCH -> /Remote_Right_Hand/JOY_SWITCH
- R2 pad 2: 3.3V_REG -> /Remote_Right_Hand/3.3V_REG
- R20 pad 1: 3.3V_REG -> /Remote_Left_Hand/3.3V_REG
- R20 pad 2: POT_1 -> /Remote_Left_Hand/VOL_POT
- R23 pad 1: Net-(U6-EN) -> /Remote_Left_Hand/EN
- R23 pad 2: 3.3V_REG -> /Remote_Left_Hand/3.3V_REG
- R28 pad 2: JST_BAT+ -> /Remote_Left_Hand/JST_BAT+
- R3 pad 2: NEOPIXEL -> /Remote_Right_Hand/NEOPIXEL
- R4 pad 1: BOOT -> /Remote_Right_Hand/BOOT
- R4 pad 2: 3.3V_REG -> /Remote_Right_Hand/3.3V_REG
- R5 pad 1: 3.3V_REG -> /Remote_Right_Hand/3.3V_REG
- R5 pad 2: POT_1 -> /Remote_Right_Hand/VOL_POT
- R8 pad 1: Net-(U2-EN) -> /Remote_Right_Hand/EN
- R8 pad 2: 3.3V_REG -> /Remote_Right_Hand/3.3V_REG
- S1 pad A1: JOY_SWITCH -> /Remote_Right_Hand/JOY_SWITCH
- S1 pad A12: JOY_X -> /Remote_Right_Hand/JOY_X
- S1 pad A13: 3.3V_REG -> /Remote_Right_Hand/3.3V_REG
- S1 pad B12: JOY_Y -> /Remote_Right_Hand/JOY_Y
- S1 pad B13: 3.3V_REG -> /Remote_Right_Hand/3.3V_REG
- S1 pad C1: JOY_SWITCH -> /Remote_Right_Hand/JOY_SWITCH
- S2 pad A1: JOY_SWITCH -> /Remote_Left_Hand/JOY_SWITCH
- S2 pad A12: JOY_X -> /Remote_Left_Hand/JOY_X
- S2 pad A13: 3.3V_REG -> /Remote_Left_Hand/3.3V_REG
- S2 pad B12: JOY_Y -> /Remote_Left_Hand/JOY_Y
- S2 pad B13: 3.3V_REG -> /Remote_Left_Hand/3.3V_REG
- S2 pad C1: JOY_SWITCH -> /Remote_Left_Hand/JOY_SWITCH
- SW1 pad 1: BTN_1 -> /Remote_Right_Hand/BTN_1
- SW10 pad 1: BOOT -> /Remote_Right_Hand/BOOT
- SW11 pad 1: CHARGER_OUT -> /Remote_Right_Hand/CHARGER_OUT
- SW11 pad 2: BAT+_SWITCHED -> /Remote_Right_Hand/BAT+_SWITCHED
- SW12 pad 1: BTN_1 -> /Remote_Left_Hand/BTN_1
- SW13 pad 1: BTN_2 -> /Remote_Left_Hand/BTN_2
- SW14 pad 1: BTN_3 -> /Remote_Left_Hand/BTN_3
- SW15 pad 1: BTN_4 -> /Remote_Left_Hand/BTN_4
- SW16 pad 1: BTN_5 -> /Remote_Left_Hand/BTN_5
- SW17 pad 1: BTN_6 -> /Remote_Left_Hand/BTN_6
- SW18 pad 1: BTN_7 -> /Remote_Left_Hand/BTN_7
- SW19 pad 1: BTN_8 -> /Remote_Left_Hand/BTN_8
- SW2 pad 1: BTN_2 -> /Remote_Right_Hand/BTN_2
- SW20 pad 2: EN -> /Remote_Left_Hand/EN
- SW21 pad 1: BOOT -> /Remote_Left_Hand/BOOT
- SW22 pad 1: CHARGER_OUT -> /Remote_Left_Hand/CHARGER_OUT
- SW22 pad 2: BAT+_SWITCHED -> /Remote_Left_Hand/BAT+_SWITCHED
- SW3 pad 1: BTN_3 -> /Remote_Right_Hand/BTN_3
- SW4 pad 1: BTN_4 -> /Remote_Right_Hand/BTN_4
- SW5 pad 1: BTN_5 -> /Remote_Right_Hand/BTN_5
- SW6 pad 1: BTN_6 -> /Remote_Right_Hand/BTN_6
- SW7 pad 1: BTN_7 -> /Remote_Right_Hand/BTN_7
- SW8 pad 1: BTN_8 -> /Remote_Right_Hand/BTN_8
- SW9 pad 2: EN -> /Remote_Right_Hand/EN
- U1 pad 1: BAT+_SWITCHED -> /Remote_Right_Hand/BAT+_SWITCHED
- U1 pad 3: BAT+_SWITCHED -> /Remote_Right_Hand/BAT+_SWITCHED
- U1 pad 5: 3.3V_REG -> /Remote_Right_Hand/3.3V_REG
- U2 pad 1: Net-(U2-GND-Pad1) -> GND
- U2 pad 10: BTN_4 -> /Remote_Right_Hand/BTN_4
- U2 pad 11: VOL_POT -> /Remote_Right_Hand/VOL_POT
- U2 pad 12: NEOPIXEL -> /Remote_Right_Hand/NEOPIXEL
- U2 pad 13: BTN_1 -> /Remote_Right_Hand/BTN_1
- U2 pad 14: NSS -> /Remote_Right_Hand/NSS
- U2 pad 15: MOSI -> /Remote_Right_Hand/MOSI
- U2 pad 16: SCK -> /Remote_Right_Hand/SCK
- U2 pad 17: MISO -> /Remote_Right_Hand/MISO
- U2 pad 18: RST -> /Remote_Right_Hand/RST
- U2 pad 19: BUSY -> /Remote_Right_Hand/BUSY
- U2 pad 2: Net-(U2-GND-Pad1) -> GND
- U2 pad 20: DIO1 -> /Remote_Right_Hand/DIO1
- U2 pad 21: BTN_5 -> /Remote_Right_Hand/BTN_5
- U2 pad 22: BTN_6 -> /Remote_Right_Hand/BTN_6
- U2 pad 23: D-_ESP -> /Remote_Right_Hand/D-_ESP
- U2 pad 24: D+_ESP -> /Remote_Right_Hand/D+_ESP
- U2 pad 25: BTN_7 -> /Remote_Right_Hand/BTN_7
- U2 pad 28: BTN_8 -> /Remote_Right_Hand/BTN_8
- U2 pad 29: unconnected-(U2-IO34-Pad29) -> /Remote_Right_Hand/RX_EN
- U2 pad 3: 3.3V_REG -> /Remote_Right_Hand/3.3V_REG
- U2 pad 34: unconnected-(U2-IO38-Pad34) -> /Remote_Right_Hand/TX_EN
- U2 pad 4: BOOT -> /Remote_Right_Hand/BOOT
- U2 pad 42: Net-(U2-GND-Pad1) -> GND
- U2 pad 43: Net-(U2-GND-Pad1) -> GND
- U2 pad 45: Net-(U2-EN) -> /Remote_Right_Hand/EN
- U2 pad 46: Net-(U2-GND-Pad1) -> GND
- U2 pad 47: Net-(U2-GND-Pad1) -> GND
- U2 pad 48: Net-(U2-GND-Pad1) -> GND
- U2 pad 49: Net-(U2-GND-Pad1) -> GND
- U2 pad 5: JOY_X -> /Remote_Right_Hand/JOY_X
- U2 pad 50: Net-(U2-GND-Pad1) -> GND
- U2 pad 51: Net-(U2-GND-Pad1) -> GND
- U2 pad 52: Net-(U2-GND-Pad1) -> GND
- U2 pad 53: Net-(U2-GND-Pad1) -> GND
- U2 pad 54: Net-(U2-GND-Pad1) -> GND
- U2 pad 55: Net-(U2-GND-Pad1) -> GND
- U2 pad 56: Net-(U2-GND-Pad1) -> GND
- U2 pad 57: Net-(U2-GND-Pad1) -> GND
- U2 pad 58: Net-(U2-GND-Pad1) -> GND
- U2 pad 59: Net-(U2-GND-Pad1) -> GND
- U2 pad 6: JOY_Y -> /Remote_Right_Hand/JOY_Y
- U2 pad 60: Net-(U2-GND-Pad1) -> GND
- U2 pad 61: Net-(U2-GND-Pad1) -> GND
- U2 pad 62: Net-(U2-GND-Pad1) -> GND
- U2 pad 63: Net-(U2-GND-Pad1) -> GND
- U2 pad 64: Net-(U2-GND-Pad1) -> GND
- U2 pad 65: Net-(U2-GND-Pad1) -> GND
- U2 pad 7: JOY_SWITCH -> /Remote_Right_Hand/JOY_SWITCH
- U2 pad 8: BTN_2 -> /Remote_Right_Hand/BTN_2
- U2 pad 9: BTN_3 -> /Remote_Right_Hand/BTN_3
- U3 pad 10: CHARGER_OUT -> /Remote_Right_Hand/CHARGER_OUT
- U3 pad 11: CHARGER_OUT -> /Remote_Right_Hand/CHARGER_OUT
- U3 pad 2: JST_BAT+ -> /Remote_Right_Hand/JST_BAT+
- U3 pad 3: JST_BAT+ -> /Remote_Right_Hand/JST_BAT+
- U3 pad 6: 3.3V_REG -> /Remote_Right_Hand/3.3V_REG
- U4 pad 1: D+_ESP -> /Remote_Right_Hand/D+_ESP
- U4 pad 3: D-_ESP -> /Remote_Right_Hand/D-_ESP
- U4 pad 4: D- -> /Remote_Right_Hand/D-
- U4 pad 5: 3.3V_REG -> /Remote_Right_Hand/3.3V_REG
- U4 pad 6: D+ -> /Remote_Right_Hand/D+
- U5 pad 1: BAT+_SWITCHED -> /Remote_Left_Hand/BAT+_SWITCHED
- U5 pad 3: BAT+_SWITCHED -> /Remote_Left_Hand/BAT+_SWITCHED
- U5 pad 5: 3.3V_REG -> /Remote_Left_Hand/3.3V_REG
- U6 pad 1: Net-(U6-GND-Pad1) -> GND
- U6 pad 10: BTN_4 -> /Remote_Left_Hand/BTN_4
- U6 pad 11: VOL_POT -> /Remote_Left_Hand/VOL_POT
- U6 pad 12: NEOPIXEL -> /Remote_Left_Hand/NEOPIXEL
- U6 pad 13: BTN_1 -> /Remote_Left_Hand/BTN_1
- U6 pad 14: NSS -> /Remote_Left_Hand/NSS
- U6 pad 15: MOSI -> /Remote_Left_Hand/MOSI
- U6 pad 16: SCK -> /Remote_Left_Hand/SCK
- U6 pad 17: MISO -> /Remote_Left_Hand/MISO
- U6 pad 18: RST -> /Remote_Left_Hand/RST
- U6 pad 19: BUSY -> /Remote_Left_Hand/BUSY
- U6 pad 2: Net-(U6-GND-Pad1) -> GND
- U6 pad 20: DIO1 -> /Remote_Left_Hand/DIO1
- U6 pad 21: BTN_5 -> /Remote_Left_Hand/BTN_5
- U6 pad 22: BTN_6 -> /Remote_Left_Hand/BTN_6
- U6 pad 23: D-_ESP -> /Remote_Left_Hand/D-_ESP
- U6 pad 24: D+_ESP -> /Remote_Left_Hand/D+_ESP
- U6 pad 25: BTN_7 -> /Remote_Left_Hand/BTN_7
- U6 pad 28: BTN_8 -> /Remote_Left_Hand/BTN_8
- U6 pad 29: unconnected-(U6-IO34-Pad29) -> /Remote_Left_Hand/RX_EN
- U6 pad 3: 3.3V_REG -> /Remote_Left_Hand/3.3V_REG
- U6 pad 34: unconnected-(U6-IO38-Pad34) -> /Remote_Left_Hand/TX_EN
- U6 pad 4: BOOT -> /Remote_Left_Hand/BOOT
- U6 pad 42: Net-(U6-GND-Pad1) -> GND
- U6 pad 43: Net-(U6-GND-Pad1) -> GND
- U6 pad 45: Net-(U6-EN) -> /Remote_Left_Hand/EN
- U6 pad 46: Net-(U6-GND-Pad1) -> GND
- U6 pad 47: Net-(U6-GND-Pad1) -> GND
- U6 pad 48: Net-(U6-GND-Pad1) -> GND
- U6 pad 49: Net-(U6-GND-Pad1) -> GND
- U6 pad 5: JOY_X -> /Remote_Left_Hand/JOY_X
- U6 pad 50: Net-(U6-GND-Pad1) -> GND
- U6 pad 51: Net-(U6-GND-Pad1) -> GND
- U6 pad 52: Net-(U6-GND-Pad1) -> GND
- U6 pad 53: Net-(U6-GND-Pad1) -> GND
- U6 pad 54: Net-(U6-GND-Pad1) -> GND
- U6 pad 55: Net-(U6-GND-Pad1) -> GND
- U6 pad 56: Net-(U6-GND-Pad1) -> GND
- U6 pad 57: Net-(U6-GND-Pad1) -> GND
- U6 pad 58: Net-(U6-GND-Pad1) -> GND
- U6 pad 59: Net-(U6-GND-Pad1) -> GND
- U6 pad 6: JOY_Y -> /Remote_Left_Hand/JOY_Y
- U6 pad 60: Net-(U6-GND-Pad1) -> GND
- U6 pad 61: Net-(U6-GND-Pad1) -> GND
- U6 pad 62: Net-(U6-GND-Pad1) -> GND
- U6 pad 63: Net-(U6-GND-Pad1) -> GND
- U6 pad 64: Net-(U6-GND-Pad1) -> GND
- U6 pad 65: Net-(U6-GND-Pad1) -> GND
- U6 pad 7: JOY_SWITCH -> /Remote_Left_Hand/JOY_SWITCH
- U6 pad 8: BTN_2 -> /Remote_Left_Hand/BTN_2
- U6 pad 9: BTN_3 -> /Remote_Left_Hand/BTN_3
- U7 pad 10: CHARGER_OUT -> /Remote_Left_Hand/CHARGER_OUT
- U7 pad 11: CHARGER_OUT -> /Remote_Left_Hand/CHARGER_OUT
- U7 pad 2: JST_BAT+ -> /Remote_Left_Hand/JST_BAT+
- U7 pad 3: JST_BAT+ -> /Remote_Left_Hand/JST_BAT+
- U7 pad 6: 3.3V_REG -> /Remote_Left_Hand/3.3V_REG
- U8 pad 1: D+_ESP -> /Remote_Left_Hand/D+_ESP
- U8 pad 3: D-_ESP -> /Remote_Left_Hand/D-_ESP
- U8 pad 4: D- -> /Remote_Left_Hand/D-
- U8 pad 5: 3.3V_REG -> /Remote_Left_Hand/3.3V_REG
- U8 pad 6: D+ -> /Remote_Left_Hand/D+
Routing:
- net GND: track 0.00 -> 684.3 mm, vias 0 -> 30
- net /Remote_Left_Hand/3.3V_REG: track 0.00 -> 230.5 mm, vias 0 -> 5
- net /Remote_Right_Hand/3.3V_REG: track 0.00 -> 226.4 mm, vias 0 -> 3
- net VBUS: track 0.00 -> 107.7 mm, vias 0 -> 6
- net /Remote_Right_Hand/D1-D2: track 0.00 -> 106.8 mm, vias 0 -> 2
- net /Remote_Left_Hand/D1-D2: track 0.00 -> 99.8 mm, vias 0 -> 2
- net /Remote_Left_Hand/NEOPIXEL: track 0.00 -> 91.0 mm, vias 0 -> 2
- net /Remote_Right_Hand/NEOPIXEL: track 0.00 -> 77.8 mm, vias 0 -> 2
- net /Remote_Right_Hand/BTN_4: track 0.00 -> 73.5 mm, vias 0 -> 2
- net /Remote_Right_Hand/D+_ESP: track 0.00 -> 72.8 mm, vias 0 -> 2
- net /Remote_Right_Hand/D-_ESP: track 0.00 -> 70.7 mm, vias 0 -> 2
- net /Remote_Left_Hand/D+_ESP: track 0.00 -> 68.1 mm, vias 0 -> 2
- net /Remote_Right_Hand/BTN_8: track 0.00 -> 68.1 mm, vias 0 -> 2
- net /Remote_Left_Hand/BTN_4: track 0.00 -> 67.2 mm, vias 0 -> 2
- net /Remote_Left_Hand/BTN_8: track 0.00 -> 66.8 mm, vias 0 -> 2
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- added copper zone on In1.Cu, net GND
- added copper zone on In2.Cu, net GND
Other:
- outline, holes or cut-outs redrawn
