File: R2_HH_Controllers/R2_HH_Controllers.kicad_pcb (KiCad board)
At the start: 4 copper layers, 56.5 x 111 mm, 122 parts, among them IC1 E22-900M22S, IC2 E22-900M22S, J1 USB4105-GF-A, J2 S2B-PH-SM4-TB_LF__SN_, J3 USB4105-GF-A, J4 S2B-PH-SM4-TB_LF__SN_, SW1 SW_Push, SW10 Boot, SW11 PCM12SMTR, SW12 SW_Push, SW13 SW_Push, SW14 SW_Push, SW15 SW_Push, SW16 SW_Push, SW17 SW_Push, SW18 SW_Push, SW19 SW_Push, SW2 SW_Push, SW20 Reset, SW21 Boot, SW22 PCM12SMTR, SW3 SW_Push, SW4 SW_Push, SW5 SW_Push, SW6 SW_Push, SW7 SW_Push, SW8 SW_Push, SW9 Reset, U1 AP2112K-3.3, U2 ESP32-S3-MINI-1, U3 BQ24074RGT, U4 USBLC6-2SC6, U5 AP2112K-3.3, U6 ESP32-S3-MINI-1, U7 BQ24074RGT, U8 USBLC6-2SC6

Commit message: updates
Parts:
- removed C11, C13, C29, C31: 1uf, Capacitor_SMD:C_0603_1608Metric
- removed C15: .1uf, Capacitor_SMD:C_0603_1608Metric
- removed U1, U5: AP2112K-3.3, Package_TO_SOT_SMD:SOT-23-5
- added C37: 1uf, Capacitor_SMD:C_0805_2012Metric_Pad1.18x1.45mm_HandSolder, B.Cu at (145.5, 124.5)
- added C38: 1uf, Capacitor_SMD:C_0805_2012Metric_Pad1.18x1.45mm_HandSolder, B.Cu at (158.0, 125.5)
- added C39: 220nf, Capacitor_SMD:C_0603_1608Metric, F.Cu at (164.0, 91.0)
- added C40: 22uf, Capacitor_SMD:C_0603_1608Metric, F.Cu at (142.1, 95.3)
- added C41: 22uf, Capacitor_SMD:C_0603_1608Metric, F.Cu at (170.8, 93.0)
- added C42: 10uf, Capacitor_SMD:C_0603_1608Metric, F.Cu at (138.9, 89.8)
- added C43: 10uf, Capacitor_SMD:C_0603_1608Metric, F.Cu at (167.5, 88.0)
- added L1: .47uH, Inductor_SMD:L_0603_1608Metric, F.Cu at (141.1, 92.8)
- added L2: .47uH, Inductor_SMD:L_0603_1608Metric, F.Cu at (170.8, 91.0)
- added R31: 470K, Resistor_SMD:R_0805_2012Metric_Pad1.20x1.40mm_HandSolder, B.Cu at (164.0, 126.0)
- added R32: 470K, Resistor_SMD:R_0805_2012Metric_Pad1.20x1.40mm_HandSolder, B.Cu at (141.5, 123.0)
- added R33: 470K, Resistor_SMD:R_0805_2012Metric_Pad1.20x1.40mm_HandSolder, B.Cu at (164.0, 124.0)
- added R34: 200K, Resistor_SMD:R_0603_1608Metric, F.Cu at (164.3, 88.0)
- added R35: 100K, Resistor_SMD:R_0603_1608Metric, F.Cu at (134.9, 90.3)
- added R36: 100K, Resistor_SMD:R_0603_1608Metric, F.Cu at (164.0, 89.5)
- added R37: 511K, Resistor_SMD:R_0603_1608Metric, F.Cu at (134.9, 94.3)
- added R38: 511K, Resistor_SMD:R_0603_1608Metric, F.Cu at (164.3, 93.0)
- added R39: 91K, Resistor_SMD:R_0603_1608Metric, F.Cu at (134.9, 95.8)
- added R40: 91K, Resistor_SMD:R_0603_1608Metric, F.Cu at (164.1, 95.0)
- added R41: 100K, Resistor_SMD:R_0603_1608Metric, F.Cu at (138.6, 95.3)
- added R42: 100K, Resistor_SMD:R_0603_1608Metric, F.Cu at (167.3, 94.0)
- added U11: ESP32-S3-MINI-1-N8, 01-Custom:XCVR_ESP32-S3-MINI-1-N8, F.Cu at (165.3, 69.0)
- added U9: ESP32-S3-MINI-1-N8, 01-Custom:XCVR_ESP32-S3-MINI-1-N8, F.Cu at (138.7, 68.8)
- C33: value .1uf -> 220nf
- D1, D2, D3, D4, D5, D6: footprint LED_SMD:LED_WS2812B-2020_PLCC4_2.0x2.0mm -> 01-Custom:LED_WS2812B-2020_PLCC4_2.0x2.0mm
- E1, E2: footprint custom:XDCR_ANT-915-USP410 -> 01-Custom:XDCR_ANT-915-USP410
- IC1, IC2: footprint custom:E22-900M22S -> 01-Custom:E22-900M22S
- R13: value 10K -> 200K
- R24, R9: value 17.8K -> 3K
- R28: value 10K -> 470K; footprint Resistor_SMD:R_0603_1608Metric -> Resistor_SMD:R_0805_2012Metric_Pad1.20x1.40mm_HandSolder; moved to B.Cu
- SW1, SW12, SW13, SW14, SW15, SW16, SW17, SW18, SW19, SW2, SW3, SW4, SW5, SW6, SW7, SW8: footprint 01-Custom:TL3360CF185Q -> 01-Custom:SW_TL3360AF185Q
- U2, U6: value ESP32-S3-MINI-1 -> TPS63802DLAR; footprint 01-Custom:ESP32-S2-MINI-1 -> 01-Custom:VREG_TPS63802DLAR
- moved R28 32.6 mm to (141.5, 125.0), turned to 0 degrees
- moved C33 29.5 mm to (134.9, 91.8), turned to 0 degrees
- moved U2 21.4 mm to (138.1, 92.8), turned to 0 degrees
- moved U6 19.7 mm to (167.3, 91.0), turned to 0 degrees
- moved R13 10.1 mm to (134.9, 88.8), turned to 0 degrees
- moved E1 7.95 mm to (137.2, 21.8)
- moved E2 7.89 mm to (166.5, 21.8)
- moved R9 5.11 mm to (136.4, 98.3)
- moved C34 5.02 mm to (166.8, 97.8)
- moved C35 5.02 mm to (169.4, 102.5)
- moved R24 5.02 mm to (163.2, 97.4)
- moved R25 5.02 mm to (169.0, 99.8)
- moved R26 5.02 mm to (161.4, 98.5)
- moved R29 5.02 mm to (160.2, 101.3)
- moved U7 5.02 mm to (164.7, 102.2)
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Connections:
- C33 pad 2: Net-(U7-TMR) -> Net-(U2-EN)
- R13 pad 1: Net-(U3-TS) -> Net-(U2-EN)
- R13 pad 2: /Remote_Right_Hand/JST_BAT+ -> /Remote_Right_Hand/BAT+_SWITCHED
- R28 pad 1: Net-(U7-TS) -> GND
- R28 pad 2: /Remote_Left_Hand/JST_BAT+ -> /Remote_Right_Hand/VBAT_SENSE
- U2 pad 1: GND -> Net-(U2-EN)
- U2 pad 10: /Remote_Right_Hand/BTN_4 -> /Remote_Right_Hand/BAT+_SWITCHED
- U2 pad 3: /Remote_Right_Hand/3.3V_REG -> GND
- U2 pad 4: /Remote_Right_Hand/BOOT -> Net-(U2-FB)
- U2 pad 5: /Remote_Right_Hand/JOY_X -> Net-(U2-PG)
- U2 pad 6: /Remote_Right_Hand/JOY_Y -> /Remote_Right_Hand/3.3V_REG
- U2 pad 7: /Remote_Right_Hand/JOY_SWITCH -> Net-(U2-L2)
- U2 pad 8: /Remote_Right_Hand/BTN_2 -> GND
- U2 pad 9: /Remote_Right_Hand/BTN_3 -> Net-(U2-L1)
- U3 pad 14: Net-(U3-TMR) -> unconnected-(U3-TMR-Pad14)
- U3 pad 5: GND -> /Remote_Right_Hand/CHARGER_OUT
- U3 pad 6: /Remote_Right_Hand/3.3V_REG -> GND
- U3 pad 7: unconnected-(U3-~{PGOOD}-Pad7) -> /Remote_Right_Hand/PWR_GOOD
- U3 pad 9: unconnected-(U3-~{CHG}-Pad9) -> /Remote_Right_Hand/CHG_STAT
- U6 pad 1: GND -> Net-(U6-EN)
- U6 pad 10: /Remote_Left_Hand/BTN_4 -> /Remote_Left_Hand/BAT+_SWITCHED
- U6 pad 3: /Remote_Left_Hand/3.3V_REG -> GND
- U6 pad 4: /Remote_Left_Hand/BOOT -> Net-(U6-FB)
- U6 pad 5: /Remote_Left_Hand/JOY_X -> Net-(U6-PG)
- U6 pad 6: /Remote_Left_Hand/JOY_Y -> /Remote_Left_Hand/3.3V_REG
- U6 pad 7: /Remote_Left_Hand/JOY_SWITCH -> Net-(U6-L2)
- U6 pad 8: /Remote_Left_Hand/BTN_2 -> GND
- U6 pad 9: /Remote_Left_Hand/BTN_3 -> Net-(U6-L1)
- U7 pad 14: Net-(U7-TMR) -> unconnected-(U7-TMR-Pad14)
- U7 pad 5: GND -> /Remote_Left_Hand/CHARGER_OUT
- U7 pad 6: /Remote_Left_Hand/3.3V_REG -> GND
- U7 pad 7: unconnected-(U7-~{PGOOD}-Pad7) -> /Remote_Left_Hand/PWR_GOOD
- U7 pad 9: unconnected-(U7-~{CHG}-Pad9) -> /Remote_Left_Hand/CHG_STAT
Routing:
- net GND: track 684.3 -> 791.9 mm
- net /Remote_Right_Hand/VBAT_SENSE: track 0.00 -> 100.8 mm, vias 0 -> 2
- net /Remote_Left_Hand/VBAT_SENSE: track 0.00 -> 82.8 mm, vias 0 -> 2
- net /Remote_Right_Hand/CHG_STAT: track 0.00 -> 50.0 mm, vias 0 -> 3
- net /Remote_Left_Hand/CHG_STAT: track 0.00 -> 48.4 mm, vias 0 -> 2
- net /Remote_Left_Hand/PWR_GOOD: track 0.00 -> 47.4 mm, vias 0 -> 2
- net /Remote_Right_Hand/PWR_GOOD: track 0.00 -> 47.0 mm, vias 0 -> 3
- net /Remote_Left_Hand/BTN_1: track 3.75 -> 32.3 mm
- net /Remote_Right_Hand/BTN_1: track 32.4 -> 9.14 mm, vias 2 -> 0
- net /Remote_Left_Hand/3.3V_REG: track 230.5 -> 250.4 mm
- net /Remote_Left_Hand/BAT+_SWITCHED: track 37.6 -> 52.1 mm, vias 2 -> 3
- net /Remote_Right_Hand/BAT+_SWITCHED: track 45.3 -> 58.7 mm
- net /Remote_Left_Hand/JST_BAT+: track 37.1 -> 48.2 mm
- net VBUS: track 107.7 -> 98.4 mm
- net Net-(U2-EN): track 0.00 -> 8.34 mm
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Other:
- board size 56.5 x 111 mm -> 56.5 x 119.5 mm
- board text added: "NaviHilt Left Hand Controller V1.1"
- board text added: "NaviHilt Right Hand Controller V1.0"
